File: proj/Synth.sch (KiCad schematic (older format))
At the start: 0 parts

Commit message: Add synth schematic
Parts:
- added C? (x2): 15p, IPC7351-Nominal:CAPC1005X55, symbol C-0402
- added C?: 680p, IPC7351-Nominal:CAPC1608X55, symbol C-0603
- added C? (x10): 1n, IPC7351-Nominal:CAPC1005X55, symbol C-0402
- added C? (x8): 220n, IPC7351-Nominal:CAPC2012X70, symbol C-0805
- added C? (x2): 10u, IPC7351-Nominal:CAPC2012X70, symbol C-0805
- added R? (x2): 100, IPC7351-Nominal:RESC1005X40, symbol R-0402
- added R?: 1k91, IPC7351-Nominal:RESC1005X40, symbol R-0402
- added R? (x6): 49R9, IPC7351-Nominal:RESC1005X40, symbol R-0402
- added R? (x4): 53R6, IPC7351-Nominal:RESC1005X40, symbol R-0402
- added R? (x8): 360, IPC7351-Nominal:RESC1005X40, symbol R-0402
- added R? (x2): 2k2, IPC7351-Nominal:RESC1005X40, symbol R-0402
- added TP?: SYNC_OUT, symbol TESTPOINT
- added TP?: SYNC_CLK, symbol TESTPOINT
- added U?: AD9958BCPZ, manuf:ANALOG-LFCSP-VQ-56, symbol AD9958BCPZ
- added U? (x4): LMH6714MF, smd-semi:SOT-23-5, symbol LMH6714MF
- added X?: 25 MHz, IPC7351-Nominal:XTAL1200X480X460, symbol XTAL-HC49US-SMD
Connections:
- new net: R?.2, R?.2, R?.2, U?.13 (CH1_IOUTp)
- new net: R?.2, R?.2, R?.2, U?.14 (CH2_IOUTn)
- new net: R?.1, U?.17 (DAC_RSET)
- new net: R?.1, U?.2 (SYNC_OUT)
- new net: C?.1, U?.22 (REFCLKn), X?.2
- new net: C?.1, U?.23 (REFCLKp), X?.1
- new net: C?.1, U?.27 (LOOP_FILTER)
- new net: R?.2, U?.54 (SYNC_CLK)
- new net: R?.2, R?.2, R?.2, U?.8 (CH0_IOUTp)
- new net: R?.2, R?.2, R?.2, U?.9 (CH0_IOUTn)
- new net: R?.2, TP?.1
- new net: R?.1, TP?.1
- new net: R?.1, R?.2, U?.4 (x2)
- new net: R?.1, R?.1, R?.2, U?.1 (x2)
- new net: R?.1, R?.2, U?.3 (x2)
- new net #CS: U?.47 (#CS)
- new net +1.8: C?.1, C?.1, C?.1, U?.45 (DVDD), U?.55 (DVDD)
- new net +1.8A: C?.1, C?.1, C?.1, C?.1, C?.1, C?.1, C?.1, C?.1, R?.1, R?.1, R?.1, R?.1, R?.1, R?.1, R?.1, R?.1, U?.11 (AVDD), U?.15 (AVDD), U?.19 (AVDD), U?.21 (AVDD), U?.24 (CLK_MODE_SEL), U?.26 (AVDD), U?.29 (AVDD), U?.30 (AVDD), U?.31 (AVDD), U?.33 (AVDD), U?.35 (AVDD), U?.36 (AVDD), U?.37 (AVDD), U?.39 (AVDD), U?.5 (AVDD), U?.7 (AVDD)
- new net +3.3: C?.1, U?.49 (DVDDIO)
- new net +5: C?.1, C?.1, C?.1, C?.1, C?.1, U?.5 (V+), U?.5 (V+)
- new net -5: C?.2, C?.2, C?.2, C?.2, C?.2, R?.2, R?.2, U?.2 (V-), U?.2 (V-)
- new net GND: C?.1, C?.1, C?.1, C?.2, C?.2, C?.2, C?.2, C?.2, C?.2, C?.2, C?.2, C?.2, C?.2, C?.2, C?.2, C?.2, C?.2, C?.2, C?.2, C?.2, C?.2, R?.1, R?.1, R?.2, U?.10 (AGND), U?.12 (AGND), U?.16 (AGND), U?.18 (AGND), U?.20 (AGND), U?.25 (AGND), U?.40 (P0), U?.41 (P1), U?.42 (P2), U?.43 (P3), U?.44 (DGND), U?.56 (DGND), U?.57 (AGND), U?.6 (AGND)
- new net IO_UPDATE: U?.46 (IO_UPDATE)
- new net MASTER_RESET: U?.3 (MASTER_RESET)
- new net OUT1: R?.1
- new net OUT2: R?.1
- new net PWR_DWN_CTL: U?.4 (PWR_DWN_CTL)
- new net SCLK: U?.48 (SCLK)
- new net SDIO_0: U?.50 (SDIO_0)
- new net SDIO_1: U?.51 (SDIO_1)
- new net SDIO_2: U?.52 (SDIO_2)
- new net SDIO_3: U?.53 (SDIO_3)
- no-connect marks 0 -> 1
Other:
- note added: "Differential T-line\nZdiff = 100, Z0 = 67\nSpecs for OSH Park 4L:\n0.1415 track, 0.1584 space (0.299 align)"
- note added: "Floating SYNC_IN is intentional.\nSee AD9958 datasheet page 29."
- note added: "Single-ended T-line\nZ0 = 50"

Commit message: Add power input circuit
Parts:
- gave numbers to parts that had none: 52

Commit message: Finish USB subcircuit
Parts:
- added E?: 2k2@100, IPC7351-Nominal:INDC2012X130, symbol BEAD-0805
Connections:
- net +1.8: now also E?.1
- net +1.8A: now also E?.2
- net CH1_P: now reaches R17.2, R20.2, R25.2, U4.13 (CH1_IOUTp)
- net CH1_N: now reaches R18.2, R22.2, R26.2, U4.14 (CH2_IOUTn)
- net CH0_P: now reaches R13.2, R19.2, R23.2, U4.8 (CH0_IOUTp)
- net CH0_N: now reaches R15.2, R21.2, R24.2, U4.9 (CH0_IOUTn)
Changed lines of the file:
@@
 $Descr USLegal 14000 8500
 encoding utf-8
-Sheet 6 14
+Sheet 4 13
 Title "Synthesizer"
 Date "2015-02-28"
@@
 $EndComp
 Wire Wire Line
-	4500 2250 4500 2300
-Wire Wire Line
-	4500 2300 4500 2400
-Wire Wire Line
-	4500 2300 4600 2300
-Wire Wire Line
-	4600 2300 4700 2300
-Wire Wire Line
-	4700 2300 4800 2300
-Wire Wire Line
-	4800 2300 4900 2300
-Wire Wire Line
-	4900 2300 5000 2300
-Wire Wire Line
-	5000 2300 5100 2300
-Wire Wire Line
-	5100 2300 5200 2300
-Wire Wire Line
-	5200 2300 5300 2300
-Wire Wire Line
-	5300 2300 5400 2300
-Wire Wire Line
-	5400 2300 5500 2300
-Wire Wire Line
-	5500 2300 5600 2300
-Wire Wire Line
-	5600 2300 5700 2300
-Wire Wire Line
-	5700 2300 5800 2300
-Wire Wire Line
-	5800 2300 5900 2300
+	4500 2250 4500 2400
+Wire Wire Line
+	4500 2300 5900 2300
 Wire Wire Line
 	5900 2300 5900 2400
@@
 Connection ~ 4600 2300
 Wire Wire Line
-	6100 2250 6100 2300
-Wire Wire Line
-	6100 2300 6100 2400
+	6100 2250 6100 2400
 Wire Wire Line
 	6100 2300 6200 2300
@@
 	4200 3100 1350 3100
 Wire Wire Line
-	2600 3300 2950 3300
-Wire Wire Line
-	2950 3300 4200 3300
-Wire Wire Line
-	2600 3600 2950 3600
-Wire Wire Line
-	2950 3600 3200 3600
+	2600 3300 4200 3300
+Wire Wire Line
+	2600 3600 3200 3600
 Wire Wire Line
 	3200 3600 3200 3400
@@
 	2400 3300 2300 3300
 Wire Wire Line
-	2300 3300 2300 3450
-Wire Wire Line
-	2300 3450 2300 3600
+	2300 3300 2300 3600
 Wire Wire Line
 	2300 3600 2400 3600
@@
 	4200 4100 4100 4100
 Wire Wire Line
-	4100 4100 4100 4200
-Wire Wire Line
-	4100 4200 4100 4300
-Wire Wire Line
-	4100 4300 4100 4400
-Wire Wire Line
-	4100 4400 4100 4450
+	4100 4100 4100 4450
 Wire Wire Line
 	4100 4400 4200 4400
@@
 	6700 2850 6700 3000
 Wire Wire Line
-	9650 3000 6700 3000
-Wire Wire Line
-	6700 3000 6600 3000
+	9650 3000 6600 3000
 Wire Wire Line
 	6900 2850 6900 3100
 Wire Wire Line
-	9750 3100 6900 3100
-Wire Wire Line
-	6900 3100 6600 3100
+	9750 3100 6600 3100
 Wire Wire Line
 	7200 2850 7200 3300
 Wire Wire Line
-	6600 3300 7200 3300
-Wire Wire Line
-	7200 3300 7900 3300
+	6600 3300 7900 3300
 Wire Wire Line
 	7400 2850 7400 3400
 Wire Wire Line
-	6600 3400 7400 3400
-Wire Wire Line
-	7400 3400 7800 3400
+	6600 3400 7800 3400
 Wire Wire Line
 	6700 2650 6700 2550
 Wire Wire Line
-	6700 2550 6800 2550
-Wire Wire Line
-	6800 2550 6900 2550
+	6700 2550 6900 2550
 Wire Wire Line
 	6900 2550 6900 2650
@@
 	7200 2650 7200 2550
 Wire Wire Line
-	7200 2550 7300 2550
-Wire Wire Line
-	7300 2550 7400 2550
+	7200 2550 7400 2550
 Wire Wire Line
 	7400 2550 7400 2650
@@
 	9650 1500 9650 1400
 Wire Wire Line
-	9650 1400 9700 1400
-Wire Wire Line
-	9700 1400 9750 1400
+	9650 1400 9750 1400
 Wire Wire Line
 	9750 1400 9750 1500
@@
 Connection ~ 9700 1400
 Wire Wire Line
-	9650 1700 9650 1800
-Wire Wire Line
-	9650 1800 9650 3000
-Wire Wire Line
-	9750 1700 9750 2500
-Wire Wire Line
-	9750 2500 9750 3100
+	9650 1700 9650 3000
+Wire Wire Line
+	9750 1700 9750 3100
 Connection ~ 6900 3100
 Wire Wire Line
@@
 Connection ~ 9650 1800
 Wire Wire Line
-	10650 1800 10850 1800
-Wire Wire Line
-	10850 1800 11350 1800
+	10650 1800 11350 1800
 Wire Wire Line
 	10450 2500 9750 2500
 Connection ~ 9750 2500
 Wire Wire Line
-	10650 2500 10850 2500
-Wire Wire Line
-	10850 2500 11350 2500
+	10650 2500 11350 2500
 Wire Wire Line
 	11050 2050 10850 2050
@@
 Connection ~ 10850 2500
 Wire Wire Line
-	11550 1800 11650 1800
-Wire Wire Line
-	11650 1800 11850 1800
-Wire Wire Line
-	11650 1800 11650 2150
-Wire Wire Line
-	11650 2150 11650 2550
+	11550 1800 11850 1800
+Wire Wire Line
+	11650 1800 11650 2550
 Wire Wire Line
 	11650 2150 11550 2150
@@
 	12600 1800 12050 1800
 Wire Wire Line
-	12500 1850 12500 2500
-Wire Wire Line
-	12500 2500 12500 2550
+	12500 1850 12500 2550
 Wire Wire Line
 	12500 2500 11550 2500
@@
 	9650 3500 9650 3400
 Wire Wire Line
-	9650 3400 9700 3400
-Wire Wire Line
-	9700 3400 9750 3400
+	9650 3400 9750 3400
 Wire Wire Line
 	9750 3400 9750 3500
@@
 	10450 3800 9650 3800
 Wire Wire Line
-	10650 3800 10850 3800
-Wire Wire Line
-	10850 3800 11350 3800
+	10650 3800 11350 3800
 Wire Wire Line
 	10450 4500 9750 4500
 Wire Wire Line
-	10650 4500 10850 4500
-Wire Wire Line
-	10850 4500 11350 4500
+	10650 4500 11350 4500
 Wire Wire Line
 	11050 4050 10850 4050
@@
 Connection ~ 10850 4500
 Wire Wire Line
-	11550 3800 11650 3800
-Wire Wire Line
-	11650 3800 11850 3800
-Wire Wire Line
-	11650 3800 11650 4150
-Wire Wire Line
-	11650 4150 11650 4550
+	11550 3800 11850 3800
+Wire Wire Line
+	11650 3800 11650 4550
 Wire Wire Line
 	11650 4150 11550 4150
@@
 	12600 3800 12050 3800
 Wire Wire Line
-	12500 3850 12500 4500
-Wire Wire Line
-	12500 4500 12500 4550
+	12500 3850 12500 4550
 Wire Wire Line
 	12500 4500 11550 4500
 Connection ~ 12500 4500
 Wire Wire Line
-	9650 3700 9650 3800
-Wire Wire Line
-	9650 3800 9650 4700
+	9650 3700 9650 4700
 Wire Wire Line
 	9650 4700 7900 4700
@@
 	7800 4800 9750 4800
 Wire Wire Line
-	9750 4800 9750 4500
-Wire Wire Line
-	9750 4500 9750 3700
+	9750 4800 9750 3700
 Connection ~ 7400 3400
 Connection ~ 9650 3800
@@
 $EndComp
 Wire Wire Line
-	5700 7050 5700 7150
-Wire Wire Line
-	5700 7150 5700 7250
+	5700 7050 5700 7250
 $Comp
 L GND #PWR53
@@
 $EndComp
 Wire Wire Line
-	6900 7050 6900 7150
-Wire Wire Line
-	6900 7150 6900 7250
+	6900 7050 6900 7250
 $Comp
 L GND #PWR65
@@
 $EndComp
 Wire Wire Line
-	7400 7050 7400 7150
-Wire Wire Line
-	7400 7150 7400 7250
+	7400 7050 7400 7250
 $Comp
 L GND #PWR69
@@
 Text Notes 11500 5350 0    60   ~ 0
 Single-ended T-line\nZ0 = 50
+Text Label 8100 3000 0    50   ~ 0
+CH0_P
+Text Label 8100 3100 0    50   ~ 0
+CH0_N
+Text Label 8100 4700 0    50   ~ 0
+CH1_P
+Text Label 8100 4800 0    50   ~ 0
+CH1_N
+$Comp
+L BEAD-0805 E?
+U 1 1 54F8FF17
+P 1400 6250
+F 0 "E?" H 1400 6450 50  0000 C CNN
+F 1 "2k2@100" H 1400 6350 50  0000 C CNN
+F 2 "IPC7351-Nominal:INDC2012X130" H 1400 6250 50  0001 C CNN
+F 3 "" H 1400 6300 60  0000 C CNN
+F 4 "HZ0805B222R-10" H 1400 6250 60  0001 C CNN "PN"
+F 5 "Laird" H 1400 6250 60  0001 C CNN "Manuf"
+F 6 "DIST DIGIKEY 240-2562-1-ND" H 1400 6250 60  0001 C CNN "BOM"
+	1    1400 6250
+	1    0    0    -1
+$EndComp
+$Comp
+L +1.8 #PWR?
+U 1 1 54F9001E
+P 1100 6100
+F 0 "#PWR?" H 1100 6150 30  0001 C CNN
+F 1 "+1.8" H 1100 6200 50  0000 C CNN
+F 2 "" H 1100 6100 60  0000 C CNN
+F 3 "" H 1100 6100 60  0000 C CNN
+	1    1100 6100
+	1    0    0    -1
+$EndComp
+Wire Wire Line
+	1100 6100 1100 6250
+Wire Wire Line
+	1100 6250 1300 6250
+$Comp
+L +1.8A #PWR?
+U 1 1 54F9021A
+P 1700 6100
+F 0 "#PWR?" H 1700 6150 30  0001 C CNN
+F 1 "+1.8A" H 1700 6200 50  0000 C CNN
+F 2 "" H 1700 6100 60  0000 C CNN
+F 3 "" H 1700 6100 60  0000 C CNN
+	1    1700 6100
+	1    0    0    -1
+$EndComp
+Wire Wire Line
+	1700 6100 1700 6250
+Wire Wire Line
+	1700 6250 1500 6250
 $EndSCHEMATC

Commit message: Start PCB
Parts:
- TP1, TP2: footprint (none) -> conn-test:TEST-SMD-SMALL
- gave numbers to parts that had none: 1
