File: proj/LPF.sch (KiCad schematic (older format))
At the start: 13 parts

Commit message: Add power input circuit
Parts:
- gave numbers to parts that had none: 13
Changed lines of the file:
@@
 $Descr USLegal 14000 8500
 encoding utf-8
-Sheet 7 12
+Sheet 7 13
 Title "LPF for Output Amplifier"
 Date "2015-02-28"
@@
 B
 $Comp
-L C-0402 C?
+L C-0402 C42
 U 1 1 54F2BD52
 P 5550 3700
-F 0 "C?" H 5750 3750 50  0000 C CNN
+F 0 "C42" H 5750 3750 50  0000 C CNN
 F 1 "22p" H 5750 3650 50  0000 C CNN
 F 2 "IPC7351-Nominal:CAPC1005X55" H 5550 3700 50  0001 C CNN
@@
 $EndComp
 $Comp
-L L-0402 L?
+L L-0402 L1
 U 1 1 54F2C04F
 P 6250 3400
-F 0 "L?" V 6050 3400 50  0000 C CNN
+F 0 "L1" V 6050 3400 50  0000 C CNN
 F 1 "56n" V 6150 3400 50  0000 C CNN
 F 2 "IPC7351-Nominal:INDC1005X60" H 6250 3400 50  0001 C CNN
@@
 $EndComp
 $Comp
-L C-0402 C?
+L C-0402 C43
 U 1 1 54F2C0F9
 P 5950 3700
-F 0 "C?" H 6150 3750 50  0000 C CNN
+F 0 "C43" H 6150 3750 50  0000 C CNN
 F 1 "22p" H 6150 3650 50  0000 C CNN
 F 2 "IPC7351-Nominal:CAPC1005X55" H 5950 3700 50  0001 C CNN
@@
 $EndComp
 $Comp
-L C-0402 C?
+L C-0402 C44
 U 1 1 54F2C23D
 P 6250 3050
-F 0 "C?" V 6000 3050 50  0000 C CNN
+F 0 "C44" V 6000 3050 50  0000 C CNN
 F 1 "1p5" V 6100 3050 50  0000 C CNN
 F 2 "IPC7351-Nominal:CAPC1005X55" H 6250 3050 50  0001 C CNN
@@
 $EndComp
 $Comp
-L L-0402 L?
+L L-0402 L2
 U 1 1 54F2C5D8
 P 6850 3400
-F 0 "L?" V 6650 3400 50  0000 C CNN
+F 0 "L2" V 6650 3400 50  0000 C CNN
 F 1 "47n" V 6750 3400 50  0000 C CNN
 F 2 "IPC7351-Nominal:INDC1005X60" H 6850 3400 50  0001 C CNN
@@
 $EndComp
 $Comp
-L C-0402 C?
+L C-0402 C47
 U 1 1 54F2CACC
 P 6850 3050
-F 0 "C?" V 6600 3050 50  0000 C CNN
+F 0 "C47" V 6600 3050 50  0000 C CNN
 F 1 "4p7" V 6700 3050 50  0000 C CNN
 F 2 "IPC7351-Nominal:CAPC1005X55" H 6850 3050 50  0001 C CNN
@@
 $EndComp
 $Comp
-L C-0402 C?
+L C-0402 C46
 U 1 1 54F2CB7C
 P 6850 2650
-F 0 "C?" V 6600 2650 50  0000 C CNN
+F 0 "C46" V 6600 2650 50  0000 C CNN
 F 1 "4p7" V 6700 2650 50  0000 C CNN
 F 2 "IPC7351-Nominal:CAPC1005X55" H 6850 2650 50  0001 C CNN
@@
 $EndComp
 $Comp
-L L-0402 L?
+L L-0402 L3
 U 1 1 54F2CBBD
 P 7450 3400
-F 0 "L?" V 7250 3400 50  0000 C CNN
+F 0 "L3" V 7250 3400 50  0000 C CNN
 F 1 "47n" V 7350 3400 50  0000 C CNN
 F 2 "IPC7351-Nominal:INDC1005X60" H 7450 3400 50  0001 C CNN
@@
 $EndComp
 $Comp
-L C-0402 C?
+L C-0402 C49
 U 1 1 54F2CBED
 P 7450 3050
-F 0 "C?" V 7200 3050 50  0000 C CNN
+F 0 "C49" V 7200 3050 50  0000 C CNN
 F 1 "4p7" V 7300 3050 50  0000 C CNN
 F 2 "IPC7351-Nominal:CAPC1005X55" H 7450 3050 50  0001 C CNN
@@
 $EndComp
 $Comp
-L C-0402 C?
+L C-0402 C45
 U 1 1 54F2CE50
 P 6550 3700
-F 0 "C?" H 6750 3750 50  0000 C CNN
+F 0 "C45" H 6750 3750 50  0000 C CNN
 F 1 "56p" H 6750 3650 50  0000 C CNN
 F 2 "IPC7351-Nominal:CAPC1005X55" H 6550 3700 50  0001 C CNN
@@
 $EndComp
 $Comp
-L C-0402 C?
+L C-0402 C48
 U 1 1 54F2D3A4
 P 7150 3700
-F 0 "C?" H 7350 3750 50  0000 C CNN
+F 0 "C48" H 7350 3750 50  0000 C CNN
 F 1 "56p" H 7350 3650 50  0000 C CNN
 F 2 "IPC7351-Nominal:CAPC1005X55" H 7150 3700 50  0001 C CNN
@@
 $EndComp
 $Comp
-L C-0402 C?
+L C-0402 C50
 U 1 1 54F2D3DD
 P 7750 3700
-F 0 "C?" H 7950 3750 50  0000 C CNN
+F 0 "C50" H 7950 3750 50  0000 C CNN
 F 1 "22p" H 7950 3650 50  0000 C CNN
 F 2 "IPC7351-Nominal:CAPC1005X55" H 7750 3700 50  0001 C CNN
@@
 $EndComp
 $Comp
-L C-0402 C?
+L C-0402 C51
 U 1 1 54F2D417
 P 8150 3700
-F 0 "C?" H 8350 3750 50  0000 C CNN
+F 0 "C51" H 8350 3750 50  0000 C CNN
 F 1 "18p" H 8350 3650 50  0000 C CNN
 F 2 "IPC7351-Nominal:CAPC1005X55" H 8150 3700 50  0001 C CNN
@@
 $EndComp
 $Comp
-L GND #PWR?
+L GND #PWR110
 U 1 1 54F2DC44
 P 5550 3900
-F 0 "#PWR?" H 5550 3900 30  0001 C CNN
+F 0 "#PWR110" H 5550 3900 30  0001 C CNN
 F 1 "GND" H 5550 3830 30  0001 C CNN
 F 2 "" H 5550 3900 60  0000 C CNN
@@
 	5550 3800 5550 3900
 $Comp
-L GND #PWR?
+L GND #PWR111
 U 1 1 54F2DD29
 P 5950 3900
-F 0 "#PWR?" H 5950 3900 30  0001 C CNN
+F 0 "#PWR111" H 5950 3900 30  0001 C CNN
 F 1 "GND" H 5950 3830 30  0001 C CNN
 F 2 "" H 5950 3900 60  0000 C CNN
@@
 	5950 3900 5950 3800
 $Comp
-L GND #PWR?
+L GND #PWR112
 U 1 1 54F2DD77
 P 6550 3900
-F 0 "#PWR?" H 6550 3900 30  0001 C CNN
+F 0 "#PWR112" H 6550 3900 30  0001 C CNN
 F 1 "GND" H 6550 3830 30  0001 C CNN
 F 2 "" H 6550 3900 60  0000 C CNN
@@
 	6550 3900 6550 3800
 $Comp
-L GND #PWR?
+L GND #PWR113
 U 1 1 54F2DDC6
 P 7150 3900
-F 0 "#PWR?" H 7150 3900 30  0001 C CNN
+F 0 "#PWR113" H 7150 3900 30  0001 C CNN
 F 1 "GND" H 7150 3830 30  0001 C CNN
 F 2 "" H 7150 3900 60  0000 C CNN
@@
 	7150 3900 7150 3800
 $Comp
-L GND #PWR?
+L GND #PWR114
 U 1 1 54F2DE16
 P 7750 3900
-F 0 "#PWR?" H 7750 3900 30  0001 C CNN
+F 0 "#PWR114" H 7750 3900 30  0001 C CNN
 F 1 "GND" H 7750 3830 30  0001 C CNN
 F 2 "" H 7750 3900 60  0000 C CNN
@@
 	7750 3900 7750 3800
 $Comp
-L GND #PWR?
+L GND #PWR115
 U 1 1 54F2DE67
 P 8150 3900
-F 0 "#PWR?" H 8150 3900 30  0001 C CNN
+F 0 "#PWR115" H 8150 3900 30  0001 C CNN
 F 1 "GND" H 8150 3830 30  0001 C CNN
 F 2 "" H 8150 3900 60  0000 C CNN
