File: proj/Buffer_Filter.sch (KiCad schematic (older format))
At the start: 18 parts

Commit message: Add power input circuit
Parts:
- gave numbers to parts that had none: 18
Changed lines of the file:
@@
 $Descr A4 11693 8268
 encoding utf-8
-Sheet 11 12
+Sheet 11 13
 Title "Input Buffer and Filter"
 Date "2015-02-28"
@@
 $EndDescr
 $Comp
-L R-0402 R?
+L R-0402 R70
 U 1 1 54F37119
 P 3500 3000
-F 0 "R?" H 3650 3050 50  0000 C CNN
+F 0 "R70" H 3650 3050 50  0000 C CNN
 F 1 "200" H 3650 2950 50  0000 C CNN
 F 2 "IPC7351-Nominal:RESC1005X40" H 3500 3000 50  0001 C CNN
@@
 $EndComp
 $Comp
-L R-0402 R?
+L R-0402 R71
 U 1 1 54F371B6
 P 3800 3000
-F 0 "R?" H 3950 3050 50  0000 C CNN
+F 0 "R71" H 3950 3050 50  0000 C CNN
 F 1 "200" H 3950 2950 50  0000 C CNN
 F 2 "IPC7351-Nominal:RESC1005X40" H 3800 3000 50  0001 C CNN
@@
 $EndComp
 $Comp
-L R-0402 R?
+L R-0402 R72
 U 1 1 54F371D8
 P 4100 3000
-F 0 "R?" H 4250 3050 50  0000 C CNN
+F 0 "R72" H 4250 3050 50  0000 C CNN
 F 1 "200" H 4250 2950 50  0000 C CNN
 F 2 "IPC7351-Nominal:RESC1005X40" H 4100 3000 50  0001 C CNN
@@
 $EndComp
 $Comp
-L R-0402 R?
+L R-0402 R73
 U 1 1 54F371FF
 P 4400 3000
-F 0 "R?" H 4550 3050 50  0000 C CNN
+F 0 "R73" H 4550 3050 50  0000 C CNN
 F 1 "200" H 4550 2950 50  0000 C CNN
 F 2 "IPC7351-Nominal:RESC1005X40" H 4400 3000 50  0001 C CNN
@@
 $EndComp
 $Comp
-L GND #PWR?
+L GND #PWR172
 U 1 1 54F3723B
 P 3500 3150
-F 0 "#PWR?" H 3500 3150 30  0001 C CNN
+F 0 "#PWR172" H 3500 3150 30  0001 C CNN
 F 1 "GND" H 3500 3080 30  0001 C CNN
 F 2 "" H 3500 3150 60  0000 C CNN
@@
 	3500 3150 3500 3100
 $Comp
-L GND #PWR?
+L GND #PWR173
 U 1 1 54F3725D
 P 3800 3150
-F 0 "#PWR?" H 3800 3150 30  0001 C CNN
+F 0 "#PWR173" H 3800 3150 30  0001 C CNN
 F 1 "GND" H 3800 3080 30  0001 C CNN
 F 2 "" H 3800 3150 60  0000 C CNN
@@
 	3800 3150 3800 3100
 $Comp
-L GND #PWR?
+L GND #PWR174
 U 1 1 54F37280
 P 4100 3150
-F 0 "#PWR?" H 4100 3150 30  0001 C CNN
+F 0 "#PWR174" H 4100 3150 30  0001 C CNN
 F 1 "GND" H 4100 3080 30  0001 C CNN
 F 2 "" H 4100 3150 60  0000 C CNN
@@
 	4100 3150 4100 3100
 $Comp
-L GND #PWR?
+L GND #PWR175
 U 1 1 54F372A4
 P 4400 3150
-F 0 "#PWR?" H 4400 3150 30  0001 C CNN
+F 0 "#PWR175" H 4400 3150 30  0001 C CNN
 F 1 "GND" H 4400 3080 30  0001 C CNN
 F 2 "" H 4400 3150 60  0000 C CNN
@@
 	4400 3150 4400 3100
 $Comp
-L BFR540 Q?
+L BFR540 Q11
 U 1 1 54F3761A
 P 4850 2800
-F 0 "Q?" H 5100 2850 50  0000 C CNN
+F 0 "Q11" H 5100 2850 50  0000 C CNN
 F 1 "BFR540" H 5100 2750 50  0000 C CNN
 F 2 "smd-semi:SOT-23" H 4850 2800 50  0001 C CNN
@@
 Connection ~ 3800 2800
 $Comp
-L BFR540 Q?
+L BFR540 Q12
 U 1 1 54F376D9
 P 4850 3900
-F 0 "Q?" H 5100 3950 50  0000 C CNN
+F 0 "Q12" H 5100 3950 50  0000 C CNN
 F 1 "BFR540" H 5100 3850 50  0000 C CNN
 F 2 "smd-semi:SOT-23" H 4850 3900 50  0001 C CNN
@@
 	4900 3800 4900 2900
 $Comp
-L MMBT3904 Q?
+L MMBT3904 Q10
 U 1 1 54F37ABD
 P 4700 4100
-F 0 "Q?" H 4200 4150 50  0000 C CNN
+F 0 "Q10" H 4200 4150 50  0000 C CNN
 F 1 "MMBT3904" H 4200 4050 50  0000 C CNN
 F 2 "smd-semi:SOT-23" H 4700 4100 50  0001 C CNN
@@
 	4650 3900 4650 4000
 $Comp
-L R-0402 R?
+L R-0402 R75
 U 1 1 54F37F98
 P 4900 4300
-F 0 "R?" H 5050 4350 50  0000 C CNN
+F 0 "R75" H 5050 4350 50  0000 C CNN
 F 1 "22" H 5050 4250 50  0000 C CNN
 F 2 "IPC7351-Nominal:RESC1005X40" H 4900 4300 50  0001 C CNN
@@
 Connection ~ 4900 4100
 $Comp
-L -5 #PWR?
+L -5 #PWR177
 U 1 1 54F38084
 P 4900 4600
-F 0 "#PWR?" H 4900 4550 30  0001 C CNN
+F 0 "#PWR177" H 4900 4550 30  0001 C CNN
 F 1 "-5" H 4900 4500 50  0000 C CNN
 F 2 "" H 4900 4600 60  0000 C CNN
@@
 Connection ~ 4900 4500
 $Comp
-L C-0402 C?
+L C-0402 C73
 U 1 1 54F383DE
 P 4400 4200
-F 0 "C?" H 4600 4250 50  0000 C CNN
+F 0 "C73" H 4600 4250 50  0000 C CNN
 F 1 "10n" H 4600 4150 50  0000 C CNN
 F 2 "IPC7351-Nominal:CAPC1005X55" H 4400 4200 50  0001 C CNN
@@
 Connection ~ 4650 3900
 $Comp
-L R-0402 R?
+L R-0402 R74
 U 1 1 54F3856D
 P 4400 3700
-F 0 "R?" H 4550 3750 50  0000 C CNN
+F 0 "R74" H 4550 3750 50  0000 C CNN
 F 1 "1k" H 4550 3650 50  0000 C CNN
 F 2 "IPC7351-Nominal:RESC1005X40" H 4400 3700 50  0001 C CNN
@@
 Connection ~ 4400 3900
 $Comp
-L GND #PWR?
+L GND #PWR176
 U 1 1 54F386CF
 P 4400 3550
-F 0 "#PWR?" H 4400 3550 30  0001 C CNN
+F 0 "#PWR176" H 4400 3550 30  0001 C CNN
 F 1 "GND" H 4400 3480 30  0001 C CNN
 F 2 "" H 4400 3550 60  0000 C CNN
@@
 	4400 3550 4400 3600
 $Comp
-L R-0402 R?
+L R-0402 R78
 U 1 1 54F3871E
 P 5400 3400
-F 0 "R?" V 5200 3400 50  0000 C CNN
+F 0 "R78" V 5200 3400 50  0000 C CNN
 F 1 "100" V 5300 3400 50  0000 C CNN
 F 2 "IPC7351-Nominal:RESC1005X40" H 5400 3400 50  0001 C CNN
@@
 Connection ~ 4900 3400
 $Comp
-L R-0402 R?
+L R-0402 R77
 U 1 1 54F38849
 P 5400 2100
-F 0 "R?" V 5200 2100 50  0000 C CNN
+F 0 "R77" V 5200 2100 50  0000 C CNN
 F 1 "100" V 5300 2100 50  0000 C CNN
 F 2 "IPC7351-Nominal:RESC1005X40" H 5400 2100 50  0001 C CNN
@@
 	5500 3400 6900 3400
 $Comp
-L R-0402 R?
+L R-0402 R76
 U 1 1 54F38964
 P 5100 2400
-F 0 "R?" H 5250 2450 50  0000 C CNN
+F 0 "R76" H 5250 2450 50  0000 C CNN
 F 1 "100" H 5250 2350 50  0000 C CNN
 F 2 "IPC7351-Nominal:RESC1005X40" H 5100 2400 50  0001 C CNN
@@
 Connection ~ 5100 2100
 $Comp
-L GND #PWR?
+L GND #PWR178
 U 1 1 54F38A9B
 P 5100 2550
-F 0 "#PWR?" H 5100 2550 30  0001 C CNN
+F 0 "#PWR178" H 5100 2550 30  0001 C CNN
 F 1 "GND" H 5100 2480 30  0001 C CNN
 F 2 "" H 5100 2550 60  0000 C CNN
@@
 Connection ~ 5700 3400
 $Comp
-L C-0603 C?
+L C-0603 C74
 U 1 1 54F390B6
 P 6700 3600
-F 0 "C?" H 6900 3650 50  0000 C CNN
+F 0 "C74" H 6900 3650 50  0000 C CNN
 F 1 "22p" H 6900 3550 50  0000 C CNN
 F 2 "IPC7351-Nominal:CAPC1608X55" H 6700 3600 50  0001 C CNN
@@
 $EndComp
 $Comp
-L GND #PWR?
+L GND #PWR179
 U 1 1 54F391AB
 P 6700 3750
-F 0 "#PWR?" H 6700 3750 30  0001 C CNN
+F 0 "#PWR179" H 6700 3750 30  0001 C CNN
 F 1 "GND" H 6700 3680 30  0001 C CNN
 F 2 "" H 6700 3750 60  0000 C CNN
@@
 	6700 3750 6700 3700
 $Comp
-L L-0402 L?
+L L-0402 L4
 U 1 1 54F39511
 P 7000 3400
-F 0 "L?" V 6800 3400 50  0000 C CNN
+F 0 "L4" V 6800 3400 50  0000 C CNN
 F 1 "39n" V 6900 3400 50  0000 C CNN
 F 2 "IPC7351-Nominal:INDC1005X60" H 7000 3400 50  0001 C CNN
@@
 Connection ~ 6700 3400
 $Comp
-L L-0402 L?
+L L-0402 L5
 U 1 1 54F39A44
 P 7600 3400
-F 0 "L?" V 7400 3400 50  0000 C CNN
+F 0 "L5" V 7400 3400 50  0000 C CNN
 F 1 "39n" V 7500 3400 50  0000 C CNN
 F 2 "IPC7351-Nominal:INDC1005X60" H 7600 3400 50  0001 C CNN
@@
 $EndComp
 $Comp
-L C-0603 C?
+L C-0603 C75
 U 1 1 54F39A8A
 P 7300 3600
-F 0 "C?" H 7500 3650 50  0000 C CNN
+F 0 "C75" H 7500 3650 50  0000 C CNN
 F 1 "33p" H 7500 3550 50  0000 C CNN
 F 2 "IPC7351-Nominal:CAPC1608X55" H 7300 3600 50  0001 C CNN
@@
 Connection ~ 7300 3400
 $Comp
-L GND #PWR?
+L GND #PWR180
 U 1 1 54F39BB6
 P 7300 3750
-F 0 "#PWR?" H 7300 3750 30  0001 C CNN
+F 0 "#PWR180" H 7300 3750 30  0001 C CNN
 F 1 "GND" H 7300 3680 30  0001 C CNN
 F 2 "" H 7300 3750 60  0000 C CNN
@@
 	7300 3750 7300 3700
 $Comp
-L C-0603 C?
+L C-0603 C76
 U 1 1 54F39C2D
 P 7900 3600
-F 0 "C?" H 8100 3650 50  0000 C CNN
+F 0 "C76" H 8100 3650 50  0000 C CNN
 F 1 "22p" H 8100 3550 50  0000 C CNN
 F 2 "IPC7351-Nominal:CAPC1608X55" H 7900 3600 50  0001 C CNN
@@
 	7900 3400 7900 3500
 $Comp
-L GND #PWR?
+L GND #PWR181
 U 1 1 54F39CB8
 P 7900 3750
-F 0 "#PWR?" H 7900 3750 30  0001 C CNN
+F 0 "#PWR181" H 7900 3750 30  0001 C CNN
 F 1 "GND" H 7900 3680 30  0001 C CNN
 F 2 "" H 7900 3750 60  0000 C CNN

Commit message: Finish USB subcircuit
Connections:
- net +5: now reaches Q11.3
Changed lines of the file:
@@
 $Descr A4 11693 8268
 encoding utf-8
-Sheet 11 14
+Sheet 10 13
 Title "Input Buffer and Filter"
 Date "2015-02-28"
@@
 OUT
 Connection ~ 7900 3400
+$Comp
+L +5 #PWR?
+U 1 1 54F9478F
+P 4900 2650
+F 0 "#PWR?" H 4900 2700 30  0001 C CNN
+F 1 "+5" H 4900 2750 50  0000 C CNN
+F 2 "" H 4900 2650 60  0000 C CNN
+F 3 "" H 4900 2650 60  0000 C CNN
+	1    4900 2650
+	1    0    0    -1
+$EndComp
+Wire Wire Line
+	4900 2650 4900 2700
 $EndSCHEMATC
