File: proj/Protection.sch (KiCad schematic (older format))
At the start: 18 parts

Commit message: Add power input circuit
Parts:
- gave numbers to parts that had none: 18
Changed lines of the file:
@@
 $Descr USLegal 14000 8500
 encoding utf-8
-Sheet 9 12
+Sheet 9 13
 Title "Input Protection"
 Date "2015-02-28"
@@
 	2400 2300 3400 2300
 $Comp
-L R-0402 R?
+L R-0402 R54
 U 1 1 54F30EB5
 P 2900 2600
-F 0 "R?" H 3050 2650 50  0000 C CNN
+F 0 "R54" H 3050 2650 50  0000 C CNN
 F 1 "1k6" H 3050 2550 50  0000 C CNN
 F 2 "IPC7351-Nominal:RESC1005X40" H 2900 2600 50  0001 C CNN
@@
 $EndComp
 $Comp
-L R-0402 R?
+L R-0402 R55
 U 1 1 54F30F49
 P 3200 2600
-F 0 "R?" H 3350 2650 50  0000 C CNN
+F 0 "R55" H 3350 2650 50  0000 C CNN
 F 1 "1k6" H 3350 2550 50  0000 C CNN
 F 2 "IPC7351-Nominal:RESC1005X40" H 3200 2600 50  0001 C CNN
@@
 Connection ~ 2900 2300
 $Comp
-L GND #PWR?
+L GND #PWR153
 U 1 1 54F30F78
 P 2900 2800
-F 0 "#PWR?" H 2900 2800 30  0001 C CNN
+F 0 "#PWR153" H 2900 2800 30  0001 C CNN
 F 1 "GND" H 2900 2730 30  0001 C CNN
 F 2 "" H 2900 2800 60  0000 C CNN
@@
 	2900 2800 2900 2700
 $Comp
-L GND #PWR?
+L GND #PWR155
 U 1 1 54F30F98
 P 3200 2800
-F 0 "#PWR?" H 3200 2800 30  0001 C CNN
+F 0 "#PWR155" H 3200 2800 30  0001 C CNN
 F 1 "GND" H 3200 2730 30  0001 C CNN
 F 2 "" H 3200 2800 60  0000 C CNN
@@
 Connection ~ 3200 2300
 $Comp
-L R-0402 R?
+L R-0402 R57
 U 1 1 54F312FC
 P 3500 2300
-F 0 "R?" V 3300 2300 50  0000 C CNN
+F 0 "R57" V 3300 2300 50  0000 C CNN
 F 1 "3R3" V 3400 2300 50  0000 C CNN
 F 2 "IPC7351-Nominal:RESC1005X40" H 3500 2300 50  0001 C CNN
@@
 $EndComp
 $Comp
-L ESD9L DZ?
+L ESD9L DZ1
 U 1 1 54F315E0
 P 3750 3500
-F 0 "DZ?" H 3950 3450 50  0000 C CNN
+F 0 "DZ1" H 3950 3450 50  0000 C CNN
 F 1 "ESD9L5.0ST5G" H 4150 3550 50  0000 C CNN
 F 2 "smd-semi:SOD-923" H 3750 3500 50  0001 C CNN
@@
 $EndComp
 $Comp
-L ESD9L DZ?
+L ESD9L DZ3
 U 1 1 54F316A8
 P 4550 3500
-F 0 "DZ?" H 4350 3550 50  0000 C CNN
+F 0 "DZ3" H 4350 3550 50  0000 C CNN
 F 1 "ESD9L5.0ST5G" H 4950 3550 50  0001 C CNN
 F 2 "smd-semi:SOD-923" H 4550 3500 50  0001 C CNN
@@
 $EndComp
 $Comp
-L BZX84 DZ?
+L BZX84 DZ2
 U 1 1 54F319D0
 P 3750 3900
-F 0 "DZ?" H 3950 3950 50  0000 C CNN
+F 0 "DZ2" H 3950 3950 50  0000 C CNN
 F 1 "BZX84C2V7" H 4150 3850 50  0000 C CNN
 F 2 "smd-semi:SOT-23" H 3750 3900 50  0001 C CNN
@@
 $EndComp
 $Comp
-L BZX84 DZ?
+L BZX84 DZ4
 U 1 1 54F321AA
 P 4550 3900
-F 0 "DZ?" H 4350 3850 50  0000 C CNN
+F 0 "DZ4" H 4350 3850 50  0000 C CNN
 F 1 "BZX84C2V7" H 4950 3850 50  0001 C CNN
 F 2 "smd-semi:SOT-23" H 4550 3900 50  0001 C CNN
@@
 	4550 4100 4550 4000
 $Comp
-L GND #PWR?
+L GND #PWR156
 U 1 1 54F327AC
 P 4150 4150
-F 0 "#PWR?" H 4150 4150 30  0001 C CNN
+F 0 "#PWR156" H 4150 4150 30  0001 C CNN
 F 1 "GND" H 4150 4080 30  0001 C CNN
 F 2 "" H 4150 4150 60  0000 C CNN
@@
 Connection ~ 4150 4100
 $Comp
-L R-0402 R?
+L R-0402 R56
 U 1 1 54F327E4
 P 3400 3700
-F 0 "R?" V 3200 3700 50  0000 C CNN
+F 0 "R56" V 3200 3700 50  0000 C CNN
 F 1 "1k" V 3300 3700 50  0000 C CNN
 F 2 "IPC7351-Nominal:RESC1005X40" H 3400 3700 50  0001 C CNN
@@
 Connection ~ 3750 3700
 $Comp
-L +5 #PWR?
+L +5 #PWR154
 U 1 1 54F328CE
 P 3100 3650
-F 0 "#PWR?" H 3100 3700 30  0001 C CNN
+F 0 "#PWR154" H 3100 3700 30  0001 C CNN
 F 1 "+5" H 3100 3750 50  0000 C CNN
 F 2 "" H 3100 3650 60  0000 C CNN
@@
 	3100 3700 3300 3700
 $Comp
-L R-0402 R?
+L R-0402 R58
 U 1 1 54F3293C
 P 4900 3700
-F 0 "R?" V 4700 3700 50  0000 C CNN
+F 0 "R58" V 4700 3700 50  0000 C CNN
 F 1 "1k" V 4800 3700 50  0000 C CNN
 F 2 "IPC7351-Nominal:RESC1005X40" H 4900 3700 50  0001 C CNN
@@
 Connection ~ 4550 3700
 $Comp
-L -5 #PWR?
+L -5 #PWR157
 U 1 1 54F329A1
 P 5200 3800
-F 0 "#PWR?" H 5200 3750 30  0001 C CNN
+F 0 "#PWR157" H 5200 3750 30  0001 C CNN
 F 1 "-5" H 5200 3700 50  0000 C CNN
 F 2 "" H 5200 3800 60  0000 C CNN
@@
 	6400 2300 7400 2300
 $Comp
-L R-0402 R?
+L R-0402 R59
 U 1 1 54F32BFC
 P 6900 2600
-F 0 "R?" H 7050 2650 50  0000 C CNN
+F 0 "R59" H 7050 2650 50  0000 C CNN
 F 1 "1k6" H 7050 2550 50  0000 C CNN
 F 2 "IPC7351-Nominal:RESC1005X40" H 6900 2600 50  0001 C CNN
@@
 $EndComp
 $Comp
-L R-0402 R?
+L R-0402 R60
 U 1 1 54F32C04
 P 7200 2600
-F 0 "R?" H 7350 2650 50  0000 C CNN
+F 0 "R60" H 7350 2650 50  0000 C CNN
 F 1 "1k6" H 7350 2550 50  0000 C CNN
 F 2 "IPC7351-Nominal:RESC1005X40" H 7200 2600 50  0001 C CNN
@@
 Connection ~ 6900 2300
 $Comp
-L GND #PWR?
+L GND #PWR158
 U 1 1 54F32C0D
 P 6900 2800
-F 0 "#PWR?" H 6900 2800 30  0001 C CNN
+F 0 "#PWR158" H 6900 2800 30  0001 C CNN
 F 1 "GND" H 6900 2730 30  0001 C CNN
 F 2 "" H 6900 2800 60  0000 C CNN
@@
 	6900 2800 6900 2700
 $Comp
-L GND #PWR?
+L GND #PWR160
 U 1 1 54F32C14
 P 7200 2800
-F 0 "#PWR?" H 7200 2800 30  0001 C CNN
+F 0 "#PWR160" H 7200 2800 30  0001 C CNN
 F 1 "GND" H 7200 2730 30  0001 C CNN
 F 2 "" H 7200 2800 60  0000 C CNN
@@
 Connection ~ 7200 2300
 $Comp
-L R-0402 R?
+L R-0402 R62
 U 1 1 54F32C1E
 P 7500 2300
-F 0 "R?" V 7300 2300 50  0000 C CNN
+F 0 "R62" V 7300 2300 50  0000 C CNN
 F 1 "3R3" V 7400 2300 50  0000 C CNN
 F 2 "IPC7351-Nominal:RESC1005X40" H 7500 2300 50  0001 C CNN
@@
 $EndComp
 $Comp
-L ESD9L DZ?
+L ESD9L DZ5
 U 1 1 54F32C26
 P 7750 3500
-F 0 "DZ?" H 7950 3450 50  0000 C CNN
+F 0 "DZ5" H 7950 3450 50  0000 C CNN
 F 1 "ESD9L5.0ST5G" H 8150 3550 50  0000 C CNN
 F 2 "smd-semi:SOD-923" H 7750 3500 50  0001 C CNN
@@
 $EndComp
 $Comp
-L ESD9L DZ?
+L ESD9L DZ7
 U 1 1 54F32C2F
 P 8550 3500
-F 0 "DZ?" H 8350 3550 50  0000 C CNN
+F 0 "DZ7" H 8350 3550 50  0000 C CNN
 F 1 "ESD9L5.0ST5G" H 8950 3550 50  0001 C CNN
 F 2 "smd-semi:SOD-923" H 8550 3500 50  0001 C CNN
@@
 $EndComp
 $Comp
-L BZX84 DZ?
+L BZX84 DZ6
 U 1 1 54F32C38
 P 7750 3900
-F 0 "DZ?" H 7950 3950 50  0000 C CNN
+F 0 "DZ6" H 7950 3950 50  0000 C CNN
 F 1 "BZX84C2V7" H 8150 3850 50  0000 C CNN
 F 2 "smd-semi:SOT-23" H 7750 3900 50  0001 C CNN
@@
 $EndComp
 $Comp
-L BZX84 DZ?
+L BZX84 DZ8
 U 1 1 54F32C41
 P 8550 3900
-F 0 "DZ?" H 8350 3850 50  0000 C CNN
+F 0 "DZ8" H 8350 3850 50  0000 C CNN
 F 1 "BZX84C2V7" H 8950 3850 50  0001 C CNN
 F 2 "smd-semi:SOT-23" H 8550 3900 50  0001 C CNN
@@
 	8550 4100 8550 4000
 $Comp
-L GND #PWR?
+L GND #PWR161
 U 1 1 54F32C4C
 P 8150 4150
-F 0 "#PWR?" H 8150 4150 30  0001 C CNN
+F 0 "#PWR161" H 8150 4150 30  0001 C CNN
 F 1 "GND" H 8150 4080 30  0001 C CNN
 F 2 "" H 8150 4150 60  0000 C CNN
@@
 Connection ~ 8150 4100
 $Comp
-L R-0402 R?
+L R-0402 R61
 U 1 1 54F32C56
 P 7400 3700
-F 0 "R?" V 7200 3700 50  0000 C CNN
+F 0 "R61" V 7200 3700 50  0000 C CNN
 F 1 "1k" V 7300 3700 50  0000 C CNN
 F 2 "IPC7351-Nominal:RESC1005X40" H 7400 3700 50  0001 C CNN
@@
 Connection ~ 7750 3700
 $Comp
-L +5 #PWR?
+L +5 #PWR159
 U 1 1 54F32C5E
 P 7100 3650
-F 0 "#PWR?" H 7100 3700 30  0001 C CNN
+F 0 "#PWR159" H 7100 3700 30  0001 C CNN
 F 1 "+5" H 7100 3750 50  0000 C CNN
 F 2 "" H 7100 3650 60  0000 C CNN
@@
 	7100 3700 7300 3700
 $Comp
-L R-0402 R?
+L R-0402 R63
 U 1 1 54F32C68
 P 8900 3700
-F 0 "R?" V 8700 3700 50  0000 C CNN
+F 0 "R63" V 8700 3700 50  0000 C CNN
 F 1 "1k" V 8800 3700 50  0000 C CNN
 F 2 "IPC7351-Nominal:RESC1005X40" H 8900 3700 50  0001 C CNN
@@
 Connection ~ 8550 3700
 $Comp
-L -5 #PWR?
+L -5 #PWR162
 U 1 1 54F32C70
 P 9200 3800
-F 0 "#PWR?" H 9200 3750 30  0001 C CNN
+F 0 "#PWR162" H 9200 3750 30  0001 C CNN
 F 1 "-5" H 9200 3700 50  0000 C CNN
 F 2 "" H 9200 3800 60  0000 C CNN
