File: proj/Switching.sch (KiCad schematic (older format))
At the start: 13 parts

Commit message: Add power input circuit
Parts:
- gave numbers to parts that had none: 13
Changed lines of the file:
@@
 $Descr USLegal 14000 8500
 encoding utf-8
-Sheet 10 12
+Sheet 10 13
 Title "Input Switching"
 Date "2015-02-28"
@@
 $EndDescr
 $Comp
-L MASWSS0162 U?
+L MASWSS0162 U9
 U 1 1 54F34173
 P 6600 2500
-F 0 "U?" H 6250 2150 50  0000 C CNN
+F 0 "U9" H 6250 2150 50  0000 C CNN
 F 1 "MASWSS0162" H 6750 2150 50  0000 C CNN
 F 2 "IPC7351-Nominal:SOIC127P600X175-8" H 6600 2500 50  0001 C CNN
@@
 $EndComp
 $Comp
-L MASWSS0162 U?
+L MASWSS0162 U10
 U 1 1 54F3428A
 P 6600 3300
-F 0 "U?" H 6250 2950 50  0000 C CNN
+F 0 "U10" H 6250 2950 50  0000 C CNN
 F 1 "MASWSS0162" H 6750 2950 50  0000 C CNN
 F 2 "IPC7351-Nominal:SOIC127P600X175-8" H 6600 3300 50  0001 C CNN
@@
 Layout: These stubs must be /very/ short!
 $Comp
-L C-0402 C?
+L C-0402 C71
 U 1 1 54F34AF4
 P 5400 4700
-F 0 "C?" H 5600 4750 50  0000 C CNN
+F 0 "C71" H 5600 4750 50  0000 C CNN
 F 1 "1n" H 5600 4650 50  0000 C CNN
 F 2 "IPC7351-Nominal:CAPC1005X55" H 5400 4700 50  0001 C CNN
@@
 $EndComp
 $Comp
-L C-0402 C?
+L C-0402 C72
 U 1 1 54F34B15
 P 5600 4700
-F 0 "C?" H 5800 4750 50  0000 C CNN
+F 0 "C72" H 5800 4750 50  0000 C CNN
 F 1 "1n" H 5800 4650 50  0000 C CNN
 F 2 "IPC7351-Nominal:CAPC1005X55" H 5600 4700 50  0001 C CNN
@@
 $EndComp
 $Comp
-L R-0402 R?
+L R-0402 R66
 U 1 1 54F34BE3
 P 6100 4500
-F 0 "R?" V 5850 4500 50  0000 C CNN
+F 0 "R66" V 5850 4500 50  0000 C CNN
 F 1 "220" V 5950 4500 50  0000 C CNN
 F 2 "IPC7351-Nominal:RESC1005X40" H 6100 4500 50  0001 C CNN
@@
 $EndComp
 $Comp
-L R-0402 R?
+L R-0402 R67
 U 1 1 54F34D1E
 P 6350 4400
-F 0 "R?" V 6150 4400 50  0000 C CNN
+F 0 "R67" V 6150 4400 50  0000 C CNN
 F 1 "220" V 6250 4400 50  0000 C CNN
 F 2 "IPC7351-Nominal:RESC1005X40" H 6350 4400 50  0001 C CNN
@@
 $EndComp
 $Comp
-L R-0402 R?
+L R-0402 R68
 U 1 1 54F35056
 P 6700 4200
-F 0 "R?" H 6850 4250 50  0000 C CNN
+F 0 "R68" H 6850 4250 50  0000 C CNN
 F 1 "10k" H 6850 4150 50  0000 C CNN
 F 2 "IPC7351-Nominal:RESC1005X40" H 6700 4200 50  0001 C CNN
@@
 $EndComp
 $Comp
-L GND #PWR?
+L GND #PWR167
 U 1 1 54F35197
 P 6700 4000
-F 0 "#PWR?" H 6700 4000 30  0001 C CNN
+F 0 "#PWR167" H 6700 4000 30  0001 C CNN
 F 1 "GND" H 6700 3930 30  0001 C CNN
 F 2 "" H 6700 4000 60  0000 C CNN
@@
 $EndComp
 $Comp
-L R-0402 R?
+L R-0402 R69
 U 1 1 54F351E5
 P 7100 4200
-F 0 "R?" H 7250 4250 50  0000 C CNN
+F 0 "R69" H 7250 4250 50  0000 C CNN
 F 1 "10k" H 7250 4150 50  0000 C CNN
 F 2 "IPC7351-Nominal:RESC1005X40" H 7100 4200 50  0001 C CNN
@@
 $EndComp
 $Comp
-L GND #PWR?
+L GND #PWR169
 U 1 1 54F3526C
 P 7100 4000
-F 0 "#PWR?" H 7100 4000 30  0001 C CNN
+F 0 "#PWR169" H 7100 4000 30  0001 C CNN
 F 1 "GND" H 7100 3930 30  0001 C CNN
 F 2 "" H 7100 4000 60  0000 C CNN
@@
 $EndComp
 $Comp
-L GND #PWR?
+L GND #PWR163
 U 1 1 54F3552B
 P 5400 4850
-F 0 "#PWR?" H 5400 4850 30  0001 C CNN
+F 0 "#PWR163" H 5400 4850 30  0001 C CNN
 F 1 "GND" H 5400 4780 30  0001 C CNN
 F 2 "" H 5400 4850 60  0000 C CNN
@@
 $EndComp
 $Comp
-L GND #PWR?
+L GND #PWR164
 U 1 1 54F3557E
 P 5600 4850
-F 0 "#PWR?" H 5600 4850 30  0001 C CNN
+F 0 "#PWR164" H 5600 4850 30  0001 C CNN
 F 1 "GND" H 5600 4780 30  0001 C CNN
 F 2 "" H 5600 4850 60  0000 C CNN
@@
 IN2
 $Comp
-L 2N7002 Q?
+L 2N7002 Q8
 U 1 1 54F3585D
 P 6650 6100
-F 0 "Q?" H 6800 6200 50  0000 C CNN
+F 0 "Q8" H 6800 6200 50  0000 C CNN
 F 1 "2N7002" H 6900 6050 50  0001 C CNN
 F 2 "smd-semi:SOT-23" H 6650 6100 50  0001 C CNN
@@
 $EndComp
 $Comp
-L 2N7002 Q?
+L 2N7002 Q9
 U 1 1 54F359AE
 P 7050 6100
-F 0 "Q?" H 7300 6150 50  0000 C CNN
+F 0 "Q9" H 7300 6150 50  0000 C CNN
 F 1 "2N7002" H 7300 6050 50  0000 C CNN
 F 2 "smd-semi:SOT-23" H 7050 6100 50  0001 C CNN
@@
 Connection ~ 6700 5850
 $Comp
-L -5 #PWR?
+L -5 #PWR168
 U 1 1 54F35B7E
 P 6700 6250
-F 0 "#PWR?" H 6700 6200 30  0001 C CNN
+F 0 "#PWR168" H 6700 6200 30  0001 C CNN
 F 1 "-5" H 6700 6150 50  0000 C CNN
 F 2 "" H 6700 6250 60  0000 C CNN
@@
 	6700 6250 6700 6200
 $Comp
-L -5 #PWR?
+L -5 #PWR170
 U 1 1 54F35BE5
 P 7100 6250
-F 0 "#PWR?" H 7100 6200 30  0001 C CNN
+F 0 "#PWR170" H 7100 6200 30  0001 C CNN
 F 1 "-5" H 7100 6150 50  0000 C CNN
 F 2 "" H 7100 6250 60  0000 C CNN
@@
 	7100 6250 7100 6200
 $Comp
-L R-0402 R?
+L R-0402 R65
 U 1 1 54F35C3E
 P 6050 6300
-F 0 "R?" H 6200 6350 50  0000 C CNN
+F 0 "R65" H 6200 6350 50  0000 C CNN
 F 1 "10k" H 6200 6250 50  0000 C CNN
 F 2 "IPC7351-Nominal:RESC1005X40" H 6050 6300 50  0001 C CNN
@@
 	6050 6100 6600 6100
 $Comp
-L -5 #PWR?
+L -5 #PWR166
 U 1 1 54F35DDE
 P 6050 6450
-F 0 "#PWR?" H 6050 6400 30  0001 C CNN
+F 0 "#PWR166" H 6050 6400 30  0001 C CNN
 F 1 "-5" H 6050 6350 50  0000 C CNN
 F 2 "" H 6050 6450 60  0000 C CNN
@@
 	6050 6450 6050 6400
 $Comp
-L R-0402 R?
+L R-0402 R64
 U 1 1 54F35E96
 P 6050 5600
-F 0 "R?" H 6200 5650 50  0000 C CNN
+F 0 "R64" H 6200 5650 50  0000 C CNN
 F 1 "1k" H 6200 5550 50  0000 C CNN
 F 2 "IPC7351-Nominal:RESC1005X40" H 6050 5600 50  0001 C CNN
@@
 $EndComp
 $Comp
-L MMBT3906 Q?
+L MMBT3906 Q7
 U 1 1 54F35F38
 P 6000 5900
-F 0 "Q?" H 6300 5950 50  0000 C CNN
+F 0 "Q7" H 6300 5950 50  0000 C CNN
 F 1 "MMBT3906" H 6300 5850 50  0000 C CNN
 F 2 "smd-semi:SOT-23" H 6000 5900 50  0001 C CNN
@@
 $EndComp
 $Comp
-L GND #PWR?
+L GND #PWR165
 U 1 1 54F35FD4
 P 5800 5900
-F 0 "#PWR?" H 5800 5900 30  0001 C CNN
+F 0 "#PWR165" H 5800 5900 30  0001 C CNN
 F 1 "GND" H 5800 5830 30  0001 C CNN
 F 2 "" H 5800 5900 60  0000 C CNN
@@
 CTRL
 $Comp
-L GND #PWR?
+L GND #PWR171
 U 1 1 54F36542
 P 7300 3600
-F 0 "#PWR?" H 7300 3600 30  0001 C CNN
+F 0 "#PWR171" H 7300 3600 30  0001 C CNN
 F 1 "GND" H 7300 3530 30  0001 C CNN
 F 2 "" H 7300 3600 60  0000 C CNN
