File: proj/DCDC.sch (KiCad schematic (older format))
At the start: 55 parts, among them Q13 MMBT3904, Q15 MMBT3904, Q16 MMBT3904, Q17 PZT2907A, Q18 PZT2907A, Q19 MMBT3904, U14 L78M05CDT, U15 MC79M05CDT, U16 AZ1117CH-1.8TRG1, U17 MCP1700T-vv02E/TT

Commit message: Clean up resistor BOM
Parts:
- R82, R92: value 10k -> 4k7; BOM RES SMD 1k 5% [0402] -> RES SMD 4.7k 5% [0402]
- R83, R84, R93, R94: value 1k -> 1k6; BOM RES SMD 1k 5% [0402] -> RES SMD 1.6k 5% [0402]
- R97, R98: value 2R2 -> 3R3; BOM RES SMD 2.2 5% [0402] -> RES SMD 3.3 5% [0402]
Changed lines of the file:
@@
 AR Path="/54F4F7B6/54F4E4A1" Ref="R83"  Part="1"
 F 0 "R83" H 4800 1150 50  0000 C CNN
-F 1 "1k" H 4800 1050 50  0000 C CNN
+F 1 "1k6" H 4800 1050 50  0000 C CNN
 F 2 "IPC7351-Nominal:RESC1005X40" H 4650 1100 50  0001 C CNN
 F 3 "" H 4650 1150 60  0000 C CNN
 F 4 "Value" H 4650 1100 60  0001 C CNN "Manuf"
-F 5 "RES SMD 1k 5% [0402]" H 5400 1650 60  0001 C CNN "BOM"
+F 5 "RES SMD 1.6k 5% [0402]" H 5400 1650 60  0001 C CNN "BOM"
 	1    4650 1100
 	1    0    0    -1
@@
 AR Path="/54F4F7B6/54F4E693" Ref="R84"  Part="1"
 F 0 "R84" H 4800 1550 50  0000 C CNN
-F 1 "1k" H 4800 1450 50  0000 C CNN
+F 1 "1k6" H 4800 1450 50  0000 C CNN
 F 2 "IPC7351-Nominal:RESC1005X40" H 4650 1500 50  0001 C CNN
 F 3 "" H 4650 1550 60  0000 C CNN
 F 4 "Value" H 4650 1500 60  0001 C CNN "Manuf"
-F 5 "RES SMD 1k 5% [0402]" H 5400 2050 60  0001 C CNN "BOM"
+F 5 "RES SMD 1.6k 5% [0402]" H 5400 2050 60  0001 C CNN "BOM"
 	1    4650 1500
 	1    0    0    -1
@@
 AR Path="/54F4F7B6/54F4F882" Ref="R82"  Part="1"
 F 0 "R82" H 4450 1550 50  0000 C CNN
-F 1 "10k" H 4450 1450 50  0000 C CNN
+F 1 "4k7" H 4450 1450 50  0000 C CNN
 F 2 "IPC7351-Nominal:RESC1005X40" H 4300 1500 50  0001 C CNN
 F 3 "" H 4300 1550 60  0000 C CNN
 F 4 "Value" H 4300 1500 60  0001 C CNN "Manuf"
-F 5 "RES SMD 1k 5% [0402]" H 5050 2050 60  0001 C CNN "BOM"
+F 5 "RES SMD 4.7k 5% [0402]" H 5050 2050 60  0001 C CNN "BOM"
 	1    4300 1500
 	1    0    0    -1
@@
 P 7200 2400
 AR Path="/54F1FAAC/54F4F7B6/54F50066" Ref="#PWR8"  Part="1"
-AR Path="/54F4F7B6/54F50066" Ref="#PWR0208"  Part="1"
-F 0 "#PWR0208" H 7200 2400 30  0001 C CNN
+AR Path="/54F4F7B6/54F50066" Ref="#PWR0206"  Part="1"
+F 0 "#PWR0206" H 7200 2400 30  0001 C CNN
 F 1 "GND" H 7200 2330 30  0001 C CNN
 F 2 "" H 7200 2400 60  0000 C CNN
@@
 AR Path="/54F4F7B6/54F53F7B" Ref="R93"  Part="1"
 F 0 "R93" H 4800 3550 50  0000 C CNN
-F 1 "1k" H 4800 3450 50  0000 C CNN
+F 1 "1k6" H 4800 3450 50  0000 C CNN
 F 2 "IPC7351-Nominal:RESC1005X40" H 4650 3500 50  0001 C CNN
 F 3 "" H 4650 3550 60  0000 C CNN
 F 4 "Value" H 4650 3500 60  0001 C CNN "Manuf"
-F 5 "RES SMD 1k 5% [0402]" H 5400 4050 60  0001 C CNN "BOM"
+F 5 "RES SMD 1.6k 5% [0402]" H 5400 4050 60  0001 C CNN "BOM"
 	1    4650 3500
 	1    0    0    -1
@@
 AR Path="/54F4F7B6/54F53F83" Ref="R94"  Part="1"
 F 0 "R94" H 4800 3950 50  0000 C CNN
-F 1 "1k" H 4800 3850 50  0000 C CNN
+F 1 "1k6" H 4800 3850 50  0000 C CNN
 F 2 "IPC7351-Nominal:RESC1005X40" H 4650 3900 50  0001 C CNN
 F 3 "" H 4650 3950 60  0000 C CNN
 F 4 "Value" H 4650 3900 60  0001 C CNN "Manuf"
-F 5 "RES SMD 1k 5% [0402]" H 5400 4450 60  0001 C CNN "BOM"
+F 5 "RES SMD 1.6k 5% [0402]" H 5400 4450 60  0001 C CNN "BOM"
 	1    4650 3900
 	1    0    0    -1
@@
 AR Path="/54F4F7B6/54F53FE2" Ref="R92"  Part="1"
 F 0 "R92" H 4450 3950 50  0000 C CNN
-F 1 "10k" H 4450 3850 50  0000 C CNN
+F 1 "4k7" H 4450 3850 50  0000 C CNN
 F 2 "IPC7351-Nominal:RESC1005X40" H 4300 3900 50  0001 C CNN
 F 3 "" H 4300 3950 60  0000 C CNN
 F 4 "Value" H 4300 3900 60  0001 C CNN "Manuf"
-F 5 "RES SMD 1k 5% [0402]" H 5050 4450 60  0001 C CNN "BOM"
+F 5 "RES SMD 4.7k 5% [0402]" H 5050 4450 60  0001 C CNN "BOM"
 	1    4300 3900
 	1    0    0    -1
@@
 P 7050 5400
 AR Path="/54F1FAAC/54F4F7B6/54F543B2" Ref="#PWR?"  Part="1"
-AR Path="/54F4F7B6/54F543B2" Ref="#PWR0209"  Part="1"
-F 0 "#PWR0209" H 7050 5400 30  0001 C CNN
+AR Path="/54F4F7B6/54F543B2" Ref="#PWR0207"  Part="1"
+F 0 "#PWR0207" H 7050 5400 30  0001 C CNN
 F 1 "GND" H 7050 5330 30  0001 C CNN
 F 2 "" H 7050 5400 60  0000 C CNN
@@
 P 8900 1400
 AR Path="/54F1FAAC/54F4F7B6/54F64B84" Ref="#PWR?"  Part="1"
-AR Path="/54F4F7B6/54F64B84" Ref="#PWR0210"  Part="1"
-F 0 "#PWR0210" H 8900 1400 30  0001 C CNN
+AR Path="/54F4F7B6/54F64B84" Ref="#PWR0208"  Part="1"
+F 0 "#PWR0208" H 8900 1400 30  0001 C CNN
 F 1 "GND" H 8900 1330 30  0001 C CNN
 F 2 "" H 8900 1400 60  0000 C CNN
@@
 P 8900 2200
 AR Path="/54F1FAAC/54F4F7B6/54F676AE" Ref="#PWR?"  Part="1"
-AR Path="/54F4F7B6/54F676AE" Ref="#PWR0211"  Part="1"
-F 0 "#PWR0211" H 8900 2200 30  0001 C CNN
+AR Path="/54F4F7B6/54F676AE" Ref="#PWR0209"  Part="1"
+F 0 "#PWR0209" H 8900 2200 30  0001 C CNN
 F 1 "GND" H 8900 2130 30  0001 C CNN
 F 2 "" H 8900 2200 60  0000 C CNN
@@
 P 8200 2250
 AR Path="/54F1FAAC/54F4F7B6/54F67A48" Ref="#PWR?"  Part="1"
-AR Path="/54F4F7B6/54F67A48" Ref="#PWR0212"  Part="1"
-F 0 "#PWR0212" H 8200 2250 30  0001 C CNN
+AR Path="/54F4F7B6/54F67A48" Ref="#PWR0210"  Part="1"
+F 0 "#PWR0210" H 8200 2250 30  0001 C CNN
 F 1 "GND" H 8200 2180 30  0001 C CNN
 F 2 "" H 8200 2250 60  0000 C CNN
@@
 P 9400 2250
 AR Path="/54F1FAAC/54F4F7B6/54F687DB" Ref="#PWR?"  Part="1"
-AR Path="/54F4F7B6/54F687DB" Ref="#PWR0213"  Part="1"
-F 0 "#PWR0213" H 9400 2250 30  0001 C CNN
+AR Path="/54F4F7B6/54F687DB" Ref="#PWR0211"  Part="1"
+F 0 "#PWR0211" H 9400 2250 30  0001 C CNN
 F 1 "GND" H 9400 2180 30  0001 C CNN
 F 2 "" H 9400 2250 60  0000 C CNN
@@
 AR Path="/54F4F7B6/54F6951D" Ref="R97"  Part="1"
 F 0 "R97" H 10100 2400 50  0000 C CNN
-F 1 "2R2" H 10100 2300 50  0000 C CNN
+F 1 "3R3" H 10100 2300 50  0000 C CNN
 F 2 "IPC7351-Nominal:RESC1005X40" H 9900 2350 50  0001 C CNN
 F 3 "" H 9900 2400 60  0000 C CNN
 F 4 "Value" H 9900 2350 60  0001 C CNN "Manuf"
-F 5 "RES SMD 2.2 5% [0402]" H 10650 2900 60  0001 C CNN "BOM"
+F 5 "RES SMD 3.3 5% [0402]" H 10650 2900 60  0001 C CNN "BOM"
 	1    9900 2350
 	1    0    0    -1
@@
 P 9900 2500
 AR Path="/54F1FAAC/54F4F7B6/54F6971F" Ref="#PWR?"  Part="1"
-AR Path="/54F4F7B6/54F6971F" Ref="#PWR0214"  Part="1"
-F 0 "#PWR0214" H 9900 2500 30  0001 C CNN
+AR Path="/54F4F7B6/54F6971F" Ref="#PWR0212"  Part="1"
+F 0 "#PWR0212" H 9900 2500 30  0001 C CNN
 F 1 "GND" H 9900 2430 30  0001 C CNN
 F 2 "" H 9900 2500 60  0000 C CNN
@@
 P 8200 3850
 AR Path="/54F1FAAC/54F4F7B6/54F6B841" Ref="#PWR?"  Part="1"
-AR Path="/54F4F7B6/54F6B841" Ref="#PWR0215"  Part="1"
-F 0 "#PWR0215" H 8200 3850 30  0001 C CNN
+AR Path="/54F4F7B6/54F6B841" Ref="#PWR0213"  Part="1"
+F 0 "#PWR0213" H 8200 3850 30  0001 C CNN
 F 1 "GND" H 8200 3780 30  0001 C CNN
 F 2 "" H 8200 3850 60  0000 C CNN
@@
 AR Path="/54F4F7B6/54F6BDB1" Ref="R98"  Part="1"
 F 0 "R98" H 10100 4000 50  0000 C CNN
-F 1 "2R2" H 10100 3900 50  0000 C CNN
+F 1 "3R3" H 10100 3900 50  0000 C CNN
 F 2 "IPC7351-Nominal:RESC1005X40" H 9900 3950 50  0001 C CNN
 F 3 "" H 9900 4000 60  0000 C CNN
 F 4 "Value" H 9900 3950 60  0001 C CNN "Manuf"
-F 5 "RES SMD 2.2 5% [0402]" H 10650 4500 60  0001 C CNN "BOM"
+F 5 "RES SMD 3.3 5% [0402]" H 10650 4500 60  0001 C CNN "BOM"
 	1    9900 3950
 	1    0    0    -1
@@
 P 9900 4150
 AR Path="/54F1FAAC/54F4F7B6/54F6BEED" Ref="#PWR?"  Part="1"
-AR Path="/54F4F7B6/54F6BEED" Ref="#PWR0216"  Part="1"
-F 0 "#PWR0216" H 9900 4150 30  0001 C CNN
+AR Path="/54F4F7B6/54F6BEED" Ref="#PWR0214"  Part="1"
+F 0 "#PWR0214" H 9900 4150 30  0001 C CNN
 F 1 "GND" H 9900 4080 30  0001 C CNN
 F 2 "" H 9900 4150 60  0000 C CNN
@@
 P 9400 3850
 AR Path="/54F1FAAC/54F4F7B6/54F6BFFB" Ref="#PWR?"  Part="1"
-AR Path="/54F4F7B6/54F6BFFB" Ref="#PWR0217"  Part="1"
-F 0 "#PWR0217" H 9400 3850 30  0001 C CNN
+AR Path="/54F4F7B6/54F6BFFB" Ref="#PWR0215"  Part="1"
+F 0 "#PWR0215" H 9400 3850 30  0001 C CNN
 F 1 "GND" H 9400 3780 30  0001 C CNN
 F 2 "" H 9400 3850 60  0000 C CNN
@@
 P 8900 3850
 AR Path="/54F1FAAC/54F4F7B6/54F6C162" Ref="#PWR?"  Part="1"
-AR Path="/54F4F7B6/54F6C162" Ref="#PWR0218"  Part="1"
-F 0 "#PWR0218" H 8900 3850 30  0001 C CNN
+AR Path="/54F4F7B6/54F6C162" Ref="#PWR0216"  Part="1"
+F 0 "#PWR0216" H 8900 3850 30  0001 C CNN
 F 1 "GND" H 8900 3780 30  0001 C CNN
 F 2 "" H 8900 3850 60  0000 C CNN
@@
 P 8200 5450
 AR Path="/54F1FAAC/54F4F7B6/54F708B6" Ref="#PWR?"  Part="1"
-AR Path="/54F4F7B6/54F708B6" Ref="#PWR0219"  Part="1"
-F 0 "#PWR0219" H 8200 5450 30  0001 C CNN
+AR Path="/54F4F7B6/54F708B6" Ref="#PWR0217"  Part="1"
+F 0 "#PWR0217" H 8200 5450 30  0001 C CNN
 F 1 "GND" H 8200 5380 30  0001 C CNN
 F 2 "" H 8200 5450 60  0000 C CNN
@@
 P 8950 5450
 AR Path="/54F1FAAC/54F4F7B6/54F70A31" Ref="#PWR?"  Part="1"
-AR Path="/54F4F7B6/54F70A31" Ref="#PWR0220"  Part="1"
-F 0 "#PWR0220" H 8950 5450 30  0001 C CNN
+AR Path="/54F4F7B6/54F70A31" Ref="#PWR0218"  Part="1"
+F 0 "#PWR0218" H 8950 5450 30  0001 C CNN
 F 1 "GND" H 8950 5380 30  0001 C CNN
 F 2 "" H 8950 5450 60  0000 C CNN
@@
 P 9500 5450
 AR Path="/54F1FAAC/54F4F7B6/54F71350" Ref="#PWR?"  Part="1"
-AR Path="/54F4F7B6/54F71350" Ref="#PWR0221"  Part="1"
-F 0 "#PWR0221" H 9500 5450 30  0001 C CNN
+AR Path="/54F4F7B6/54F71350" Ref="#PWR0219"  Part="1"
+F 0 "#PWR0219" H 9500 5450 30  0001 C CNN
 F 1 "GND" H 9500 5380 30  0001 C CNN
 F 2 "" H 9500 5450 60  0000 C CNN
@@
 P 8200 6700
 AR Path="/54F1FAAC/54F4F7B6/54F777AE" Ref="#PWR?"  Part="1"
-AR Path="/54F4F7B6/54F777AE" Ref="#PWR0222"  Part="1"
-F 0 "#PWR0222" H 8200 6700 30  0001 C CNN
+AR Path="/54F4F7B6/54F777AE" Ref="#PWR0220"  Part="1"
+F 0 "#PWR0220" H 8200 6700 30  0001 C CNN
 F 1 "GND" H 8200 6630 30  0001 C CNN
 F 2 "" H 8200 6700 60  0000 C CNN
@@
 P 8950 6700
 AR Path="/54F1FAAC/54F4F7B6/54F779B8" Ref="#PWR?"  Part="1"
-AR Path="/54F4F7B6/54F779B8" Ref="#PWR0223"  Part="1"
-F 0 "#PWR0223" H 8950 6700 30  0001 C CNN
+AR Path="/54F4F7B6/54F779B8" Ref="#PWR0221"  Part="1"
+F 0 "#PWR0221" H 8950 6700 30  0001 C CNN
 F 1 "GND" H 8950 6630 30  0001 C CNN
 F 2 "" H 8950 6700 60  0000 C CNN
@@
 P 9500 6700
 AR Path="/54F1FAAC/54F4F7B6/54F78198" Ref="#PWR?"  Part="1"
-AR Path="/54F4F7B6/54F78198" Ref="#PWR0224"  Part="1"
-F 0 "#PWR0224" H 9500 6700 30  0001 C CNN
+AR Path="/54F4F7B6/54F78198" Ref="#PWR0222"  Part="1"
+F 0 "#PWR0222" H 9500 6700 30  0001 C CNN
 F 1 "GND" H 9500 6630 30  0001 C CNN
 F 2 "" H 9500 6700 60  0000 C CNN
@@
 $EndComp
 $Comp
-L GND #PWR0225
+L GND #PWR0223
 U 1 1 54F66084
 P 3800 2150
-F 0 "#PWR0225" H 3800 2150 30  0001 C CNN
+F 0 "#PWR0223" H 3800 2150 30  0001 C CNN
 F 1 "GND" H 3800 2080 30  0001 C CNN
 F 2 "" H 3800 2150 60  0000 C CNN

Commit message: Tweak layout
Parts:
- removed C108, C109: 100n, IPC7351-Nominal:CAPC2012X70, symbol C-0805
- C100, C101, C96, C97: BOM DIST DIGIKEY 493-3919-1-ND -> DIST DIGIKEY P16468CT-ND; Manuf Nichicon -> Panasonic; PN UCL1C101MCL1GS -> 16SVPC100M
- R82, R92: value 4k7 -> 3k3; BOM RES SMD 4.7k 5% [0402] -> RES SMD 3.3k 5% [0402]
- R84, R94: value 1k6 -> 750; BOM RES SMD 1.6k 5% [0402] -> RES SMD 750 5% [0402]
Other:
- moved on the sheet: C112, C113, R97, R98
