File: wcp52/Buffer_Filter.sch (KiCad schematic (older format))
At the start: 18 parts, among them Q10 BFR540, Q8 MMBT3904, Q9 BFR540

Commit message: Prepare to fab
Changed lines of the file:
@@
 $EndComp
 Wire Wire Line
-	3000 2600 3700 2600
-Wire Wire Line
-	3700 2600 4000 2600
-Wire Wire Line
-	4000 2600 4300 2600
-Wire Wire Line
-	4300 2600 4600 2600
-Wire Wire Line
-	4600 2600 4950 2600
+	3000 2600 4950 2600
 Wire Wire Line
 	4600 2600 4600 2700
@@
 $EndComp
 Wire Wire Line
-	5100 2700 5100 3200
-Wire Wire Line
-	5100 3200 5100 3600
+	5100 2700 5100 3600
 $Comp
 L MMBT3904 Q8
@@
 $EndComp
 Wire Wire Line
-	5100 3800 5100 5300
-Wire Wire Line
-	5100 5300 5100 5400
+	5100 3800 5100 5400
 Wire Wire Line
 	5100 5300 5000 5300
@@
 	4550 5050 4850 5050
 Wire Wire Line
-	4850 3700 4850 5050
-Wire Wire Line
-	4850 5050 4850 5200
+	4850 3700 4850 5200
 Connection ~ 5100 5300
 $Comp
@@
 $EndComp
 Wire Wire Line
-	5100 5600 5100 5700
-Wire Wire Line
-	5100 5700 5100 5800
+	5100 5600 5100 5800
 Wire Wire Line
 	4850 5700 5100 5700
@@
 PHASEREF
 Wire Wire Line
-	2100 1900 5300 1900
-Wire Wire Line
-	5300 1900 5500 1900
+	2100 1900 5500 1900
 Text HLabel 3000 2600 0    50   Input ~ 0
 IN
@@
 	5900 1900 5900 3200
 Wire Wire Line
-	5700 3200 5900 3200
-Wire Wire Line
-	5900 3200 6900 3200
-Wire Wire Line
-	6900 3200 7100 3200
+	5700 3200 7100 3200
 Wire Wire Line
 	5300 2100 5300 1900
@@
 	7500 3300 7500 3200
 Wire Wire Line
-	7300 3200 7500 3200
-Wire Wire Line
-	7500 3200 7700 3200
+	7300 3200 7700 3200
 Connection ~ 7500 3200
 $Comp
@@
 $EndComp
 Wire Wire Line
-	7900 3200 8100 3200
-Wire Wire Line
-	8100 3200 8800 3200
+	7900 3200 8800 3200
 Wire Wire Line
 	8100 3200 8100 3300
@@
 $EndComp
 Wire Wire Line
-	4550 3700 4850 3700
-Wire Wire Line
-	4850 3700 4950 3700
+	4550 3700 4950 3700
 Wire Wire Line
 	4550 3850 4550 3700
 Connection ~ 4850 3700
 $Comp
-L -5 #PWR?
+L -5 #PWR0198
 U 1 1 55058533
 P 4550 4100
-F 0 "#PWR?" H 4550 4050 30  0001 C CNN
+F 0 "#PWR0198" H 4550 4050 30  0001 C CNN
 F 1 "-5" H 4550 4000 50  0000 C CNN
 F 2 "" H 4550 4100 60  0000 C CNN

Commit message: BOM line fixes
Parts:
- C59, Q8, R69, R70, R71, R72, R73, R74, R75, R76, R77: Manuf Value -> (none)
- C60, C62: Description (none) -> CAP MLCC 22pF C0G [0402]
- C61: Description (none) -> CAP MLCC 33pF C0G [0402]
- L4, L5: Description (none) -> IND CHIP 39nH
Changed lines of the file:
@@
 EESchema Schematic File Version 2
+LIBS:Altera
+LIBS:AnalogDevices
+LIBS:Atmel
+LIBS:conn-2mm
+LIBS:conn-100mil
+LIBS:conn-cui
+LIBS:conn-fci
+LIBS:conn-linx
+LIBS:conn-molex
+LIBS:conn-tagconnect
+LIBS:conn-test
+LIBS:DiodesInc
+LIBS:display
+LIBS:_electromech
+LIBS:Fairchild
+LIBS:FTDI
+LIBS:Intersil
+LIBS:Lattice
+LIBS:_linear
+LIBS:LinearTech
+LIBS:Littelfuse
+LIBS:logic-4000
+LIBS:logic-7400
+LIBS:MACOM
+LIBS:maxim
+LIBS:mechanical
+LIBS:Microchip
+LIBS:Micron
+LIBS:NXP
+LIBS:onsemi
+LIBS:passive
+LIBS:pasv-BiTech
+LIBS:pasv-Bourns
+LIBS:pasv-cap
+LIBS:pasv-ind
+LIBS:pasv-res
+LIBS:pcb
+LIBS:power
+LIBS:_semi
+LIBS:semi-diode-1N
+LIBS:semi-diode-BA
+LIBS:semi-diode-MCC
+LIBS:semi-diode-MMB
+LIBS:semi-diode-NXP
+LIBS:semi-diode-OnSemi
+LIBS:semi-diode-Vishay
+LIBS:semi-opto-misc
+LIBS:semi-thyristor-2N
+LIBS:semi-trans-2N
+LIBS:semi-trans-AO
+LIBS:semi-trans-BC
+LIBS:semi-trans-DiodesInc
+LIBS:semi-trans-Fairchild
+LIBS:semi-trans-Infineon
+LIBS:semi-trans-IntRect
+LIBS:semi-trans-IXYS
+LIBS:semi-trans-misc
+LIBS:semi-trans-MMB
+LIBS:semi-trans-MPS
+LIBS:semi-trans-NXP
+LIBS:semi-trans-PZT
+LIBS:semi-trans-TI
+LIBS:semi-trans-TIP
+LIBS:semi-trans-Toshiba
+LIBS:silabs
+LIBS:skyworks
+LIBS:ST
+LIBS:st_ic
+LIBS:st_semi
+LIBS:supertex
+LIBS:symbol
+LIBS:TexasInstruments
+LIBS:vishay_semi
+LIBS:Xilinx
+LIBS:pasv-xtal
+LIBS:conn-te
 LIBS:wcp52-cache
 EELAYER 25 0
@@
 F 2 "smd-semi:SOT-23" H 4900 5300 50  0001 C CNN
 F 3 "" H 4900 5300 60  0000 C CNN
-F 4 "Value" H 4900 5300 60  0001 C CNN "Manuf"
+F 4 "" H 4900 5300 60  0001 C CNN "Manuf"
 F 5 "SEMI GENERIC MMBT3904" H 5700 5850 60  0001 C CNN "BOM"
 F 6 "Q10" H 4900 5300 50  0001 C CNN "OldReference"
@@
 F 5 "TDK" H 6900 3400 60  0001 C CNN "Manuf"
 F 6 "DIST DIGIKEY 445-5366-1-ND" H 7700 3950 60  0001 C CNN "BOM"
-F 7 "C74" H 6900 3400 50  0001 C CNN "OldReference"
+F 7 "CAP MLCC 22pF C0G [0402]" H 6900 3400 60  0001 C CNN "Description"
+F 8 "C74" H 6900 3400 50  0001 C CNN "OldReference"
 	1    6900 3400
 	1    0    0    -1
@@
 F 5 "Panasonic" H 7200 3200 60  0001 C CNN "Manuf"
 F 6 "DIST DIGIKEY PCD1917CT-ND" H 7200 3200 60  0001 C CNN "BOM"
-F 7 "L4" H 7200 3200 50  0001 C CNN "OldReference"
+F 7 "IND CHIP 39nH" H 7200 3200 60  0001 C CNN "Description"
+F 8 "L4" H 7200 3200 50  0001 C CNN "OldReference"
 	1    7200 3200
 	0    1    1    0
@@
 F 5 "Panasonic" H 7800 3200 60  0001 C CNN "Manuf"
 F 6 "DIST DIGIKEY PCD1917CT-ND" H 7800 3200 60  0001 C CNN "BOM"
-F 7 "L5" H 7800 3200 50  0001 C CNN "OldReference"
+F 7 "IND CHIP 39nH" H 7800 3200 60  0001 C CNN "Description"
+F 8 "L5" H 7800 3200 50  0001 C CNN "OldReference"
 	1    7800 3200
 	0    1    1    0
@@
 F 5 "TDK" H 7500 3400 60  0001 C CNN "Manuf"
 F 6 "DIST DIGIKEY 445-7027-1-ND" H 8300 3950 60  0001 C CNN "BOM"
-F 7 "C75" H 7500 3400 50  0001 C CNN "OldReference"
+F 7 "CAP MLCC 33pF C0G [0402]" H 7500 3400 60  0001 C CNN "Description"
+F 8 "C75" H 7500 3400 50  0001 C CNN "OldReference"
 	1    7500 3400
 	1    0    0    -1
@@
 F 5 "TDK" H 8100 3400 60  0001 C CNN "Manuf"
 F 6 "DIST DIGIKEY 445-5366-1-ND" H 8900 3950 60  0001 C CNN "BOM"
-F 7 "C76" H 8100 3400 50  0001 C CNN "OldReference"
+F 7 "CAP MLCC 22pF C0G [0402]" H 8100 3400 60  0001 C CNN "Description"
+F 8 "C76" H 8100 3400 50  0001 C CNN "OldReference"
 	1    8100 3400
 	1    0    0    -1
@@
 F 2 "IPC7351-Nominal:CAPC1608X55" H 4550 3950 50  0001 C CNN
 F 3 "" H 4540 3925 60  0000 C CNN
-F 4 "Value" H 4550 3950 60  0001 C CNN "Manuf"
+F 4 "" H 4550 3950 60  0001 C CNN "Manuf"
 F 5 "CAP MLCC 100n ≥X7R 16V 10% [0603]" H 5350 4500 60  0001 C CNN "BOM"
 F 6 "C56" H 4550 3950 50  0001 C CNN "OldReference"
@@
 F 2 "IPC7351-Nominal:RESC1608X50" H 5100 5500 50  0001 C CNN
 F 3 "" H 5100 5550 60  0000 C CNN
-F 4 "Value" H 5100 5500 60  0001 C CNN "Manuf"
+F 4 "" H 5100 5500 60  0001 C CNN "Manuf"
 F 5 "RES SMD 22 5% [0603]" H 5850 6050 60  0001 C CNN "BOM"
 F 6 "R75" H 5100 5500 50  0001 C CNN "OldReference"
@@
 F 2 "IPC7351-Nominal:RESC1608X50" H 4550 4850 50  0001 C CNN
 F 3 "" H 4550 4900 60  0000 C CNN
-F 4 "Value" H 4550 4850 60  0001 C CNN "Manuf"
+F 4 "" H 4550 4850 60  0001 C CNN "Manuf"
 F 5 "RES SMD 1.6k 1% [0603]" H 5300 5400 60  0001 C CNN "BOM"
 F 6 "R74" H 4550 4850 50  0001 C CNN "OldReference"
@@
 F 2 "IPC7351-Nominal:RESC1608X50" H 3700 2800 50  0001 C CNN
 F 3 "" H 3700 2850 60  0000 C CNN
-F 4 "Value" H 3700 2800 60  0001 C CNN "Manuf"
+F 4 "" H 3700 2800 60  0001 C CNN "Manuf"
 F 5 "RES SMD 200 1% [0603]" H 4450 3350 60  0001 C CNN "BOM"
 F 6 "R70" H 3700 2800 50  0001 C CNN "OldReference"
@@
 F 2 "IPC7351-Nominal:RESC1608X50" H 4000 2800 50  0001 C CNN
 F 3 "" H 4000 2850 60  0000 C CNN
-F 4 "Value" H 4000 2800 60  0001 C CNN "Manuf"
+F 4 "" H 4000 2800 60  0001 C CNN "Manuf"
 F 5 "RES SMD 200 1% [0603]" H 4750 3350 60  0001 C CNN "BOM"
 F 6 "R71" H 4000 2800 50  0001 C CNN "OldReference"
@@
 F 2 "IPC7351-Nominal:RESC1608X50" H 4300 2800 50  0001 C CNN
 F 3 "" H 4300 2850 60  0000 C CNN
-F 4 "Value" H 4300 2800 60  0001 C CNN "Manuf"
+F 4 "" H 4300 2800 60  0001 C CNN "Manuf"
 F 5 "RES SMD 200 1% [0603]" H 5050 3350 60  0001 C CNN "BOM"
 F 6 "R72" H 4300 2800 50  0001 C CNN "OldReference"
@@
 F 2 "IPC7351-Nominal:RESC1608X50" H 4600 2800 50  0001 C CNN
 F 3 "" H 4600 2850 60  0000 C CNN
-F 4 "Value" H 4600 2800 60  0001 C CNN "Manuf"
+F 4 "" H 4600 2800 60  0001 C CNN "Manuf"
 F 5 "RES SMD 200 1% [0603]" H 5350 3350 60  0001 C CNN "BOM"
 F 6 "R73" H 4600 2800 50  0001 C CNN "OldReference"
@@
 F 2 "IPC7351-Nominal:RESC1608X50" H 5600 1900 50  0001 C CNN
 F 3 "" H 5600 1950 60  0000 C CNN
-F 4 "Value" H 5600 1900 60  0001 C CNN "Manuf"
+F 4 "" H 5600 1900 60  0001 C CNN "Manuf"
 F 5 "RES SMD 100 1% [0603]" H 6350 2450 60  0001 C CNN "BOM"
 F 6 "R77" H 5600 1900 50  0001 C CNN "OldReference"
@@
 F 2 "IPC7351-Nominal:RESC1608X50" H 5300 2200 50  0001 C CNN
 F 3 "" H 5300 2250 60  0000 C CNN
-F 4 "Value" H 5300 2200 60  0001 C CNN "Manuf"
+F 4 "" H 5300 2200 60  0001 C CNN "Manuf"
 F 5 "RES SMD 100 1% [0603]" H 6050 2750 60  0001 C CNN "BOM"
 F 6 "R76" H 5300 2200 50  0001 C CNN "OldReference"
@@
 F 2 "IPC7351-Nominal:RESC1608X50" H 5600 3200 50  0001 C CNN
 F 3 "" H 5600 3250 60  0000 C CNN
-F 4 "Value" H 5600 3200 60  0001 C CNN "Manuf"
+F 4 "" H 5600 3200 60  0001 C CNN "Manuf"
 F 5 "RES SMD 100 1% [0603]" H 6350 3750 60  0001 C CNN "BOM"
 F 6 "R78" H 5600 3200 50  0001 C CNN "OldReference"
