File: wcp52/DCDCneg9.sch (KiCad schematic (older format))
At the start: 13 parts, among them Q13 MMBT3904, Q14 MMBT2907A, Q15 MMBT3904

Commit message: Reannotate parts. May need to tweak silkscreen
Parts:
- C86: OldReference (none) -> C86
- C87: OldReference (none) -> C87
- C88: OldReference (none) -> C88
- D3: OldReference (none) -> D3
- DZ9: OldReference (none) -> DZ9
- L6: OldReference (none) -> L6
- Q13: OldReference (none) -> Q13
- Q14: OldReference (none) -> Q14
- Q15: OldReference (none) -> Q15
- R82: OldReference (none) -> R82
- R83: OldReference (none) -> R83
- R84: OldReference (none) -> R84
- R85: OldReference (none) -> R85
Changed lines of the file:
@@
 F 2 "IPC-semi-nominal:SOT-23" H 6600 2800 50  0001 C CNN
 F 3 "" H 6600 2800 60  0000 C CNN
+F 4 "Q14" H 6600 2800 50 0001 C CNN "OldReference"
 	1    6600 2800
 	1    0    0    -1
@@
 F 4 "Value" H 6150 2600 60  0001 C CNN "Manuf"
 F 5 "RES SMD 1k 5% [0402]" H 6900 3150 60  0001 C CNN "BOM"
+F 6 "R83" H 6150 2600 50 0001 C CNN "OldReference"
 	1    6150 2600
 	1    0    0    -1
@@
 F 4 "Value" H 6150 3000 60  0001 C CNN "Manuf"
 F 5 "RES SMD 1k 5% [0402]" H 6900 3550 60  0001 C CNN "BOM"
+F 6 "R84" H 6150 3000 50 0001 C CNN "OldReference"
 	1    6150 3000
 	1    0    0    -1
@@
 F 2 "" H 7250 3150 60  0000 C CNN
 F 3 "" H 7250 3150 60  0000 C CNN
+F 4 "L6" H 7250 3100 50 0001 C CNN "OldReference"
 	1    7250 3100
 	0    1    1    0
@@
 F 2 "" H 6650 4150 60  0000 C CNN
 F 3 "" H 6650 4150 60  0000 C CNN
+F 4 "D3" H 6650 4150 50 0001 C CNN "OldReference"
 	1    6650 4150
 	1    0    0    1
@@
 F 4 "SEMI GENERIC MMBT3904" H 6900 3850 60  0001 C CNN "BOM"
 F 5 "Value" H 6100 3300 60  0001 C CNN "Manuf"
+F 6 "Q13" H 6100 3300 50 0001 C CNN "OldReference"
 	1    6100 3300
 	1    0    0    -1
@@
 F 2 "" H 7990 4075 60  0000 C CNN
 F 3 "" H 7990 4075 60  0000 C CNN
+F 4 "C88" H 8000 4100 50 0001 C CNN "OldReference"
 	1    8000 4100
 	1    0    0    -1
@@
 F 4 "Value" H 7750 3100 60  0001 C CNN "Manuf"
 F 5 "RES SMD 1 5% [1210]" H 8500 3650 60  0001 C CNN "BOM"
+F 6 "R85" H 7750 3100 50 0001 C CNN "OldReference"
 	1    7750 3100
 	0    1    1    0
@@
 F 4 "Value" H 6250 3900 60  0001 C CNN "Manuf"
 F 5 "CAP MLCC 1nF C0G 10V 5% [0402]" H 7050 4450 60  0001 C CNN "BOM"
+F 6 "C87" H 6250 3900 50 0001 C CNN "OldReference"
 	1    6250 3900
 	0    1    1    0
@@
 F 4 "Value" H 5800 4150 60  0001 C CNN "Manuf"
 F 5 "CAP MLCC 10n ≥X5R 25V 10% [0402]" H 6600 4700 60  0001 C CNN "BOM"
+F 6 "C86" H 5800 4150 50 0001 C CNN "OldReference"
 	1    5800 4150
 	1    0    0    1
@@
 F 4 "Value" H 5800 3000 60  0001 C CNN "Manuf"
 F 5 "RES SMD 1k 5% [0402]" H 6550 3550 60  0001 C CNN "BOM"
+F 6 "R82" H 5800 3000 50 0001 C CNN "OldReference"
 	1    5800 3000
 	1    0    0    -1
@@
 F 4 "SEMI GENERIC MMBT3904" H 8750 3350 60  0001 C CNN "BOM"
 F 5 "Value" H 7950 2800 60  0001 C CNN "Manuf"
+F 6 "Q15" H 7950 2800 50 0001 C CNN "OldReference"
 	1    7950 2800
 	1    0    0    -1
@@
 F 2 "smd-semi:SOT-23" H 8550 4100 50  0001 C CNN
 F 3 "" H 8550 4100 60  0000 C CNN
+F 4 "DZ9" H 8550 4100 50 0001 C CNN "OldReference"
 	1    8550 4100
 	1    0    0    -1
@@
 F 2 "" H 8150 3900 60  0000 C CNN
 F 3 "" H 8150 3900 60  0000 C CNN
+F 4 "#PWR8" H 8150 3900 50 0001 C CNN "OldReference"
 	1    8150 3900
 	0    -1   -1   0

Commit message: BOM line fixes
Parts:
- C86, C87, Q13, Q15, R82, R83, R84, R85: Manuf Value -> (none)
Changed lines of the file:
@@
 F 2 "IPC7351-Nominal:RESC1005X40" H 6150 2600 50  0001 C CNN
 F 3 "" H 6150 2650 60  0000 C CNN
-F 4 "Value" H 6150 2600 60  0001 C CNN "Manuf"
+F 4 "" H 6150 2600 60  0001 C CNN "Manuf"
 F 5 "RES SMD 1k 5% [0402]" H 6900 3150 60  0001 C CNN "BOM"
 F 6 "R83" H 6150 2600 50 0001 C CNN "OldReference"
@@
 F 2 "IPC7351-Nominal:RESC1005X40" H 6150 3000 50  0001 C CNN
 F 3 "" H 6150 3050 60  0000 C CNN
-F 4 "Value" H 6150 3000 60  0001 C CNN "Manuf"
+F 4 "" H 6150 3000 60  0001 C CNN "Manuf"
 F 5 "RES SMD 1k 5% [0402]" H 6900 3550 60  0001 C CNN "BOM"
 F 6 "R84" H 6150 3000 50 0001 C CNN "OldReference"
@@
 F 3 "" H 6100 3300 60  0000 C CNN
 F 4 "SEMI GENERIC MMBT3904" H 6900 3850 60  0001 C CNN "BOM"
-F 5 "Value" H 6100 3300 60  0001 C CNN "Manuf"
+F 5 "" H 6100 3300 60  0001 C CNN "Manuf"
 F 6 "Q13" H 6100 3300 50 0001 C CNN "OldReference"
 	1    6100 3300
@@
 F 2 "IPC7351-Nominal:RESC3225X60" H 7750 3100 50  0001 C CNN
 F 3 "" H 7750 3150 60  0000 C CNN
-F 4 "Value" H 7750 3100 60  0001 C CNN "Manuf"
+F 4 "" H 7750 3100 60  0001 C CNN "Manuf"
 F 5 "RES SMD 1 5% [1210]" H 8500 3650 60  0001 C CNN "BOM"
 F 6 "R85" H 7750 3100 50 0001 C CNN "OldReference"
@@
 F 2 "IPC7351-Nominal:CAPC1005X55" H 6250 3900 50  0001 C CNN
 F 3 "" H 6240 3875 60  0000 C CNN
-F 4 "Value" H 6250 3900 60  0001 C CNN "Manuf"
+F 4 "" H 6250 3900 60  0001 C CNN "Manuf"
 F 5 "CAP MLCC 1nF C0G 10V 5% [0402]" H 7050 4450 60  0001 C CNN "BOM"
 F 6 "C87" H 6250 3900 50 0001 C CNN "OldReference"
@@
 F 2 "IPC7351-Nominal:CAPC1005X55" H 5800 4150 50  0001 C CNN
 F 3 "" H 5790 4125 60  0000 C CNN
-F 4 "Value" H 5800 4150 60  0001 C CNN "Manuf"
+F 4 "" H 5800 4150 60  0001 C CNN "Manuf"
 F 5 "CAP MLCC 10n ≥X5R 25V 10% [0402]" H 6600 4700 60  0001 C CNN "BOM"
 F 6 "C86" H 5800 4150 50 0001 C CNN "OldReference"
@@
 F 2 "IPC7351-Nominal:RESC1005X40" H 5800 3000 50  0001 C CNN
 F 3 "" H 5800 3050 60  0000 C CNN
-F 4 "Value" H 5800 3000 60  0001 C CNN "Manuf"
+F 4 "" H 5800 3000 60  0001 C CNN "Manuf"
 F 5 "RES SMD 1k 5% [0402]" H 6550 3550 60  0001 C CNN "BOM"
 F 6 "R82" H 5800 3000 50 0001 C CNN "OldReference"
@@
 F 3 "" H 7950 2800 60  0000 C CNN
 F 4 "SEMI GENERIC MMBT3904" H 8750 3350 60  0001 C CNN "BOM"
-F 5 "Value" H 7950 2800 60  0001 C CNN "Manuf"
+F 5 "" H 7950 2800 60  0001 C CNN "Manuf"
 F 6 "Q15" H 7950 2800 50 0001 C CNN "OldReference"
 	1    7950 2800
