File: wcp52/Protection.sch (KiCad schematic (older format))
At the start: 14 parts

Commit message: More doc fixes
Changed lines of the file:
@@
 	0    1    1    0
 $EndComp
+Wire Wire Line
+	2350 2600 2375 2625
+Wire Wire Line
+	2375 2625 3325 2625
+Wire Wire Line
+	3325 2625 3350 2600
+Wire Wire Line
+	3550 2600 3575 2625
+Wire Wire Line
+	3575 2625 4625 2625
+Wire Wire Line
+	4625 2625 4650 2600
+Wire Wire Line
+	6350 2600 6375 2625
+Wire Wire Line
+	6375 2625 7325 2625
+Wire Wire Line
+	7325 2625 7350 2600
+Wire Wire Line
+	7550 2600 7575 2625
+Wire Wire Line
+	7575 2625 8625 2625
+Wire Wire Line
+	8625 2625 8650 2600
 $EndSCHEMATC

Commit message: Nicer BOM lines
Parts:
- DZ3: BOM SEMI ONSEMI ESD9L5.0ST5G -> TVS ONSEMI ESD9L5.0ST5G; OldReference DZ1 -> (none)
- DZ4: BOM SEMI ONSEMI ESD9L5.0ST5G -> TVS ONSEMI ESD9L5.0ST5G; OldReference DZ3 -> (none)
- DZ5: BOM SEMI GENERIC BZX84C2V7 -> ZENER BZX84C2V7; OldReference DZ2 -> (none)
- DZ6: BOM SEMI GENERIC BZX84C2V7 -> ZENER BZX84C2V7; OldReference DZ4 -> (none)
- DZ7: BOM SEMI ONSEMI ESD9L5.0ST5G -> TVS ONSEMI ESD9L5.0ST5G; OldReference DZ5 -> (none)
- DZ8: BOM SEMI ONSEMI ESD9L5.0ST5G -> TVS ONSEMI ESD9L5.0ST5G; OldReference DZ7 -> (none)
- R57: OldReference R54 -> (none)
- R58: OldReference R55 -> (none)
- R59: OldReference R57 -> (none)
- R60: OldReference R56 -> (none)
- R61: OldReference R58 -> (none)
- R62: OldReference R59 -> (none)
- R63: OldReference R60 -> (none)
- R64: OldReference R62 -> (none)
Changed lines of the file:
@@
 F 2 "" H 2850 3100 60  0000 C CNN
 F 3 "" H 2850 3100 60  0000 C CNN
-F 4 "#PWR0171" H 2850 3100 50  0001 C CNN "OldReference"
 	1    2850 3100
 	1    0    0    -1
@@
 F 2 "" H 3150 3100 60  0000 C CNN
 F 3 "" H 3150 3100 60  0000 C CNN
-F 4 "#PWR0172" H 3150 3100 50  0001 C CNN "OldReference"
 	1    3150 3100
 	1    0    0    -1
@@
 F 4 "ESD9L5.0ST5G" H 3700 3800 60  0001 C CNN "PN"
 F 5 "ONSemi" H 3700 3800 60  0001 C CNN "Manuf"
-F 6 "SEMI ONSEMI ESD9L5.0ST5G" H 3700 3800 60  0001 C CNN "BOM"
-F 7 "DZ1" H 3700 3800 50  0001 C CNN "OldReference"
+F 6 "TVS ONSEMI ESD9L5.0ST5G" H 3700 3800 60  0001 C CNN "BOM"
 	1    3700 3800
 	1    0    0    1
@@
 F 4 "ESD9L5.0ST5G" H 4500 3800 60  0001 C CNN "PN"
 F 5 "ONSemi" H 4500 3800 60  0001 C CNN "Manuf"
-F 6 "SEMI ONSEMI ESD9L5.0ST5G" H 4500 3800 60  0001 C CNN "BOM"
-F 7 "DZ3" H 4500 3800 50  0001 C CNN "OldReference"
+F 6 "TVS ONSEMI ESD9L5.0ST5G" H 4500 3800 60  0001 C CNN "BOM"
 	1    4500 3800
 	1    0    0    -1
@@
 F 3 "" H 5350 5400 60  0000 C CNN
 F 4 "BZX84C2V7" H 5350 5400 60  0001 C CNN "PN"
-F 5 "SEMI GENERIC BZX84C2V7" H 5350 5400 60  0001 C CNN "BOM"
-F 6 "DZ2" H 5350 5400 50  0001 C CNN "OldReference"
+F 5 "ZENER BZX84C2V7" H 5350 5400 60  0001 C CNN "BOM"
 	1    5350 5400
 	1    0    0    -1
@@
 F 3 "" H 6150 5400 60  0000 C CNN
 F 4 "BZX84C2V7" H 6150 5400 60  0001 C CNN "PN"
-F 5 "SEMI GENERIC BZX84C2V7" H 6150 5400 60  0001 C CNN "BOM"
-F 6 "DZ4" H 6150 5400 50  0001 C CNN "OldReference"
+F 5 "ZENER BZX84C2V7" H 6150 5400 60  0001 C CNN "BOM"
 	1    6150 5400
 	1    0    0    1
@@
 F 2 "" H 5750 5650 60  0000 C CNN
 F 3 "" H 5750 5650 60  0000 C CNN
-F 4 "#PWR0173" H 5750 5650 50  0001 C CNN "OldReference"
 	1    5750 5650
 	1    0    0    -1
@@
 F 2 "" H 4700 5150 60  0000 C CNN
 F 3 "" H 4700 5150 60  0000 C CNN
-F 4 "#PWR0174" H 4700 5150 50  0001 C CNN "OldReference"
 	1    4700 5150
 	1    0    0    -1
@@
 F 2 "" H 6800 5300 60  0000 C CNN
 F 3 "" H 6800 5300 60  0000 C CNN
-F 4 "#PWR0175" H 6800 5300 50  0001 C CNN "OldReference"
 	1    6800 5300
 	1    0    0    -1
@@
 F 2 "" H 6850 3100 60  0000 C CNN
 F 3 "" H 6850 3100 60  0000 C CNN
-F 4 "#PWR0176" H 6850 3100 50  0001 C CNN "OldReference"
 	1    6850 3100
 	1    0    0    -1
@@
 F 2 "" H 7150 3100 60  0000 C CNN
 F 3 "" H 7150 3100 60  0000 C CNN
-F 4 "#PWR0177" H 7150 3100 50  0001 C CNN "OldReference"
 	1    7150 3100
 	1    0    0    -1
@@
 F 4 "ESD9L5.0ST5G" H 7700 3800 60  0001 C CNN "PN"
 F 5 "ONSemi" H 7700 3800 60  0001 C CNN "Manuf"
-F 6 "SEMI ONSEMI ESD9L5.0ST5G" H 7700 3800 60  0001 C CNN "BOM"
-F 7 "DZ5" H 7700 3800 50  0001 C CNN "OldReference"
+F 6 "TVS ONSEMI ESD9L5.0ST5G" H 7700 3800 60  0001 C CNN "BOM"
 	1    7700 3800
 	1    0    0    1
@@
 F 4 "ESD9L5.0ST5G" H 8500 3800 60  0001 C CNN "PN"
 F 5 "ONSemi" H 8500 3800 60  0001 C CNN "Manuf"
-F 6 "SEMI ONSEMI ESD9L5.0ST5G" H 8500 3800 60  0001 C CNN "BOM"
-F 7 "DZ7" H 8500 3800 50  0001 C CNN "OldReference"
+F 6 "TVS ONSEMI ESD9L5.0ST5G" H 8500 3800 60  0001 C CNN "BOM"
 	1    8500 3800
 	1    0    0    -1
@@
 F 4 "" H 2850 2900 60  0001 C CNN "Manuf"
 F 5 "RES SMD 1.6k 1% [0603]" H 3600 3450 60  0001 C CNN "BOM"
-F 6 "R54" H 2850 2900 50  0001 C CNN "OldReference"
 	1    2850 2900
 	1    0    0    -1
@@
 F 4 "" H 3150 2900 60  0001 C CNN "Manuf"
 F 5 "RES SMD 1.6k 1% [0603]" H 3900 3450 60  0001 C CNN "BOM"
-F 6 "R55" H 3150 2900 50  0001 C CNN "OldReference"
 	1    3150 2900
 	1    0    0    -1
@@
 F 4 "" H 6850 2900 60  0001 C CNN "Manuf"
 F 5 "RES SMD 1.6k 1% [0603]" H 7600 3450 60  0001 C CNN "BOM"
-F 6 "R59" H 6850 2900 50  0001 C CNN "OldReference"
 	1    6850 2900
 	1    0    0    -1
@@
 F 4 "" H 7150 2900 60  0001 C CNN "Manuf"
 F 5 "RES SMD 1.6k 1% [0603]" H 7900 3450 60  0001 C CNN "BOM"
-F 6 "R60" H 7150 2900 50  0001 C CNN "OldReference"
 	1    7150 2900
 	1    0    0    -1
@@
 F 3 "" H 3450 2650 60  0000 C CNN
 F 4 "RES SMD 3.3 10% [0603]" H 4200 3150 60  0001 C CNN "BOM"
-F 5 "R57" H 3450 2600 50  0001 C CNN "OldReference"
 	1    3450 2600
 	0    1    1    0
@@
 F 3 "" H 7450 2650 60  0000 C CNN
 F 4 "RES SMD 3.3 10% [0603]" H 8200 3150 60  0001 C CNN "BOM"
-F 5 "R62" H 7450 2600 50  0001 C CNN "OldReference"
 	1    7450 2600
 	0    1    1    0
@@
 F 4 "" H 5000 5200 60  0001 C CNN "Manuf"
 F 5 "RES SMD 750 1% [0603]" H 5750 5750 60  0001 C CNN "BOM"
-F 6 "R56" H 5000 5200 50  0001 C CNN "OldReference"
 	1    5000 5200
 	0    1    1    0
@@
 F 4 "" H 6500 5200 60  0001 C CNN "Manuf"
 F 5 "RES SMD 750 1% [0603]" H 7250 5750 60  0001 C CNN "BOM"
-F 6 "R58" H 6500 5200 50  0001 C CNN "OldReference"
 	1    6500 5200
 	0    1    1    0
