File: wcp52/wcp52.sch (KiCad schematic (older format))
At the start: 34 parts, among them J1 9V 300mA, J2 IN1, J3 IN2, J4 OUT, J5 AUX

Commit message: BOM fixes
Parts:
- DZ1: BOM SEMI ONSEMI 1SMA59xxBT3G -> SEMI ONSEMI 1SMA5914BT3G; PN 1SMA59xxBT3G -> 1SMA5914BT3G
Changed lines of the file:
@@
 EESchema Schematic File Version 2
-LIBS:Altera
-LIBS:AnalogDevices
-LIBS:Atmel
-LIBS:conn-2mm
-LIBS:conn-100mil
-LIBS:conn-cui
-LIBS:conn-fci
-LIBS:conn-linx
-LIBS:conn-molex
-LIBS:conn-tagconnect
-LIBS:conn-test
-LIBS:DiodesInc
-LIBS:display
-LIBS:_electromech
-LIBS:Fairchild
-LIBS:FTDI
-LIBS:Intersil
-LIBS:Lattice
-LIBS:_linear
-LIBS:LinearTech
-LIBS:Littelfuse
-LIBS:logic-4000
-LIBS:logic-7400
-LIBS:MACOM
-LIBS:maxim
-LIBS:mechanical
-LIBS:Microchip
-LIBS:Micron
-LIBS:NXP
-LIBS:onsemi
-LIBS:passive
-LIBS:pasv-BiTech
-LIBS:pasv-Bourns
-LIBS:pasv-cap
-LIBS:pasv-ind
-LIBS:pasv-res
-LIBS:pcb
-LIBS:power
-LIBS:_semi
-LIBS:semi-diode-1N
-LIBS:semi-diode-BA
-LIBS:semi-diode-MCC
-LIBS:semi-diode-MMB
-LIBS:semi-diode-NXP
-LIBS:semi-diode-OnSemi
-LIBS:semi-diode-Vishay
-LIBS:semi-opto-misc
-LIBS:semi-thyristor-2N
-LIBS:semi-trans-2N
-LIBS:semi-trans-AO
-LIBS:semi-trans-BC
-LIBS:semi-trans-DiodesInc
-LIBS:semi-trans-Fairchild
-LIBS:semi-trans-Infineon
-LIBS:semi-trans-IntRect
-LIBS:semi-trans-IXYS
-LIBS:semi-trans-misc
-LIBS:semi-trans-MMB
-LIBS:semi-trans-MPS
-LIBS:semi-trans-NXP
-LIBS:semi-trans-PZT
-LIBS:semi-trans-TI
-LIBS:semi-trans-TIP
-LIBS:semi-trans-Toshiba
-LIBS:silabs
-LIBS:skyworks
-LIBS:ST
-LIBS:st_ic
-LIBS:st_semi
-LIBS:supertex
-LIBS:symbol
-LIBS:TexasInstruments
-LIBS:vishay_semi
-LIBS:Xilinx
-LIBS:pasv-xtal
-LIBS:conn-te
 LIBS:wcp52-cache
 EELAYER 25 0
@@
 F 2 "IPC7351-Nominal:DIOM5226X203" H 9950 700 60  0001 C CNN
 F 3 "" H 9700 750 60  0000 C CNN
-F 4 "1SMA59xxBT3G" H 10150 900 50  0001 C CNN "PN"
+F 4 "1SMA5914BT3G" H 10150 900 50  0001 C CNN "PN"
 F 5 "ONSemi" H 9700 750 50  0001 C CNN "Manuf"
-F 6 "SEMI ONSEMI 1SMA59xxBT3G" H 10550 1300 50  0001 C CNN "BOM"
+F 6 "SEMI ONSEMI 1SMA5914BT3G" H 10550 1300 50  0001 C CNN "BOM"
 F 7 "DZ12" H 9700 750 50  0001 C CNN "OldReference"
 	1    9700 750

Commit message: Prepare to fab
Changed lines of the file:
@@
 	10250 1500 10150 1500
 Wire Wire Line
-	5600 1100 7900 1100
+	5600 1100 10250 1100
 Wire Wire Line
-	7900 1100 10250 1100
-Wire Wire Line
-	5700 1400 7600 1400
-Wire Wire Line
-	7600 1400 10250 1400
+	5700 1400 10250 1400
 Wire Wire Line
 	8300 1200 8300 1000
@@
 $EndComp
 Wire Wire Line
-	8300 1300 8500 1300
+	8300 1300 9100 1300
 Wire Wire Line
-	8500 1300 9100 1300
-Wire Wire Line
-	8300 1200 8500 1200
-Wire Wire Line
-	8500 1200 9100 1200
+	8300 1200 9100 1200
 Wire Wire Line
 	9300 1200 10250 1200
@@
 $EndComp
 Wire Wire Line
-	9400 1000 9700 1000
-Wire Wire Line
-	9700 1000 9900 1000
+	9400 1000 9900 1000
 Wire Wire Line
 	10100 1000 10250 1000

Commit message: BOM line fixes
Parts:
- DS2, DS3, DS4, DS5, DS6, DS7, R1, R2, R3, R4, R5, R6, R7, R8, R9: Manuf Value -> (none)
- J1: Description (none) -> CONN BARREL 2x6.5MM
- J2, J3, J4: Description (none) -> CONN SMA RIGHTANGLE FEMALE; Manuf (none) -> TE; PN (none) -> 5-1814400-1
- R10, R11, R12: Description (none) -> PPTC 50mA/150mA 60V [1206]
Changed lines of the file:
@@
 EESchema Schematic File Version 2
+LIBS:Altera
+LIBS:AnalogDevices
+LIBS:Atmel
+LIBS:conn-2mm
+LIBS:conn-100mil
+LIBS:conn-cui
+LIBS:conn-fci
+LIBS:conn-linx
+LIBS:conn-molex
+LIBS:conn-tagconnect
+LIBS:conn-test
+LIBS:DiodesInc
+LIBS:display
+LIBS:_electromech
+LIBS:Fairchild
+LIBS:FTDI
+LIBS:Intersil
+LIBS:Lattice
+LIBS:_linear
+LIBS:LinearTech
+LIBS:Littelfuse
+LIBS:logic-4000
+LIBS:logic-7400
+LIBS:MACOM
+LIBS:maxim
+LIBS:mechanical
+LIBS:Microchip
+LIBS:Micron
+LIBS:NXP
+LIBS:onsemi
+LIBS:passive
+LIBS:pasv-BiTech
+LIBS:pasv-Bourns
+LIBS:pasv-cap
+LIBS:pasv-ind
+LIBS:pasv-res
+LIBS:pcb
+LIBS:power
+LIBS:_semi
+LIBS:semi-diode-1N
+LIBS:semi-diode-BA
+LIBS:semi-diode-MCC
+LIBS:semi-diode-MMB
+LIBS:semi-diode-NXP
+LIBS:semi-diode-OnSemi
+LIBS:semi-diode-Vishay
+LIBS:semi-opto-misc
+LIBS:semi-thyristor-2N
+LIBS:semi-trans-2N
+LIBS:semi-trans-AO
+LIBS:semi-trans-BC
+LIBS:semi-trans-DiodesInc
+LIBS:semi-trans-Fairchild
+LIBS:semi-trans-Infineon
+LIBS:semi-trans-IntRect
+LIBS:semi-trans-IXYS
+LIBS:semi-trans-misc
+LIBS:semi-trans-MMB
+LIBS:semi-trans-MPS
+LIBS:semi-trans-NXP
+LIBS:semi-trans-PZT
+LIBS:semi-trans-TI
+LIBS:semi-trans-TIP
+LIBS:semi-trans-Toshiba
+LIBS:silabs
+LIBS:skyworks
+LIBS:ST
+LIBS:st_ic
+LIBS:st_semi
+LIBS:supertex
+LIBS:symbol
+LIBS:TexasInstruments
+LIBS:vishay_semi
+LIBS:Xilinx
+LIBS:pasv-xtal
+LIBS:conn-te
 LIBS:wcp52-cache
 EELAYER 25 0
@@
 F 5 "CUI" H 1050 1700 60  0001 C CNN "Manuf"
 F 6 "DIST DIGIKEY CP-037A-ND" H 1050 1700 60  0001 C CNN "BOM"
-F 7 "J5" H 1050 1700 50  0001 C CNN "OldReference"
+F 7 "CONN BARREL 2x6.5MM" H 1050 1700 60  0001 C CNN "Description"
+F 8 "J5" H 1050 1700 50  0001 C CNN "OldReference"
 	1    1050 1700
 	-1   0    0    -1
@@
 F 2 "manuf:CONN-TE-1814400" H 10300 2300 50  0001 C CNN
 F 3 "" H 10300 2300 50  0000 C CNN
-F 4 "DIST DIGIKEY A97593-ND" H 10300 2300 60  0001 C CNN "BOM"
-F 5 "J2" H 10300 2300 50  0001 C CNN "OldReference"
+F 4 "5-1814400-1" H 10300 2300 60  0001 C CNN "PN"
+F 5 "TE" H 10300 2300 60  0001 C CNN "Manuf"
+F 6 "DIST DIGIKEY A97593-ND" H 10300 2300 60  0001 C CNN "BOM"
+F 7 "CONN SMA RIGHTANGLE FEMALE" H 10300 2300 60  0001 C CNN "Description"
+F 8 "J2" H 10300 2300 50  0001 C CNN "OldReference"
 	1    10300 2300
 	-1   0    0    -1
@@
 F 2 "manuf:CONN-TE-1814400" H 10300 2800 50  0001 C CNN
 F 3 "" H 10300 2800 50  0000 C CNN
-F 4 "DIST DIGIKEY A97593-ND" H 10300 2800 60  0001 C CNN "BOM"
-F 5 "J3" H 10300 2800 50  0001 C CNN "OldReference"
+F 4 "5-1814400-1" H 10300 2800 60  0001 C CNN "PN"
+F 5 "TE" H 10300 2800 60  0001 C CNN "Manuf"
+F 6 "DIST DIGIKEY A97593-ND" H 10300 2800 60  0001 C CNN "BOM"
+F 7 "CONN SMA RIGHTANGLE FEMALE" H 10300 2800 60  0001 C CNN "Description"
+F 8 "J3" H 10300 2800 50  0001 C CNN "OldReference"
 	1    10300 2800
 	-1   0    0    -1
@@
 F 2 "manuf:CONN-TE-1814400" H 10300 4200 50  0001 C CNN
 F 3 "" H 10300 4200 50  0000 C CNN
-F 4 "DIST DIGIKEY A97593-ND" H 10300 4200 60  0001 C CNN "BOM"
-F 5 "J4" H 10300 4200 50  0001 C CNN "OldReference"
+F 4 "5-1814400-1" H 10300 4200 60  0001 C CNN "PN"
+F 5 "TE" H 10300 4200 60  0001 C CNN "Manuf"
+F 6 "DIST DIGIKEY A97593-ND" H 10300 4200 60  0001 C CNN "BOM"
+F 7 "CONN SMA RIGHTANGLE FEMALE" H 10300 4200 60  0001 C CNN "Description"
+F 8 "J4" H 10300 4200 50  0001 C CNN "OldReference"
 	1    10300 4200
 	-1   0    0    -1
@@
 F 5 "Bel Fuse" H 9200 1200 60  0001 C CNN "Manuf"
 F 6 "DIST DIGIKEY 507-1793-1-ND" V 9200 1200 60  0001 C CNN "BOM"
-F 7 "R106" H 9200 1200 50  0001 C CNN "OldReference"
+F 7 "PPTC 50mA/150mA 60V [1206]" H 9200 1200 60  0001 C CNN "Description"
+F 8 "R106" H 9200 1200 50  0001 C CNN "OldReference"
 	1    9200 1200
 	0    -1   1    0
@@
 F 5 "Bel Fuse" H 9200 1300 60  0001 C CNN "Manuf"
 F 6 "DIST DIGIKEY 507-1793-1-ND" V 9200 1300 60  0001 C CNN "BOM"
-F 7 "R107" H 9200 1300 50  0001 C CNN "OldReference"
+F 7 "PPTC 50mA/150mA 60V [1206]" H 9200 1300 60  0001 C CNN "Description"
+F 8 "R107" H 9200 1300 50  0001 C CNN "OldReference"
 	1    9200 1300
 	0    -1   1    0
@@
 F 5 "Bel Fuse" H 10000 1000 60  0001 C CNN "Manuf"
 F 6 "DIST DIGIKEY 507-1793-1-ND" V 10000 1000 60  0001 C CNN "BOM"
-F 7 "R105" H 10000 1000 50  0001 C CNN "OldReference"
+F 7 "PPTC 50mA/150mA 60V [1206]" H 10000 1000 60  0001 C CNN "Description"
+F 8 "R105" H 10000 1000 50  0001 C CNN "OldReference"
 	1    10000 1000
 	0    -1   1    0
@@
 F 2 "smd-semi:LED-0603" H 3200 7650 50  0001 C CNN
 F 3 "" H 3200 7650 60  0000 C CNN
-F 4 "Value" H 3200 7650 60  0001 C CNN "Manuf"
+F 4 "" H 3200 7650 60  0001 C CNN "Manuf"
 F 5 "SEMI GENERIC LED RED [0603]" H 4050 8200 60  0001 C CNN "BOM"
 F 6 "DS2" H 3200 7650 50  0001 C CNN "OldReference"
@@
 F 2 "IPC7351-Nominal:RESC1608X50" H 3200 7350 50  0001 C CNN
 F 3 "" H 3200 7400 60  0000 C CNN
-F 4 "Value" H 3200 7350 60  0001 C CNN "Manuf"
+F 4 "" H 3200 7350 60  0001 C CNN "Manuf"
 F 5 "RES SMD 1.6k 1% [0603]" H 3950 7900 60  0001 C CNN "BOM"
 F 6 "R90" H 3200 7350 50  0001 C CNN "OldReference"
@@
 F 2 "IPC7351-Nominal:RESC1608X50" H 7600 900 50  0001 C CNN
 F 3 "" H 7600 950 60  0000 C CNN
-F 4 "Value" H 7600 900 60  0001 C CNN "Manuf"
+F 4 "" H 7600 900 60  0001 C CNN "Manuf"
 F 5 "RES SMD 3.3k 5% [0603]" H 8350 1450 60  0001 C CNN "BOM"
 F 6 "R91" H 7600 900 50  0001 C CNN "OldReference"
@@
 F 2 "IPC7351-Nominal:RESC1608X50" H 7900 900 50  0001 C CNN
 F 3 "" H 7900 950 60  0000 C CNN
-F 4 "Value" H 7900 900 60  0001 C CNN "Manuf"
+F 4 "" H 7900 900 60  0001 C CNN "Manuf"
 F 5 "RES SMD 3.3k 5% [0603]" H 8650 1450 60  0001 C CNN "BOM"
 F 6 "R92" H 7900 900 50  0001 C CNN "OldReference"
@@
 F 2 "IPC7351-Nominal:RESC1608X50" H 2700 7350 50  0001 C CNN
 F 3 "" H 2700 7400 60  0000 C CNN
-F 4 "Value" H 2700 7350 60  0001 C CNN "Manuf"
+F 4 "" H 2700 7350 60  0001 C CNN "Manuf"
 F 5 "RES SMD 3.3k 5% [0603]" H 3450 7900 60  0001 C CNN "BOM"
 F 6 "R53" H 2700 7350 50  0001 C CNN "OldReference"
@@
 F 2 "smd-semi:LED-0603" H 5150 7650 50  0001 C CNN
 F 3 "" H 5150 7650 60  0000 C CNN
-F 4 "Value" H 5150 7650 60  0001 C CNN "Manuf"
+F 4 "" H 5150 7650 60  0001 C CNN "Manuf"
 F 5 "SEMI GENERIC LED RED [0603]" H 6000 8200 60  0001 C CNN "BOM"
 F 6 "DS7" H 5150 7650 50  0001 C CNN "OldReference"
@@
 F 2 "IPC7351-Nominal:RESC1608X50" H 5150 7350 50  0001 C CNN
 F 3 "" H 5150 7400 60  0000 C CNN
-F 4 "Value" H 5150 7350 60  0001 C CNN "Manuf"
+F 4 "" H 5150 7350 60  0001 C CNN "Manuf"
 F 5 "RES SMD 1.6k 1% [0603]" H 5900 7900 60  0001 C CNN "BOM"
 F 6 "R111" H 5150 7350 50  0001 C CNN "OldReference"
@@
 F 2 "smd-semi:LED-0603" H 5600 7650 50  0001 C CNN
 F 3 "" H 5600 7650 60  0000 C CNN
-F 4 "Value" H 5600 7650 60  0001 C CNN "Manuf"
+F 4 "" H 5600 7650 60  0001 C CNN "Manuf"
 F 5 "SEMI GENERIC LED RED [0603]" H 6450 8200 60  0001 C CNN "BOM"
 F 6 "DS8" H 5600 7650 50  0001 C CNN "OldReference"
@@
 F 2 "IPC7351-Nominal:RESC1608X50" H 5600 7350 50  0001 C CNN
 F 3 "" H 5600 7400 60  0000 C CNN
-F 4 "Value" H 5600 7350 60  0001 C CNN "Manuf"
+F 4 "" H 5600 7350 60  0001 C CNN "Manuf"
 F 5 "RES SMD 3.3k 5% [0603]" H 6350 7900 60  0001 C CNN "BOM"
 F 6 "R113" H 5600 7350 50  0001 C CNN "OldReference"
@@
 F 2 "smd-semi:LED-0603" H 3650 7650 50  0001 C CNN
 F 3 "" H 3650 7650 60  0000 C CNN
-F 4 "Value" H 3650 7650 60  0001 C CNN "Manuf"
+F 4 "" H 3650 7650 60  0001 C CNN "Manuf"
 F 5 "SEMI GENERIC LED RED [0603]" H 4500 8200 60  0001 C CNN "BOM"
 F 6 "DS9" H 3650 7650 50  0001 C CNN "OldReference"
@@
 F 2 "IPC7351-Nominal:RESC1608X50" H 3650 7350 50  0001 C CNN
 F 3 "" H 3650 7400 60  0000 C CNN
-F 4 "Value" H 3650 7350 60  0001 C CNN "Manuf"
+F 4 "" H 3650 7350 60  0001 C CNN "Manuf"
 F 5 "RES SMD 1.6k 1% [0603]" H 4400 7900 60  0001 C CNN "BOM"
 F 6 "R114" H 3650 7350 50  0001 C CNN "OldReference"
@@
 F 2 "smd-semi:LED-0603" H 4650 7650 50  0001 C CNN
 F 3 "" H 4650 7650 60  0000 C CNN
-F 4 "Value" H 4650 7650 60  0001 C CNN "Manuf"
+F 4 "" H 4650 7650 60  0001 C CNN "Manuf"
 F 5 "SEMI GENERIC LED RED [0603]" H 5500 8200 60  0001 C CNN "BOM"
 F 6 "DS10" H 4650 7650 50  0001 C CNN "OldReference"
@@
 F 2 "IPC7351-Nominal:RESC1608X50" H 4650 7350 50  0001 C CNN
 F 3 "" H 4650 7400 60  0000 C CNN
-F 4 "Value" H 4650 7350 60  0001 C CNN "Manuf"
+F 4 "" H 4650 7350 60  0001 C CNN "Manuf"
 F 5 "RES SMD 1.6k 1% [0603]" H 5400 7900 60  0001 C CNN "BOM"
 F 6 "R115" H 4650 7350 50  0001 C CNN "OldReference"
@@
 F 2 "smd-semi:LED-0603" H 4100 7650 50  0001 C CNN
 F 3 "" H 4100 7650 60  0000 C CNN
-F 4 "Value" H 4100 7650 60  0001 C CNN "Manuf"
+F 4 "" H 4100 7650 60  0001 C CNN "Manuf"
 F 5 "SEMI GENERIC LED RED [0603]" H 4950 8200 60  0001 C CNN "BOM"
 F 6 "DS11" H 4100 7650 50  0001 C CNN "OldReference"
@@
 F 2 "IPC7351-Nominal:RESC1608X50" H 4100 7350 50  0001 C CNN
 F 3 "" H 4100 7400 60  0000 C CNN
-F 4 "Value" H 4100 7350 60  0001 C CNN "Manuf"
+F 4 "" H 4100 7350 60  0001 C CNN "Manuf"
 F 5 "RES SMD 1.6k 1% [0603]" H 4850 7900 60  0001 C CNN "BOM"
 F 6 "R116" H 4100 7350 50  0001 C CNN "OldReference"

Commit message: BOM corrections/combinations, etc
Add configuration for bomtool
Remove old schematic file no longer used
Parts:
- DS1: BOM (none) -> SEMI GENERIC LED RED [3mm]
Changed lines of the file:
@@
 F 2 "pth-semi:LED-3mm" H 2700 7650 50  0001 C CNN
 F 3 "" H 2700 7650 60  0000 C CNN
-F 4 "DS6" H 2700 7650 50  0001 C CNN "OldReference"
+F 4 "SEMI GENERIC LED RED [3mm]" H 2700 7650 60  0001 C CNN "BOM"
+F 5 "DS6" H 2700 7650 50  0001 C CNN "OldReference"
 	1    2700 7650
 	1    0    0    -1

Commit message: Schematic/doc work
Parts:
- added C1, C2: 10n, IPC7351-Nominal:CAPC1608X55, symbol C-0603
- added J6: MicroUSB-B, conn-fci:CONN-10118194-0001LF-FCI, symbol CONN-10118194-0001LF-UUSB-B
- added R13: 1M, IPC7351-Nominal:RESC1608X50, symbol R-0603
Connections:
- net GND: now also C1.2, C2.2, J6.5 (GND), R13.2
- new net Comm/EXT_USBD_N: J6.2 (D-)
- new net Comm/EXT_USBD_P: J6.3 (D+)
- new net Comm/EXT_VBUS: C2.1, J6.1 (V+)
- new net USBSHIELD: C1.1, J6.SH (SHIELD), R13.1
- no-connect marks 0 -> 1
Other:
- note added: "Arrows indicate direction\nof signal path"
- note added: "Double-struck wire indicates\nmajor signal path"
- note added: "EMI Filtering"
- note added: "Indicates predominantly\nsinusoidal signal at high speed"
- note added: "Indicates predominantly\nsquare signal"
- note added: "LEGEND"

Commit message: Schematic updates for documentation
Other:
- note added: "Sinusoidal signal"
- note added: "Square signal"
- note removed: "Indicates predominantly\nsinusoidal signal at high speed"
- note removed: "Indicates predominantly\nsquare signal"

Commit message: More doc fixes
Changed lines of the file:
@@
 Text Notes 8950 5250 0    50   ~ 0
 Sinusoidal signal
-$Comp
-L SQUARE #SYM35
-U 1 1 5512AFDA
-P 8700 5500
-F 0 "#SYM35" H 8700 5500 60  0001 C CNN
-F 1 "SQUARE" H 8700 5500 60  0001 C CNN
-F 2 "" H 8700 5500 60  0000 C CNN
-F 3 "" H 8700 5500 60  0000 C CNN
-	1    8700 5500
-	1    0    0    -1
-$EndComp
 Text Notes 8950 5550 0    50   ~ 0
 Square signal
-$Comp
-L SINE-FAST #SYM25
-U 1 1 5512CD34
-P 7100 3800
-F 0 "#SYM25" H 7100 3800 60  0001 C CNN
-F 1 "SINE-FAST" H 7100 3800 60  0001 C CNN
-F 2 "" H 7100 3800 60  0000 C CNN
-F 3 "" H 7100 3800 60  0000 C CNN
-	1    7100 3800
-	1    0    0    1
-$EndComp
 $Comp
 L SINE-ACCURATE #SYM38
@@
 	1    0    0    -1
 $EndComp
+$Comp
+L SINE-ACCURATE #SYM?
+U 1 1 550DC49A
+P 7100 3750
+F 0 "#SYM?" H 7100 3750 60  0001 C CNN
+F 1 "SINE-ACCURATE" H 7100 3750 60  0001 C CNN
+F 2 "" H 7100 3750 60  0000 C CNN
+F 3 "" H 7100 3750 60  0000 C CNN
+	1    7100 3750
+	1    0    0    1
+$EndComp
+$Comp
+L SQUARE-FAST #SYM?
+U 1 1 550DEAA5
+P 8700 5500
+F 0 "#SYM?" H 8700 5500 60  0001 C CNN
+F 1 "SQUARE-FAST" H 8700 5500 60  0001 C CNN
+F 2 "" H 8700 5500 60  0000 C CNN
+F 3 "" H 8700 5500 60  0000 C CNN
+	1    8700 5500
+	1    0    0    -1
+$EndComp

Commit message: More doc fixes
Other:
- note added: "PCB: 4-layer, ɛ approx= 3.66\nStackup:\n - 1oz/35µm copper outside, 0.5oz/17µm copper inside\n - prepreg: 200µm\n - core: 1.2mm\n\nDifferential T-line Zdiff = 100, Z0 = 67\n0.21 track, 0.16 space\nUse a recent devel version of KiCad with\ndifferential routing\n\nSingle-ended T-line Z0 = 50\n0.35 track"
- note added: "Power supply status LEDs"
- note added: "STANDARD PARTS, UNLESS LABELED:"
- note removed: "PCB: 4-layer, ɛ approx= 3.66\nStackup:\n - 1oz/35µm copper outside, 0.5oz/17µm copper inside\n - prepreg: 200µm\n - core: 1.2mm\n\nDifferential T-line Zdiff = 100, Z0 = 67\n0.21 track, 0.16 space\nUse a recent devel version of KiCad with differential routing\n\nSingle-ended T-line Z0 = 50\n0.35 track"
- moved on the sheet: DS1, J4, R1
