File: wcp52/Comm.sch (KiCad schematic (older format))
At the start: 17 parts, among them Q1 IRLML6402, U1 FT230XS_DNP

Commit message: Nicer BOM lines
Parts:
- C3: OldReference C63 -> (none)
- C4: OldReference C64 -> (none)
- C5: OldReference C92 -> (none)
- C6: OldReference C32 -> (none)
- C7: OldReference C33 -> (none)
- D3: BOM SEMI GENERIC MMBD4148 -> DIODE MMBD4148; OldReference D8 -> (none)
- D4: BOM SEMI GENERIC MMBD4148 -> DIODE MMBD4148; OldReference D9 -> (none)
- DZ2: BOM SEMI LITTELFUSE SP0503BAHT -> TVS LITTELFUSE SP0503BAHT; OldReference DZ10 -> (none)
- E1: OldReference E1 -> (none)
- Q1: BOM SEMI IRF IRLML6402 -> PMOS IRF IRLML6402; OldReference Q20 -> (none)
- R14: OldReference R7 -> (none)
- R15: OldReference R8 -> (none)
- R16: OldReference R37 -> (none)
- R17: OldReference R16 -> (none)
- TP4: OldReference TP3 -> (none)
- TP5: OldReference TP4 -> (none)
- U1: OldReference U13 -> (none)
Changed lines of the file:
@@
 F 5 "FTDI" H 7000 4200 60  0001 C CNN "Manuf"
 F 6 "#IC FTDI FT230XS" H 7000 4200 60  0001 C CNN "BOM"
-F 7 "U13" H 7000 4200 50  0001 C CNN "OldReference"
 	1    7000 4200
 	1    0    0    -1
@@
 F 4 "SP0503BAHTG" H 3150 4600 60  0001 C CNN "PN"
 F 5 "Littelfuse" H 3150 4600 60  0001 C CNN "Manuf"
-F 6 "SEMI LITTELFUSE SP0503BAHT" H 3150 4600 60  0001 C CNN "BOM"
-F 7 "DZ10" H 3150 4600 50  0001 C CNN "OldReference"
+F 6 "TVS LITTELFUSE SP0503BAHT" H 3150 4600 60  0001 C CNN "BOM"
 	1    3150 4600
 	1    0    0    -1
@@
 F 2 "" H 3150 4900 60  0000 C CNN
 F 3 "" H 3150 4900 60  0000 C CNN
-F 4 "#PWR042" H 3150 4900 50  0001 C CNN "OldReference"
 	1    3150 4900
 	1    0    0    -1
@@
 F 6 "DIST DIGIKEY 240-2562-1-ND" H 2250 3200 60  0001 C CNN "BOM"
 F 7 "FERRITE CHIP 2.2k @ 100MHz [0805]" H 2250 3200 60  0001 C CNN "Description"
-F 8 "E1" H 2250 3200 50  0001 C CNN "OldReference"
 	1    2250 3200
 	1    0    0    -1
@@
 F 4 "" H 5100 3400 60  0001 C CNN "Manuf"
 F 5 "CAP MLCC 10u ≥X5R 10V 10% [0805]" H 5900 3950 60  0001 C CNN "BOM"
-F 6 "C92" H 5100 3400 50  0001 C CNN "OldReference"
 	1    5100 3400
 	1    0    0    -1
@@
 F 2 "" H 5100 3600 60  0000 C CNN
 F 3 "" H 5100 3600 60  0000 C CNN
-F 4 "#PWR047" H 5100 3600 50  0001 C CNN "OldReference"
 	1    5100 3600
 	1    0    0    -1
@@
 F 2 "" H 5800 3800 60  0000 C CNN
 F 3 "" H 5800 3800 60  0000 C CNN
-F 4 "#PWR048" H 5800 3800 50  0001 C CNN "OldReference"
 	1    5800 3800
 	0    1    1    0
@@
 F 2 "" H 6300 4900 60  0000 C CNN
 F 3 "" H 6300 4900 60  0000 C CNN
-F 4 "#PWR049" H 6300 4900 50  0001 C CNN "OldReference"
 	1    6300 4900
 	1    0    0    -1
@@
 F 2 "" H 7700 4900 60  0000 C CNN
 F 3 "" H 7700 4900 60  0000 C CNN
-F 4 "#PWR050" H 7700 4900 50  0001 C CNN "OldReference"
 	1    7700 4900
 	1    0    0    -1
@@
 F 2 "conn-test:TEST-SMD-SMALL" H 8400 3750 50  0001 C CNN
 F 3 "" H 8400 3750 50  0000 C CNN
-F 4 "TP3" H 8400 3750 50  0001 C CNN "OldReference"
 	1    8400 3750
 	1    0    0    -1
@@
 F 2 "conn-test:TEST-SMD-SMALL" H 8700 3750 50  0001 C CNN
 F 3 "" H 8700 3750 50  0000 C CNN
-F 4 "TP4" H 8700 3750 50  0001 C CNN "OldReference"
 	1    8700 3750
 	1    0    0    -1
@@
 F 2 "" H 7900 3550 60  0000 C CNN
 F 3 "" H 7900 3550 60  0000 C CNN
-F 4 "#PWR051" H 7900 3550 50  0001 C CNN "OldReference"
 	1    7900 3550
 	1    0    0    -1
@@
 F 3 "" H 5990 3775 60  0000 C CNN
 F 4 "#CAP MLCC 100n ≥X7R 16V 10% [0603]" H 6800 4350 60  0001 C CNN "BOM"
-F 5 "C32" H 6000 3800 50  0001 C CNN "OldReference"
 	1    6000 3800
 	0    1    1    0
@@
 F 3 "" H 7890 3375 60  0000 C CNN
 F 4 "#CAP MLCC 100n ≥X7R 16V 10% [0603]" H 8700 3950 60  0001 C CNN "BOM"
-F 5 "C33" H 7900 3400 50  0001 C CNN "OldReference"
 	1    7900 3400
 	-1   0    0    1
@@
 F 4 "IRLML6402TRPBF" H 4250 3400 60  0001 C CNN "PN"
 F 5 "IRF" H 3850 3250 100 0001 C CNN "Manuf"
-F 6 "SEMI IRF IRLML6402" H 4650 3800 60  0001 C CNN "BOM"
-F 7 "Q20" H 3850 3250 50  0001 C CNN "OldReference"
+F 6 "PMOS IRF IRLML6402" H 4650 3800 60  0001 C CNN "BOM"
 	1    3850 3250
 	0    -1   -1   0
@@
 F 4 "" H 3350 3550 60  0001 C CNN "Manuf"
 F 5 "CAP MLCC 100n ≥X7R 16V 10% [0603]" H 4150 4100 60  0001 C CNN "BOM"
-F 6 "C63" H 3350 3550 50  0001 C CNN "OldReference"
 	1    3350 3550
 	0    1    1    0
@@
 F 4 "" H 4500 3550 60  0001 C CNN "Manuf"
 F 5 "CAP MLCC 10n ≥X5R 50V 10% [0603]" H 5300 4100 60  0001 C CNN "BOM"
-F 6 "C64" H 4500 3550 50  0001 C CNN "OldReference"
 	1    4500 3550
 	0    1    -1   0
@@
 F 2 "" H 3950 3900 60  0000 C CNN
 F 3 "" H 3950 3900 60  0000 C CNN
-F 4 "#PWR052" H 3950 3900 50  0001 C CNN "OldReference"
 	1    3950 3900
 	1    0    0    -1
@@
 F 2 "smd-semi:SOT-23" H 4200 2700 50  0001 C CNN
 F 3 "" H 4200 2700 60  0000 C CNN
-F 4 "SEMI GENERIC MMBD4148" H 4200 2700 60  0001 C CNN "BOM"
-F 5 "D8" H 4200 2700 50  0001 C CNN "OldReference"
+F 4 "DIODE MMBD4148" H 4200 2700 60  0001 C CNN "BOM"
 	1    4200 2700
 	-1   0    0    -1
@@
 F 2 "smd-semi:SOT-23" H 4400 2700 50  0001 C CNN
 F 3 "" H 4400 2700 60  0000 C CNN
-F 4 "SEMI GENERIC MMBD4148" H 4400 2700 60  0001 C CNN "BOM"
-F 5 "D9" H 4400 2700 50  0001 C CNN "OldReference"
+F 4 "DIODE MMBD4148" H 4400 2700 60  0001 C CNN "BOM"
 	1    4400 2700
 	1    0    0    -1
@@
 F 2 "" H 4300 2450 60  0000 C CNN
 F 3 "" H 4300 2450 60  0000 C CNN
-F 4 "#PWR053" H 4300 2450 50  0001 C CNN "OldReference"
 	1    4300 2450
 	1    0    0    -1
@@
 F 3 "" H 2250 4050 60  0000 C CNN
 F 4 "RES SMD 30 1% [0603]" H 3000 4550 60  0001 C CNN "BOM"
-F 5 "R7" H 2250 4000 50  0001 C CNN "OldReference"
 	1    2250 4000
 	0    1    1    0
@@
 F 3 "" H 2250 4150 60  0000 C CNN
 F 4 "RES SMD 30 1% [0603]" H 3000 4650 60  0001 C CNN "BOM"
-F 5 "R8" H 2250 4100 50  0001 C CNN "OldReference"
 	1    2250 4100
 	0    1    -1   0
@@
 F 4 "" H 3950 3750 60  0001 C CNN "Manuf"
 F 5 "RES SMD 1M 5% [0603]" H 4700 4300 60  0001 C CNN "BOM"
-F 6 "R16" H 3950 3750 50  0001 C CNN "OldReference"
 	1    3950 3750
 	1    0    0    -1
@@
 F 4 "" H 3550 3400 60  0001 C CNN "Manuf"
 F 5 "RES SMD 1M 5% [0603]" H 4300 3950 60  0001 C CNN "BOM"
-F 6 "R37" H 3550 3400 50  0001 C CNN "OldReference"
 	1    3550 3400
 	1    0    0    -1

Commit message: Add post-testing revision, todo notes
Other:
- note added: "TODO (REV 2):\n- Remove unnecessary U1, tidy routing"
Changed lines of the file:
@@
 Sheet 2 13
 Title "USB Communications"
-Date "2015-03-21"
-Rev ""
+Date "2015-03-31"
+Rev "1"
 Comp "WCP52"
 Comment1 "Gain/Phase Analyzer"
@@
 $EndComp
 $Comp
-L GND #PWR46
+L GND #PWR046
 U 1 1 54F70169
 P 3150 4900
-F 0 "#PWR46" H 3150 4900 30  0001 C CNN
+F 0 "#PWR046" H 3150 4900 30  0001 C CNN
 F 1 "GND" H 3150 4830 30  0001 C CNN
 F 2 "" H 3150 4900 60  0000 C CNN
@@
 $EndComp
 $Comp
-L GND #PWR49
+L GND #PWR047
 U 1 1 54F7543C
 P 5100 3600
-F 0 "#PWR49" H 5100 3600 30  0001 C CNN
+F 0 "#PWR047" H 5100 3600 30  0001 C CNN
 F 1 "GND" H 5100 3530 30  0001 C CNN
 F 2 "" H 5100 3600 60  0000 C CNN
@@
 $EndComp
 $Comp
-L GND #PWR50
+L GND #PWR048
 U 1 1 54F76B86
 P 5800 3800
-F 0 "#PWR50" H 5800 3800 30  0001 C CNN
+F 0 "#PWR048" H 5800 3800 30  0001 C CNN
 F 1 "GND" H 5800 3730 30  0001 C CNN
 F 2 "" H 5800 3800 60  0000 C CNN
@@
 $EndComp
 $Comp
-L GND #PWR51
+L GND #PWR049
 U 1 1 54F76CB4
 P 6300 4900
-F 0 "#PWR51" H 6300 4900 30  0001 C CNN
+F 0 "#PWR049" H 6300 4900 30  0001 C CNN
 F 1 "GND" H 6300 4830 30  0001 C CNN
 F 2 "" H 6300 4900 60  0000 C CNN
@@
 $EndComp
 $Comp
-L GND #PWR52
+L GND #PWR050
 U 1 1 54F76DBE
 P 7700 4900
-F 0 "#PWR52" H 7700 4900 30  0001 C CNN
+F 0 "#PWR050" H 7700 4900 30  0001 C CNN
 F 1 "GND" H 7700 4830 30  0001 C CNN
 F 2 "" H 7700 4900 60  0000 C CNN
@@
 USBPWR
 $Comp
-L GND #PWR53
+L GND #PWR051
 U 1 1 54F81F0B
 P 7900 3550
-F 0 "#PWR53" H 7900 3550 30  0001 C CNN
+F 0 "#PWR051" H 7900 3550 30  0001 C CNN
 F 1 "GND" H 7900 3480 30  0001 C CNN
 F 2 "" H 7900 3550 60  0000 C CNN
@@
 $EndComp
 $Comp
-L GND #PWR47
+L GND #PWR052
 U 1 1 54FE37FA
 P 3950 3900
-F 0 "#PWR47" H 3950 3900 30  0001 C CNN
+F 0 "#PWR052" H 3950 3900 30  0001 C CNN
 F 1 "GND" H 3950 3830 30  0001 C CNN
 F 2 "" H 3950 3900 60  0000 C CNN
@@
 $EndComp
 $Comp
-L +5 #PWR48
+L +5 #PWR053
 U 1 1 54FE450B
 P 4300 2450
-F 0 "#PWR48" H 4300 2500 30  0001 C CNN
+F 0 "#PWR053" H 4300 2500 30  0001 C CNN
 F 1 "+5" H 4300 2550 50  0000 C CNN
 F 2 "" H 4300 2450 60  0000 C CNN
@@
 USB pickoff to microcontroller\nThis is the intended normal mode of communcation, rather\nthan installing the above USB-UART interface device.
 $Comp
-L SIGPATH_SM #SYM44
+L SIGPATH_SM #SYM42
 U 1 1 550EDEC1
 P 8100 3800
-F 0 "#SYM44" H 8100 3800 60  0001 C CNN
+F 0 "#SYM42" H 8100 3800 60  0001 C CNN
 F 1 "SIGPATH_SM" H 8100 3800 60  0001 C CNN
 F 2 "" H 8100 3800 60  0000 C CNN
@@
 $EndComp
 $Comp
-L SIGPATH_SM #SYM45
+L SIGPATH_SM #SYM44
 U 1 1 550EDEF5
 P 8100 4000
-F 0 "#SYM45" H 8100 4000 60  0001 C CNN
+F 0 "#SYM44" H 8100 4000 60  0001 C CNN
 F 1 "SIGPATH_SM" H 8100 4000 60  0001 C CNN
 F 2 "" H 8100 4000 60  0000 C CNN
@@
 $EndComp
 $Comp
-L MSIGPATH_SM #SYM42
+L MSIGPATH_SM #SYM43
 U 1 1 550EDF24
 P 7950 3900
-F 0 "#SYM42" H 7950 3900 60  0001 C CNN
+F 0 "#SYM43" H 7950 3900 60  0001 C CNN
 F 1 "MSIGPATH_SM" H 7950 3900 60  0001 C CNN
 F 2 "" H 7950 3900 60  0000 C CNN
@@
 $EndComp
 $Comp
-L MSIGPATH_SM #SYM43
+L MSIGPATH_SM #SYM45
 U 1 1 550EDF58
 P 7950 4100
-F 0 "#SYM43" H 7950 4100 60  0001 C CNN
+F 0 "#SYM45" H 7950 4100 60  0001 C CNN
 F 1 "MSIGPATH_SM" H 7950 4100 60  0001 C CNN
 F 2 "" H 7950 4100 60  0000 C CNN
@@
 	1    0    0    -1
 $EndComp
+Text Notes 650  7800 0    50   ~ 0
+TODO (REV 2):\n- Remove unnecessary U1, tidy routing
 $EndSCHEMATC
