File: wcp52/InputFrontend.sch (KiCad schematic (older format))
At the start: 6 parts

Commit message: Prepare to fab
Changed lines of the file:
@@
 	9200 1300 2100 1300
 Wire Wire Line
-	8300 3300 8400 3300
-Wire Wire Line
-	8400 3300 9600 3300
+	8300 3300 9600 3300
 Wire Wire Line
 	8400 3300 8400 3400

Commit message: BOM line fixes
Parts:
- C53, C54, C55, C56, R56: Manuf Value -> (none)
- MP5: Description (none) -> RF SHIELD TWO-PIECE
Changed lines of the file:
@@
 EESchema Schematic File Version 2
+LIBS:Altera
+LIBS:AnalogDevices
+LIBS:Atmel
+LIBS:conn-2mm
+LIBS:conn-100mil
+LIBS:conn-cui
+LIBS:conn-fci
+LIBS:conn-linx
+LIBS:conn-molex
+LIBS:conn-tagconnect
+LIBS:conn-test
+LIBS:DiodesInc
+LIBS:display
+LIBS:_electromech
+LIBS:Fairchild
+LIBS:FTDI
+LIBS:Intersil
+LIBS:Lattice
+LIBS:_linear
+LIBS:LinearTech
+LIBS:Littelfuse
+LIBS:logic-4000
+LIBS:logic-7400
+LIBS:MACOM
+LIBS:maxim
+LIBS:mechanical
+LIBS:Microchip
+LIBS:Micron
+LIBS:NXP
+LIBS:onsemi
+LIBS:passive
+LIBS:pasv-BiTech
+LIBS:pasv-Bourns
+LIBS:pasv-cap
+LIBS:pasv-ind
+LIBS:pasv-res
+LIBS:pcb
+LIBS:power
+LIBS:_semi
+LIBS:semi-diode-1N
+LIBS:semi-diode-BA
+LIBS:semi-diode-MCC
+LIBS:semi-diode-MMB
+LIBS:semi-diode-NXP
+LIBS:semi-diode-OnSemi
+LIBS:semi-diode-Vishay
+LIBS:semi-opto-misc
+LIBS:semi-thyristor-2N
+LIBS:semi-trans-2N
+LIBS:semi-trans-AO
+LIBS:semi-trans-BC
+LIBS:semi-trans-DiodesInc
+LIBS:semi-trans-Fairchild
+LIBS:semi-trans-Infineon
+LIBS:semi-trans-IntRect
+LIBS:semi-trans-IXYS
+LIBS:semi-trans-misc
+LIBS:semi-trans-MMB
+LIBS:semi-trans-MPS
+LIBS:semi-trans-NXP
+LIBS:semi-trans-PZT
+LIBS:semi-trans-TI
+LIBS:semi-trans-TIP
+LIBS:semi-trans-Toshiba
+LIBS:silabs
+LIBS:skyworks
+LIBS:ST
+LIBS:st_ic
+LIBS:st_semi
+LIBS:supertex
+LIBS:symbol
+LIBS:TexasInstruments
+LIBS:vishay_semi
+LIBS:Xilinx
+LIBS:pasv-xtal
+LIBS:conn-te
 LIBS:wcp52-cache
 EELAYER 25 0
@@
 F 5 "Laird" H 2400 4300 60  0001 C CNN "Manuf"
 F 6 "DIST DIGIKEY 903-1052-1-ND; DIST DIGIKEY 903-1015-ND" H 2400 4300 60  0001 C CNN "BOM"
-F 7 "MP1" H 2400 4300 50  0001 C CNN "OldReference"
+F 7 "RF SHIELD TWO-PIECE" H 2400 4300 60  0001 C CNN "Description"
+F 8 "MP1" H 2400 4300 50  0001 C CNN "OldReference"
 	1    2400 4300
 	1    0    0    -1
@@
 F 2 "IPC7351-Nominal:CAPC3216X70" H 2400 1700 50  0001 C CNN
 F 3 "" H 2390 1675 60  0000 C CNN
-F 4 "Value" H 2400 1700 60  0001 C CNN "Manuf"
+F 4 "" H 2400 1700 60  0001 C CNN "Manuf"
 F 5 "CAP MLCC 47u ≥X5R 10V 20% [1206]" H 3200 2250 60  0001 C CNN "BOM"
 F 6 "C52" H 2400 1700 50  0001 C CNN "OldReference"
@@
 F 2 "IPC7351-Nominal:CAPC2012X70" H 3300 1700 50  0001 C CNN
 F 3 "" H 3290 1675 60  0000 C CNN
-F 4 "Value" H 3300 1700 60  0001 C CNN "Manuf"
+F 4 "" H 3300 1700 60  0001 C CNN "Manuf"
 F 5 "CAP MLCC 220n ≥X5R 16V 10% [0805]" H 4100 2250 60  0001 C CNN "BOM"
 F 6 "C65" H 3300 1700 50  0001 C CNN "OldReference"
@@
 F 2 "IPC7351-Nominal:CAPC1608X55" H 2850 1700 50  0001 C CNN
 F 3 "" H 2840 1675 60  0000 C CNN
-F 4 "Value" H 2850 1700 60  0001 C CNN "Manuf"
+F 4 "" H 2850 1700 60  0001 C CNN "Manuf"
 F 5 "CAP MLCC 1n C0G 50V 10% [0603]" H 3650 2250 60  0001 C CNN "BOM"
 F 6 "C53" H 2850 1700 50  0001 C CNN "OldReference"
@@
 F 2 "IPC7351-Nominal:CAPC1608X55" H 8400 3500 50  0001 C CNN
 F 3 "" H 8390 3475 60  0000 C CNN
-F 4 "Value" H 8400 3500 60  0001 C CNN "Manuf"
+F 4 "" H 8400 3500 60  0001 C CNN "Manuf"
 F 5 "CAP MLCC 10n ≥X5R 50V 10% [0603]" H 9200 4050 60  0001 C CNN "BOM"
 F 6 "C69" H 8400 3500 50  0001 C CNN "OldReference"
@@
 F 2 "IPC7351-Nominal:RESC1608X50" H 8200 3300 50  0001 C CNN
 F 3 "" H 8200 3350 60  0000 C CNN
-F 4 "Value" H 8200 3300 60  0001 C CNN "Manuf"
+F 4 "" H 8200 3300 60  0001 C CNN "Manuf"
 F 5 "RES SMD 49.9 1% [0603]" H 8950 3850 60  0001 C CNN "BOM"
 F 6 "R52" H 8200 3300 50  0001 C CNN "OldReference"

Commit message: BOM corrections/combinations, etc
Add configuration for bomtool
Remove old schematic file no longer used
Parts:
- C55: value 220n -> 100n; BOM CAP MLCC 220n ≥X5R 16V 10% [0805] -> CAP MLCC 100n ≥X7R 20V 10% [0805]
Changed lines of the file:
@@
 P 3300 1700
 F 0 "C55" H 3550 1750 50  0000 C CNN
-F 1 "220n" H 3550 1650 50  0000 C CNN
+F 1 "100n" H 3550 1650 50  0000 C CNN
 F 2 "IPC7351-Nominal:CAPC2012X70" H 3300 1700 50  0001 C CNN
 F 3 "" H 3290 1675 60  0000 C CNN
-F 4 "" H 3300 1700 60  0001 C CNN "Manuf"
-F 5 "CAP MLCC 220n ≥X5R 16V 10% [0805]" H 4100 2250 60  0001 C CNN "BOM"
-F 6 "C65" H 3300 1700 50  0001 C CNN "OldReference"
+F 4 "CAP MLCC 100n ≥X7R 20V 10% [0805]" H 4100 2250 60  0001 C CNN "BOM"
+F 5 "C65" H 3300 1700 50  0001 C CNN "OldReference"
 	1    3300 1700
 	1    0    0    -1

Commit message: Schematic updates for documentation
Changed lines of the file:
@@
 $EndComp
 $Comp
-L GND #PWR0163
+L GND #PWR165
 U 1 1 54F2F4A0
 P 2400 4400
-F 0 "#PWR0163" H 2400 4400 30  0001 C CNN
+F 0 "#PWR165" H 2400 4400 30  0001 C CNN
 F 1 "GND" H 2400 4330 30  0001 C CNN
 F 2 "" H 2400 4400 60  0000 C CNN
@@
 	9200 1300 2100 1300
 Wire Wire Line
-	8300 3300 9600 3300
+	8300 3300 10100 3300
 Wire Wire Line
 	8400 3300 8400 3400
 Connection ~ 8400 3300
-Text HLabel 9600 3300 2    60   Output ~ 0
+Text HLabel 10100 3300 2    60   Output ~ 0
 OUT
 $Comp
-L GND #PWR0164
+L GND #PWR170
 U 1 1 54F3075A
 P 8400 3700
-F 0 "#PWR0164" H 8400 3700 30  0001 C CNN
+F 0 "#PWR170" H 8400 3700 30  0001 C CNN
 F 1 "GND" H 8400 3630 30  0001 C CNN
 F 2 "" H 8400 3700 60  0000 C CNN
@@
 	8400 3600 8400 3700
 Wire Wire Line
-	2800 3300 1800 3300
-Wire Wire Line
-	2800 3700 1800 3700
-Text HLabel 1800 3300 0    60   Input ~ 0
+	2800 3300 1400 3300
+Wire Wire Line
+	2800 3700 1400 3700
+Text HLabel 1400 3300 0    60   Input ~ 0
 IN1
-Text HLabel 1800 3700 0    60   Input ~ 0
+Text HLabel 1400 3700 0    60   Input ~ 0
 IN2
 Wire Wire Line
@@
 $EndComp
 $Comp
-L -5 #PWR0165
+L -5 #PWR163
 U 1 1 54F26D5C
 P 2400 1550
-F 0 "#PWR0165" H 2400 1500 30  0001 C CNN
+F 0 "#PWR163" H 2400 1500 30  0001 C CNN
 F 1 "-5" H 2400 1450 50  0000 C CNN
 F 2 "" H 2400 1550 60  0000 C CNN
@@
 	2400 1550 2400 1600
 $Comp
-L GND #PWR0166
+L GND #PWR164
 U 1 1 54F26E11
 P 2400 1850
-F 0 "#PWR0166" H 2400 1850 30  0001 C CNN
+F 0 "#PWR164" H 2400 1850 30  0001 C CNN
 F 1 "GND" H 2400 1780 30  0001 C CNN
 F 2 "" H 2400 1850 60  0000 C CNN
@@
 	2850 1550 2850 1600
 $Comp
-L GND #PWR0167
+L GND #PWR167
 U 1 1 54F288BE
 P 2850 1850
-F 0 "#PWR0167" H 2850 1850 30  0001 C CNN
+F 0 "#PWR167" H 2850 1850 30  0001 C CNN
 F 1 "GND" H 2850 1780 30  0001 C CNN
 F 2 "" H 2850 1850 60  0000 C CNN
@@
 	2850 1850 2850 1800
 $Comp
-L +5 #PWR0168
+L +5 #PWR166
 U 1 1 54F2892E
 P 2850 1550
-F 0 "#PWR0168" H 2850 1600 30  0001 C CNN
+F 0 "#PWR166" H 2850 1600 30  0001 C CNN
 F 1 "+5" H 2850 1650 50  0000 C CNN
 F 2 "" H 2850 1550 60  0000 C CNN
@@
 	3300 1550 3300 1600
 $Comp
-L GND #PWR0169
+L GND #PWR169
 U 1 1 54F29C50
 P 3300 1850
-F 0 "#PWR0169" H 3300 1850 30  0001 C CNN
+F 0 "#PWR169" H 3300 1850 30  0001 C CNN
 F 1 "GND" H 3300 1780 30  0001 C CNN
 F 2 "" H 3300 1850 60  0000 C CNN
@@
 	3300 1850 3300 1800
 $Comp
-L +5 #PWR0170
+L +5 #PWR168
 U 1 1 54F29C57
 P 3300 1550
-F 0 "#PWR0170" H 3300 1600 30  0001 C CNN
+F 0 "#PWR168" H 3300 1600 30  0001 C CNN
 F 1 "+5" H 3300 1650 50  0000 C CNN
 F 2 "" H 3300 1550 60  0000 C CNN
@@
 Wire Notes Line
 	9200 4300 2100 4300
+$Comp
+L SINE-ACCURATE #SYM68
+U 1 1 550F3E55
+P 1550 3200
+F 0 "#SYM68" H 1550 3200 60  0001 C CNN
+F 1 "SINE-ACCURATE" H 1550 3200 60  0001 C CNN
+F 2 "" H 1550 3200 60  0000 C CNN
+F 3 "" H 1550 3200 60  0000 C CNN
+	1    1550 3200
+	1    0    0    -1
+$EndComp
+$Comp
+L SINE-ACCURATE #SYM69
+U 1 1 550F3E9A
+P 1550 3600
+F 0 "#SYM69" H 1550 3600 60  0001 C CNN
+F 1 "SINE-ACCURATE" H 1550 3600 60  0001 C CNN
+F 2 "" H 1550 3600 60  0000 C CNN
+F 3 "" H 1550 3600 60  0000 C CNN
+	1    1550 3600
+	1    0    0    -1
+$EndComp
 $EndSCHEMATC

Commit message: More doc fixes
Changed lines of the file:
@@
 	1    0    0    -1
 $EndComp
-Wire Wire Line
-	2400 4400 2400 4350
 $Sheet
 S 2800 3100 1000 800
@@
 F3 "IN" I L 6900 3300 60
 $EndSheet
-Wire Notes Line
-	2100 1300 2100 4300
-Wire Notes Line
-	9200 1300 2100 1300
-Wire Wire Line
-	8300 3300 10100 3300
-Wire Wire Line
-	8400 3300 8400 3400
-Connection ~ 8400 3300
 Text HLabel 10100 3300 2    60   Output ~ 0
 OUT
@@
 	1    0    0    -1
 $EndComp
-Wire Wire Line
-	8400 3600 8400 3700
-Wire Wire Line
-	2800 3300 1400 3300
-Wire Wire Line
-	2800 3700 1400 3700
 Text HLabel 1400 3300 0    60   Input ~ 0
 IN1
 Text HLabel 1400 3700 0    60   Input ~ 0
 IN2
-Wire Wire Line
-	4200 3300 3800 3300
-Wire Wire Line
-	3800 3700 4200 3700
 Text HLabel 1800 5200 0    60   Input ~ 0
 INPUTSEL
-Wire Wire Line
-	1800 5200 4200 5200
 Text HLabel 1800 5600 0    60   Input ~ 0
 PHASEREF
-Wire Wire Line
-	1800 5600 5500 5600
-Wire Wire Line
-	5500 3300 5100 3300
-Wire Wire Line
-	6500 3300 6900 3300
-Wire Wire Line
-	7900 3300 8100 3300
 $Comp
 L C-1206 C53
@@
 	-1   0    0    1
 $EndComp
-Wire Wire Line
-	2400 1550 2400 1600
 $Comp
 L GND #PWR164
@@
 	1    0    0    -1
 $EndComp
-Wire Wire Line
-	2400 1850 2400 1800
-Wire Wire Line
-	2850 1550 2850 1600
 $Comp
 L GND #PWR167
@@
 	1    0    0    -1
 $EndComp
-Wire Wire Line
-	2850 1850 2850 1800
 $Comp
 L +5 #PWR166
@@
 	1    0    0    -1
 $EndComp
-Wire Wire Line
-	3300 1550 3300 1600
 $Comp
 L GND #PWR169
@@
 	1    0    0    -1
 $EndComp
-Wire Wire Line
-	3300 1850 3300 1800
 $Comp
 L +5 #PWR168
@@
 	0    1    1    0
 $EndComp
+$Comp
+L SINE-ACCURATE #SYM72
+U 1 1 550F3E55
+P 1550 3200
+F 0 "#SYM72" H 1550 3200 60  0001 C CNN
+F 1 "SINE-ACCURATE" H 1550 3200 60  0001 C CNN
+F 2 "" H 1550 3200 60  0000 C CNN
+F 3 "" H 1550 3200 60  0000 C CNN
+	1    1550 3200
+	1    0    0    -1
+$EndComp
+$Comp
+L SINE-ACCURATE #SYM73
+U 1 1 550F3E9A
+P 1550 3600
+F 0 "#SYM73" H 1550 3600 60  0001 C CNN
+F 1 "SINE-ACCURATE" H 1550 3600 60  0001 C CNN
+F 2 "" H 1550 3600 60  0000 C CNN
+F 3 "" H 1550 3600 60  0000 C CNN
+	1    1550 3600
+	1    0    0    -1
+$EndComp
+Wire Wire Line
+	2400 4400 2400 4350
+Wire Notes Line
+	2100 1300 2100 4300
+Wire Notes Line
+	9200 1300 2100 1300
+Wire Wire Line
+	8300 3300 10100 3300
+Wire Wire Line
+	8400 3300 8400 3400
+Connection ~ 8400 3300
+Wire Wire Line
+	8400 3600 8400 3700
+Wire Wire Line
+	2800 3300 1400 3300
+Wire Wire Line
+	2800 3700 1400 3700
+Wire Wire Line
+	4200 3300 3800 3300
+Wire Wire Line
+	3800 3700 4200 3700
+Wire Wire Line
+	1800 5200 4200 5200
+Wire Wire Line
+	1800 5600 5500 5600
+Wire Wire Line
+	5500 3300 5100 3300
+Wire Wire Line
+	6500 3300 6900 3300
+Wire Wire Line
+	7900 3300 8100 3300
+Wire Wire Line
+	2400 1550 2400 1600
+Wire Wire Line
+	2400 1850 2400 1800
+Wire Wire Line
+	2850 1550 2850 1600
+Wire Wire Line
+	2850 1850 2850 1800
+Wire Wire Line
+	3300 1550 3300 1600
+Wire Wire Line
+	3300 1850 3300 1800
 Wire Notes Line
 	9200 1300 9200 4300
 Wire Notes Line
 	9200 4300 2100 4300
-$Comp
-L SINE-ACCURATE #SYM68
-U 1 1 550F3E55
-P 1550 3200
-F 0 "#SYM68" H 1550 3200 60  0001 C CNN
-F 1 "SINE-ACCURATE" H 1550 3200 60  0001 C CNN
-F 2 "" H 1550 3200 60  0000 C CNN
-F 3 "" H 1550 3200 60  0000 C CNN
-	1    1550 3200
-	1    0    0    -1
-$EndComp
-$Comp
-L SINE-ACCURATE #SYM69
-U 1 1 550F3E9A
-P 1550 3600
-F 0 "#SYM69" H 1550 3600 60  0001 C CNN
-F 1 "SINE-ACCURATE" H 1550 3600 60  0001 C CNN
-F 2 "" H 1550 3600 60  0000 C CNN
-F 3 "" H 1550 3600 60  0000 C CNN
-	1    1550 3600
-	1    0    0    -1
-$EndComp
+Wire Wire Line
+	1400 3300 1425 3325
+Wire Wire Line
+	1425 3325 2775 3325
+Wire Wire Line
+	2775 3325 2800 3300
+Wire Wire Line
+	1400 3700 1425 3725
+Wire Wire Line
+	1425 3725 2775 3725
+Wire Wire Line
+	2775 3725 2800 3700
+Wire Wire Line
+	3800 3300 3825 3325
+Wire Wire Line
+	3825 3325 4175 3325
+Wire Wire Line
+	4175 3325 4200 3300
+Wire Wire Line
+	3800 3700 3825 3725
+Wire Wire Line
+	3825 3725 4175 3725
+Wire Wire Line
+	4175 3725 4200 3700
+Wire Wire Line
+	5100 3300 5125 3325
+Wire Wire Line
+	5125 3325 5475 3325
+Wire Wire Line
+	5475 3325 5500 3300
+Wire Wire Line
+	6500 3300 6525 3325
+Wire Wire Line
+	6525 3325 6875 3325
+Wire Wire Line
+	6875 3325 6900 3300
+Wire Wire Line
+	7900 3300 7925 3325
+Wire Wire Line
+	7925 3325 8075 3325
+Wire Wire Line
+	8075 3325 8100 3300
+Wire Wire Line
+	8300 3300 8325 3325
+Wire Wire Line
+	8325 3325 10075 3325
+Wire Wire Line
+	10075 3325 10100 3300
 $EndSCHEMATC

Commit message: Nicer BOM lines
Parts:
- C53: OldReference C52 -> (none)
- C54: OldReference C53 -> (none)
- C55: OldReference C65 -> (none)
- C56: OldReference C69 -> (none)
- MP5: OldReference MP1 -> (none)
- R56: OldReference R52 -> (none)
Changed lines of the file:
@@
 F 6 "DIST DIGIKEY 903-1052-1-ND; DIST DIGIKEY 903-1015-ND" H 2400 4300 60  0001 C CNN "BOM"
 F 7 "RF SHIELD TWO-PIECE" H 2400 4300 60  0001 C CNN "Description"
-F 8 "MP1" H 2400 4300 50  0001 C CNN "OldReference"
 	1    2400 4300
 	1    0    0    -1
@@
 F 2 "" H 2400 4400 60  0000 C CNN
 F 3 "" H 2400 4400 60  0000 C CNN
-F 4 "#PWR0163" H 2400 4400 50  0001 C CNN "OldReference"
 	1    2400 4400
 	1    0    0    -1
@@
 F 2 "" H 8400 3700 60  0000 C CNN
 F 3 "" H 8400 3700 60  0000 C CNN
-F 4 "#PWR0164" H 8400 3700 50  0001 C CNN "OldReference"
 	1    8400 3700
 	1    0    0    -1
@@
 F 4 "" H 2400 1700 60  0001 C CNN "Manuf"
 F 5 "CAP MLCC 47u ≥X5R 10V 20% [1206]" H 3200 2250 60  0001 C CNN "BOM"
-F 6 "C52" H 2400 1700 50  0001 C CNN "OldReference"
 	1    2400 1700
 	1    0    0    -1
@@
 F 2 "" H 2400 1550 60  0000 C CNN
 F 3 "" H 2400 1550 60  0000 C CNN
-F 4 "#PWR0165" H 2400 1550 50  0001 C CNN "OldReference"
 	1    2400 1550
 	-1   0    0    1
@@
 F 2 "" H 2400 1850 60  0000 C CNN
 F 3 "" H 2400 1850 60  0000 C CNN
-F 4 "#PWR0166" H 2400 1850 50  0001 C CNN "OldReference"
 	1    2400 1850
 	1    0    0    -1
@@
 F 2 "" H 2850 1850 60  0000 C CNN
 F 3 "" H 2850 1850 60  0000 C CNN
-F 4 "#PWR0167" H 2850 1850 50  0001 C CNN "OldReference"
 	1    2850 1850
 	1    0    0    -1
@@
 F 2 "" H 2850 1550 60  0000 C CNN
 F 3 "" H 2850 1550 60  0000 C CNN
-F 4 "#PWR0168" H 2850 1550 50  0001 C CNN "OldReference"
 	1    2850 1550
 	1    0    0    -1
@@
 F 3 "" H 3290 1675 60  0000 C CNN
 F 4 "CAP MLCC 100n ≥X7R 20V 10% [0805]" H 4100 2250 60  0001 C CNN "BOM"
-F 5 "C65" H 3300 1700 50  0001 C CNN "OldReference"
 	1    3300 1700
 	1    0    0    -1
@@
 F 2 "" H 3300 1850 60  0000 C CNN
 F 3 "" H 3300 1850 60  0000 C CNN
-F 4 "#PWR0169" H 3300 1850 50  0001 C CNN "OldReference"
 	1    3300 1850
 	1    0    0    -1
@@
 F 2 "" H 3300 1550 60  0000 C CNN
 F 3 "" H 3300 1550 60  0000 C CNN
-F 4 "#PWR0170" H 3300 1550 50  0001 C CNN "OldReference"
 	1    3300 1550
 	1    0    0    -1
@@
 F 4 "" H 2850 1700 60  0001 C CNN "Manuf"
 F 5 "CAP MLCC 1n C0G 50V 10% [0603]" H 3650 2250 60  0001 C CNN "BOM"
-F 6 "C53" H 2850 1700 50  0001 C CNN "OldReference"
 	1    2850 1700
 	1    0    0    -1
@@
 F 4 "" H 8400 3500 60  0001 C CNN "Manuf"
 F 5 "CAP MLCC 10n ≥X5R 50V 10% [0603]" H 9200 4050 60  0001 C CNN "BOM"
-F 6 "C69" H 8400 3500 50  0001 C CNN "OldReference"
 	1    8400 3500
 	1    0    0    -1
@@
 F 4 "" H 8200 3300 60  0001 C CNN "Manuf"
 F 5 "RES SMD 49.9 1% [0603]" H 8950 3850 60  0001 C CNN "BOM"
-F 6 "R52" H 8200 3300 50  0001 C CNN "OldReference"
 	1    8200 3300
 	0    1    1    0
