File: wcp52/OutputAmp.sch (KiCad schematic (older format))
At the start: 33 parts, among them Q2 MMBT3906, Q3 2N7002, Q4 2N7002, U5 AD8000YRDZ, U6 THS3001IDGN, U7 MAADSS0008

Commit message: BOM line fixes
Parts:
- C32, C33, C34, C35, C36, C37, C38, C39, C40, C41, C42, Q2, Q3, Q4, R40, R42, R43, R44, R45, R46, R47, R48, R49, R50, R51, R52, R53, R54, R55, U5, U6, U7: Manuf Value -> (none)
- R41: Description (none) -> RESPACK SMD 10k 5% [4x0603]
- U5: BOM DIST DIGIKEY AD8000YRDZ-ND -> IC ADI AD8000YRDZ; Manuf Value -> (none)
- U6: BOM DIST DIGIKEY 296-12006-1-ND -> IC TI THS3001IDGN; Manuf Value -> (none)

Commit message: BOM corrections/combinations, etc
Add configuration for bomtool
Remove old schematic file no longer used
Parts:
- Q2: BOM #DIST DIGIKEY MMBT3906LT1GOSCT-ND -> SEMI GENERIC MMBT3906
- Q3, Q4: BOM #DIST DIGIKEY 568-5818-1-ND -> SEMI GENERIC 2N7002
- U5: BOM DIST DIGIKEY AD8000YRDZ-ND -> (none)
- U6: BOM DIST DIGIKEY 296-12006-1-ND -> (none)
Changed lines of the file:
@@
 F 2 "IPC7351-Nominal:SOIC127P600X175-9" H 950 7250 50  0001 C CNN
 F 3 "" H 800 7250 60  0000 C CNN
-F 4 "" H 950 7250 60  0001 C CNN "Manuf"
-F 5 "DIST DIGIKEY AD8000YRDZ-ND" H 1450 8400 60  0001 C CNN "BOM"
-F 6 "U6" H 950 7250 50  0001 C CNN "OldReference"
+F 4 "U6" H 950 7250 50  0001 C CNN "OldReference"
 	2    950  7250
 	1    0    0    -1
@@
 F 2 "IPC7351-Nominal:SOP65P490X110-9A" H 2600 6950 50  0001 C CNN
 F 3 "" H 2400 6950 60  0000 C CNN
-F 4 "" H 2600 6950 60  0001 C CNN "Manuf"
-F 5 "DIST DIGIKEY 296-12006-1-ND" H 3100 7800 60  0001 C CNN "BOM"
-F 6 "U7" H 2600 6950 50  0001 C CNN "OldReference"
+F 4 "U7" H 2600 6950 50  0001 C CNN "OldReference"
 	2    2600 6950
 	-1   0    0    -1
@@
 F 2 "smd-semi:SOT-23" H 1850 5000 50  0001 C CNN
 F 3 "" H 1850 5000 60  0000 C CNN
-F 4 "" H 1850 5000 60  0001 C CNN "Manuf"
-F 5 "#DIST DIGIKEY 568-5818-1-ND" H 2600 5550 60  0001 C CNN "BOM"
-F 6 "Q5" H 1850 5000 50  0001 C CNN "OldReference"
+F 4 "SEMI GENERIC 2N7002" H 2600 5550 60  0001 C CNN "BOM"
+F 5 "Q5" H 1850 5000 50  0001 C CNN "OldReference"
 	1    1850 5000
 	1    0    0    -1
@@
 F 2 "smd-semi:SOT-23" H 2650 5000 50  0001 C CNN
 F 3 "" H 2650 5000 60  0000 C CNN
-F 4 "" H 2650 5000 60  0001 C CNN "Manuf"
-F 5 "#DIST DIGIKEY 568-5818-1-ND" H 3400 5550 60  0001 C CNN "BOM"
-F 6 "Q6" H 2650 5000 50  0001 C CNN "OldReference"
+F 4 "SEMI GENERIC 2N7002" H 3400 5550 60  0001 C CNN "BOM"
+F 5 "Q6" H 2650 5000 50  0001 C CNN "OldReference"
 	1    2650 5000
 	1    0    0    -1
@@
 F 2 "smd-semi:SOT-23" H 1450 4800 50  0001 C CNN
 F 3 "" H 1450 4800 60  0000 C CNN
-F 4 "" H 1450 4800 60  0001 C CNN "Manuf"
-F 5 "#DIST DIGIKEY MMBT3906LT1GOSCT-ND" H 2250 5350 60  0001 C CNN "BOM"
-F 6 "Q4" H 1450 4800 50  0001 C CNN "OldReference"
+F 4 "SEMI GENERIC MMBT3906" H 2250 5350 60  0001 C CNN "BOM"
+F 5 "Q4" H 1450 4800 50  0001 C CNN "OldReference"
 	1    1450 4800
 	1    0    0    -1

Commit message: Schematic/doc work
Changed lines of the file:
@@
 Sheet 4 13
 Title "Output Amplifier"
-Date "2015-03-13"
+Date "2015-03-21"
 Rev ""
 Comp "WCP52"
@@
 Comment2 ""
 Comment3 ""
-Comment4 "Eng: Chris Pavlina"
+Comment4 ""
 $EndDescr
 Text HLabel 1200 2800 0    60   Input ~ 0
@@
 U 1 1 54F2A330
 P 1850 5000
-F 0 "Q3" H 2100 5050 50  0000 C CNN
-F 1 "2N7002" H 2100 4950 50  0000 C CNN
+F 0 "Q3" H 1800 5150 50  0000 C CNN
+F 1 "2N7002" H 2100 4950 50  0001 C CNN
 F 2 "smd-semi:SOT-23" H 1850 5000 50  0001 C CNN
 F 3 "" H 1850 5000 60  0000 C CNN
@@
 U 1 1 54F2A556
 P 2650 5000
-F 0 "Q4" H 2900 5050 50  0000 C CNN
-F 1 "2N7002" H 2900 4950 50  0000 C CNN
+F 0 "Q4" H 2600 5150 50  0000 C CNN
+F 1 "2N7002" H 2900 4950 50  0001 C CNN
 F 2 "smd-semi:SOT-23" H 2650 5000 50  0001 C CNN
 F 3 "" H 2650 5000 60  0000 C CNN
@@
 U 1 1 54F2AD1B
 P 1450 4800
-F 0 "Q2" H 1250 4700 50  0000 C CNN
-F 1 "MMBT3906" H 1250 4600 50  0000 C CNN
+F 0 "Q2" H 1350 4950 50  0000 C CNN
+F 1 "MMBT3906" H 1250 4600 50  0001 C CNN
 F 2 "smd-semi:SOT-23" H 1450 4800 50  0001 C CNN
 F 3 "" H 1450 4800 60  0000 C CNN

Commit message: Schematic updates for documentation
Changed lines of the file:
@@
 $EndSheet
 $Comp
-L FILTER-LPF #SYM5
+L FILTER-LPF #SYM66
 U 1 1 54F227F4
 P 4700 2800
-F 0 "#SYM5" H 4700 2800 60  0001 C CNN
+F 0 "#SYM66" H 4700 2800 60  0001 C CNN
 F 1 "FILTER-LPF" H 4700 2800 60  0001 C CNN
 F 2 "" H 4700 2800 60  0000 C CNN
@@
 Connection ~ 5500 2400
 $Comp
-L GND #PWR0127
+L GND #PWR154
 U 1 1 54F23A9C
 P 5000 2400
-F 0 "#PWR0127" H 5000 2400 30  0001 C CNN
+F 0 "#PWR154" H 5000 2400 30  0001 C CNN
 F 1 "GND" H 5000 2330 30  0001 C CNN
 F 2 "" H 5000 2400 60  0000 C CNN
@@
 Connection ~ 5500 2800
 $Comp
-L GND #PWR0128
+L GND #PWR155
 U 1 1 54F23C44
 P 5500 3300
-F 0 "#PWR0128" H 5500 3300 30  0001 C CNN
+F 0 "#PWR155" H 5500 3300 30  0001 C CNN
 F 1 "GND" H 5500 3230 30  0001 C CNN
 F 2 "" H 5500 3300 60  0000 C CNN
@@
 	7600 2800 7600 2900
 $Comp
-L GND #PWR0129
+L GND #PWR156
 U 1 1 54F247C7
 P 7600 3600
-F 0 "#PWR0129" H 7600 3600 30  0001 C CNN
+F 0 "#PWR156" H 7600 3600 30  0001 C CNN
 F 1 "GND" H 7600 3530 30  0001 C CNN
 F 2 "" H 7600 3600 60  0000 C CNN
@@
 $EndComp
 $Comp
-L +5 #PWR0130
+L +5 #PWR128
 U 1 1 54F25A6C
 P 1000 6700
-F 0 "#PWR0130" H 1000 6750 30  0001 C CNN
+F 0 "#PWR128" H 1000 6750 30  0001 C CNN
 F 1 "+5" H 1000 6800 50  0000 C CNN
 F 2 "" H 1000 6700 60  0000 C CNN
@@
 Connection ~ 1000 6750
 $Comp
-L -5 #PWR0131
+L -5 #PWR129
 U 1 1 54F25B88
 P 1000 7800
-F 0 "#PWR0131" H 1000 7750 30  0001 C CNN
+F 0 "#PWR129" H 1000 7750 30  0001 C CNN
 F 1 "-5" H 1000 7700 50  0000 C CNN
 F 2 "" H 1000 7800 60  0000 C CNN
@@
 	1000 7800 1000 7700
 $Comp
-L GND #PWR0132
+L GND #PWR127
 U 1 1 54F25C12
 P 900 7750
-F 0 "#PWR0132" H 900 7750 30  0001 C CNN
+F 0 "#PWR127" H 900 7750 30  0001 C CNN
 F 1 "GND" H 900 7680 30  0001 C CNN
 F 2 "" H 900 7750 60  0000 C CNN
@@
 	900  7750 900  7700
 $Comp
-L +5 #PWR0133
+L +5 #PWR131
 U 1 1 54F2615E
 P 1400 6850
-F 0 "#PWR0133" H 1400 6900 30  0001 C CNN
+F 0 "#PWR131" H 1400 6900 30  0001 C CNN
 F 1 "+5" H 1400 6950 50  0000 C CNN
 F 2 "" H 1400 6850 60  0000 C CNN
@@
 	1900 7150 1900 7350
 $Comp
-L GND #PWR0134
+L GND #PWR141
 U 1 1 54F261AA
 P 2000 7250
-F 0 "#PWR0134" H 2000 7250 30  0001 C CNN
+F 0 "#PWR141" H 2000 7250 30  0001 C CNN
 F 1 "GND" H 2000 7180 30  0001 C CNN
 F 2 "" H 2000 7250 60  0000 C CNN
@@
 Connection ~ 1900 7250
 $Comp
-L +5 #PWR0135
+L +5 #PWR139
 U 1 1 54F261B2
 P 1900 6850
-F 0 "#PWR0135" H 1900 6900 30  0001 C CNN
+F 0 "#PWR139" H 1900 6900 30  0001 C CNN
 F 1 "+5" H 1900 6950 50  0000 C CNN
 F 2 "" H 1900 6850 60  0000 C CNN
@@
 	1900 6850 1900 6950
 $Comp
-L -5 #PWR0136
+L -5 #PWR140
 U 1 1 54F261B9
 P 1900 7650
-F 0 "#PWR0136" H 1900 7600 30  0001 C CNN
+F 0 "#PWR140" H 1900 7600 30  0001 C CNN
 F 1 "-5" H 1900 7550 50  0000 C CNN
 F 2 "" H 1900 7650 60  0000 C CNN
@@
 	1900 7650 1900 7550
 $Comp
-L GND #PWR0137
+L GND #PWR135
 U 1 1 54F26652
 P 1500 7250
-F 0 "#PWR0137" H 1500 7250 30  0001 C CNN
+F 0 "#PWR135" H 1500 7250 30  0001 C CNN
 F 1 "GND" H 1500 7180 30  0001 C CNN
 F 2 "" H 1500 7250 60  0000 C CNN
@@
 Connection ~ 1400 7250
 $Comp
-L -5 #PWR0138
+L -5 #PWR132
 U 1 1 54F266D3
 P 1400 7650
-F 0 "#PWR0138" H 1400 7600 30  0001 C CNN
+F 0 "#PWR132" H 1400 7600 30  0001 C CNN
 F 1 "-5" H 1400 7550 50  0000 C CNN
 F 2 "" H 1400 7650 60  0000 C CNN
@@
 $EndComp
 $Comp
-L +9 #PWR0139
+L +9 #PWR142
 U 1 1 54F2759E
 P 2600 6800
-F 0 "#PWR0139" H 2600 6850 30  0001 C CNN
+F 0 "#PWR142" H 2600 6850 30  0001 C CNN
 F 1 "+9" H 2600 6900 50  0000 C CNN
 F 2 "" H 2600 6800 60  0000 C CNN
@@
 	2600 6800 2600 6850
 $Comp
-L -9 #PWR0140
+L -9 #PWR143
 U 1 1 54F2766A
 P 2600 7800
-F 0 "#PWR0140" H 2600 7750 30  0001 C CNN
+F 0 "#PWR143" H 2600 7750 30  0001 C CNN
 F 1 "-9" H 2600 7700 50  0000 C CNN
 F 2 "" H 2600 7800 60  0000 C CNN
@@
 	3500 7150 3500 7350
 $Comp
-L GND #PWR0141
+L GND #PWR152
 U 1 1 54F278A0
 P 3600 7250
-F 0 "#PWR0141" H 3600 7250 30  0001 C CNN
+F 0 "#PWR152" H 3600 7250 30  0001 C CNN
 F 1 "GND" H 3600 7180 30  0001 C CNN
 F 2 "" H 3600 7250 60  0000 C CNN
@@
 $EndComp
 $Comp
-L GND #PWR0142
+L GND #PWR148
 U 1 1 54F278BE
 P 3100 7250
-F 0 "#PWR0142" H 3100 7250 30  0001 C CNN
+F 0 "#PWR148" H 3100 7250 30  0001 C CNN
 F 1 "GND" H 3100 7180 30  0001 C CNN
 F 2 "" H 3100 7250 60  0000 C CNN
@@
 	3000 7650 3000 7550
 $Comp
-L +9 #PWR0143
+L +9 #PWR146
 U 1 1 54F27AB9
 P 3000 6850
-F 0 "#PWR0143" H 3000 6900 30  0001 C CNN
+F 0 "#PWR146" H 3000 6900 30  0001 C CNN
 F 1 "+9" H 3000 6950 50  0000 C CNN
 F 2 "" H 3000 6850 60  0000 C CNN
@@
 $EndComp
 $Comp
-L +9 #PWR0144
+L +9 #PWR150
 U 1 1 54F27B30
 P 3500 6850
-F 0 "#PWR0144" H 3500 6900 30  0001 C CNN
+F 0 "#PWR150" H 3500 6900 30  0001 C CNN
 F 1 "+9" H 3500 6950 50  0000 C CNN
 F 2 "" H 3500 6850 60  0000 C CNN
@@
 $EndComp
 $Comp
-L -9 #PWR0145
+L -9 #PWR147
 U 1 1 54F27B5F
 P 3000 7650
-F 0 "#PWR0145" H 3000 7600 30  0001 C CNN
+F 0 "#PWR147" H 3000 7600 30  0001 C CNN
 F 1 "-9" H 3000 7550 50  0000 C CNN
 F 2 "" H 3000 7650 60  0000 C CNN
@@
 $EndComp
 $Comp
-L -9 #PWR0146
+L -9 #PWR151
 U 1 1 54F27BD6
 P 3500 7650
-F 0 "#PWR0146" H 3500 7600 30  0001 C CNN
+F 0 "#PWR151" H 3500 7600 30  0001 C CNN
 F 1 "-9" H 3500 7550 50  0000 C CNN
 F 2 "" H 3500 7650 60  0000 C CNN
@@
 Connection ~ 2400 3000
 $Comp
-L GND #PWR0147
+L GND #PWR133
 U 1 1 54F29737
 P 1500 3500
-F 0 "#PWR0147" H 1500 3500 30  0001 C CNN
+F 0 "#PWR133" H 1500 3500 30  0001 C CNN
 F 1 "GND" H 1500 3430 30  0001 C CNN
 F 2 "" H 1500 3500 60  0000 C CNN
@@
 	1500 3500 1500 3400
 $Comp
-L GND #PWR0148
+L GND #PWR136
 U 1 1 54F2981F
 P 1700 3500
-F 0 "#PWR0148" H 1700 3500 30  0001 C CNN
+F 0 "#PWR136" H 1700 3500 30  0001 C CNN
 F 1 "GND" H 1700 3430 30  0001 C CNN
 F 2 "" H 1700 3500 60  0000 C CNN
@@
 	1700 3500 1700 3400
 $Comp
-L GND #PWR0149
+L GND #PWR137
 U 1 1 54F298E1
 P 1900 4150
-F 0 "#PWR0149" H 1900 4150 30  0001 C CNN
+F 0 "#PWR137" H 1900 4150 30  0001 C CNN
 F 1 "GND" H 1900 4080 30  0001 C CNN
 F 2 "" H 1900 4150 60  0000 C CNN
@@
 	1900 4150 1900 4200
 $Comp
-L GND #PWR0150
+L GND #PWR144
 U 1 1 54F299CB
 P 2700 4150
-F 0 "#PWR0150" H 2700 4150 30  0001 C CNN
+F 0 "#PWR144" H 2700 4150 30  0001 C CNN
 F 1 "GND" H 2700 4080 30  0001 C CNN
 F 2 "" H 2700 4150 60  0000 C CNN
@@
 Connection ~ 1900 4800
 $Comp
-L -5 #PWR0151
+L -5 #PWR145
 U 1 1 54F2A843
 P 2700 5150
-F 0 "#PWR0151" H 2700 5100 30  0001 C CNN
+F 0 "#PWR145" H 2700 5100 30  0001 C CNN
 F 1 "-5" H 2700 5050 50  0000 C CNN
 F 2 "" H 2700 5150 60  0000 C CNN
@@
 	2700 5150 2700 5100
 $Comp
-L -5 #PWR0152
+L -5 #PWR138
 U 1 1 54F2A949
 P 1900 5150
-F 0 "#PWR0152" H 1900 5100 30  0001 C CNN
+F 0 "#PWR138" H 1900 5100 30  0001 C CNN
 F 1 "-5" H 1900 5050 50  0000 C CNN
 F 2 "" H 1900 5150 60  0000 C CNN
@@
 	1900 5150 1900 5100
 $Comp
-L -5 #PWR0153
+L -5 #PWR134
 U 1 1 54F2AAA9
 P 1500 5550
-F 0 "#PWR0153" H 1500 5500 30  0001 C CNN
+F 0 "#PWR134" H 1500 5500 30  0001 C CNN
 F 1 "-5" H 1500 5450 50  0000 C CNN
 F 2 "" H 1500 5550 60  0000 C CNN
@@
 Connection ~ 1500 5000
 $Comp
-L GND #PWR0154
+L GND #PWR130
 U 1 1 54F2AED3
 P 1300 4800
-F 0 "#PWR0154" H 1300 4800 30  0001 C CNN
+F 0 "#PWR130" H 1300 4800 30  0001 C CNN
 F 1 "GND" H 1300 4730 30  0001 C CNN
 F 2 "" H 1300 4800 60  0000 C CNN
@@
 	1500 4300 1200 4300
 $Comp
-L GND #PWR0155
+L GND #PWR149
 U 1 1 54F7DEC8
 P 3400 3350
-F 0 "#PWR0155" H 3400 3350 30  0001 C CNN
+F 0 "#PWR149" H 3400 3350 30  0001 C CNN
 F 1 "GND" H 3400 3280 30  0001 C CNN
 F 2 "" H 3400 3350 60  0000 C CNN
@@
 	5000 2100 5100 2100
 $Comp
-L GND #PWR0156
+L GND #PWR153
 U 1 1 54FD5E94
 P 4750 2100
-F 0 "#PWR0156" H 4750 2100 30  0001 C CNN
+F 0 "#PWR153" H 4750 2100 30  0001 C CNN
 F 1 "GND" H 4750 2030 30  0001 C CNN
 F 2 "" H 4750 2100 60  0000 C CNN
@@
 Text Notes 4700 1700 0    50   ~ 0
 @C42 and @R44 are optional compensation devices to boost\ngain slightly at high frequency, if post-fab testing shows that\nstray capacitance from layout results in a rolloff. In the first\nrevision, do not populate them.
+$Comp
+L SINE-ACCURATE #SYM65
+U 1 1 550F357A
+P 1400 2700
+F 0 "#SYM65" H 1400 2700 60  0001 C CNN
+F 1 "SINE-ACCURATE" H 1400 2700 60  0001 C CNN
+F 2 "" H 1400 2700 60  0000 C CNN
+F 3 "" H 1400 2700 60  0000 C CNN
+	1    1400 2700
+	1    0    0    -1
+$EndComp
+$Comp
+L SINE-ACCURATE #SYM67
+U 1 1 550F396B
+P 9750 2700
+F 0 "#SYM67" H 9750 2700 60  0001 C CNN
+F 1 "SINE-ACCURATE" H 9750 2700 60  0001 C CNN
+F 2 "" H 9750 2700 60  0000 C CNN
+F 3 "" H 9750 2700 60  0000 C CNN
+	1    9750 2700
+	1    0    0    -1
+$EndComp
 $EndSCHEMATC

Commit message: More doc fixes
Other:
- note added: "-15dB"
- note added: "-5V"
- note added: "0V"
- note added: "0V7"
- note added: "0dB"
- note added: "3V3"
- note added: "ATTENUATION"
- note added: "BIAS1"
- note added: "BIAS2"
- note added: "Both paths closed"
- note added: "CTRL"
- note added: "GaAs switch bias and truth table:"
- note added: "H"
- note added: "L"
- note added: "Low = -5V High = 0V"
- note added: "SELECTED"
- note added: "Switches open"
- moved on the sheet: Q2, Q3, Q4, R40, R41A, R41B, R41C, R42, R43

Commit message: Nicer BOM lines
Parts:
- C32: OldReference C28 -> (none)
- C33: OldReference C29 -> (none)
- C34: OldReference C30 -> (none)
- C35: OldReference C31 -> (none)
- C36: OldReference C34 -> (none)
- C37: OldReference C35 -> (none)
- C38: OldReference C36 -> (none)
- C39: OldReference C37 -> (none)
- C40: OldReference C40 -> (none)
- C41: OldReference C41 -> (none)
- C42: OldReference C54 -> (none)
- Q2: BOM SEMI GENERIC MMBT3906 -> PNP MMBT3906; OldReference Q4 -> (none)
- Q3: BOM SEMI GENERIC 2N7002 -> NMOS 2N7002; OldReference Q5 -> (none)
- Q4: BOM SEMI GENERIC 2N7002 -> NMOS 2N7002; OldReference Q6 -> (none)
- R40: OldReference R35 -> (none)
- R41: OldReference R5 -> (none)
- R42: OldReference R38 -> (none)
- R43: OldReference R39 -> (none)
- R44: OldReference R41 -> (none)
- R45: OldReference R42 -> (none)
- R46: OldReference R43 -> (none)
- R47: OldReference R89 -> (none)
- R48: OldReference R44 -> (none)
- R49: OldReference R45 -> (none)
- R50: OldReference R46 -> (none)
- R51: OldReference R47 -> (none)
- R52: OldReference R48 -> (none)
- R53: OldReference R49 -> (none)
- R54: OldReference R50 -> (none)
- R55: OldReference R51 -> (none)
- U5: OldReference U6 -> (none)
- U6: OldReference U7 -> (none)
- U7: OldReference U8 -> (none)

Commit message: Add post-testing revision, todo notes
Other:
- note added: "TODO (REV 2):\n- Can we capacitively couple the signal into U5? The diff amp can\n produce significant offset. Cap-coupling 50R is impractical, but\n directly before U5 would allow removing the bias post-termination.\n- Along those lines, can U5 become a transistor amplifier? BFR540?"
