File: wcp52/LPF.sch (KiCad schematic (older format))
At the start: 13 parts

Commit message: BOM line fixes
Parts:
- C43, C44, C51, C52: Description (none) -> CAP MLCC 22pF C0G [0402]
- C45: Description (none) -> CAP MLCC 1.5pF C0G [0402]
- C46, C49: Description (none) -> CAP MLCC 56pF C0G [0402]
- C47, C48, C50: Description (none) -> CAP MLCC 4.7pF C0G [0402]
- L1: Description (none) -> IND CHIP 56nH
- L2, L3: Description (none) -> IND CHIP 47nH
Changed lines of the file:
@@
 EESchema Schematic File Version 2
+LIBS:Altera
+LIBS:AnalogDevices
+LIBS:Atmel
+LIBS:conn-2mm
+LIBS:conn-100mil
+LIBS:conn-cui
+LIBS:conn-fci
+LIBS:conn-linx
+LIBS:conn-molex
+LIBS:conn-tagconnect
+LIBS:conn-test
+LIBS:DiodesInc
+LIBS:display
+LIBS:_electromech
+LIBS:Fairchild
+LIBS:FTDI
+LIBS:Intersil
+LIBS:Lattice
+LIBS:_linear
+LIBS:LinearTech
+LIBS:Littelfuse
+LIBS:logic-4000
+LIBS:logic-7400
+LIBS:MACOM
+LIBS:maxim
+LIBS:mechanical
+LIBS:Microchip
+LIBS:Micron
+LIBS:NXP
+LIBS:onsemi
+LIBS:passive
+LIBS:pasv-BiTech
+LIBS:pasv-Bourns
+LIBS:pasv-cap
+LIBS:pasv-ind
+LIBS:pasv-res
+LIBS:pcb
+LIBS:power
+LIBS:_semi
+LIBS:semi-diode-1N
+LIBS:semi-diode-BA
+LIBS:semi-diode-MCC
+LIBS:semi-diode-MMB
+LIBS:semi-diode-NXP
+LIBS:semi-diode-OnSemi
+LIBS:semi-diode-Vishay
+LIBS:semi-opto-misc
+LIBS:semi-thyristor-2N
+LIBS:semi-trans-2N
+LIBS:semi-trans-AO
+LIBS:semi-trans-BC
+LIBS:semi-trans-DiodesInc
+LIBS:semi-trans-Fairchild
+LIBS:semi-trans-Infineon
+LIBS:semi-trans-IntRect
+LIBS:semi-trans-IXYS
+LIBS:semi-trans-misc
+LIBS:semi-trans-MMB
+LIBS:semi-trans-MPS
+LIBS:semi-trans-NXP
+LIBS:semi-trans-PZT
+LIBS:semi-trans-TI
+LIBS:semi-trans-TIP
+LIBS:semi-trans-Toshiba
+LIBS:silabs
+LIBS:skyworks
+LIBS:ST
+LIBS:st_ic
+LIBS:st_semi
+LIBS:supertex
+LIBS:symbol
+LIBS:TexasInstruments
+LIBS:vishay_semi
+LIBS:Xilinx
+LIBS:pasv-xtal
+LIBS:conn-te
 LIBS:wcp52-cache
 EELAYER 25 0
@@
 F 5 "Murata" H 3900 3600 60  0001 C CNN "Manuf"
 F 6 "DIST DIGIKEY 490-6219-1-ND" H 4700 4150 60  0001 C CNN "BOM"
-F 7 "C42" H 3900 3600 50  0001 C CNN "OldReference"
+F 7 "CAP MLCC 22pF C0G [0402]" H 3900 3600 60  0001 C CNN "Description"
+F 8 "C42" H 3900 3600 50  0001 C CNN "OldReference"
 	1    3900 3600
 	1    0    0    -1
@@
 F 5 "Samsung" H 4600 3300 60  0001 C CNN "Manuf"
 F 6 "DIST DIGIKEY 1276-6281-1-ND" H 4600 3300 60  0001 C CNN "BOM"
-F 7 "L1" H 4600 3300 50  0001 C CNN "OldReference"
+F 7 "IND CHIP 56nH" H 4600 3300 60  0001 C CNN "Description"
+F 8 "L1" H 4600 3300 50  0001 C CNN "OldReference"
 	1    4600 3300
 	0    1    1    0
@@
 F 5 "Murata" H 4300 3600 60  0001 C CNN "Manuf"
 F 6 "DIST DIGIKEY 490-6219-1-ND" H 5100 4150 60  0001 C CNN "BOM"
-F 7 "C43" H 4300 3600 50  0001 C CNN "OldReference"
+F 7 "CAP MLCC 22pF C0G [0402]" H 4300 3600 60  0001 C CNN "Description"
+F 8 "C43" H 4300 3600 50  0001 C CNN "OldReference"
 	1    4300 3600
 	1    0    0    -1
@@
 F 5 "Samsung" H 4600 2950 60  0001 C CNN "Manuf"
 F 6 "DIST DIGIKEY 1276-1656-1-ND" H 5400 3500 60  0001 C CNN "BOM"
-F 7 "C44" H 4600 2950 50  0001 C CNN "OldReference"
+F 7 "CAP MLCC 1.5pF C0G [0402]" H 4600 2950 60  0001 C CNN "Description"
+F 8 "C44" H 4600 2950 50  0001 C CNN "OldReference"
 	1    4600 2950
 	0    1    1    0
@@
 F 5 "Samsung" H 5200 3300 60  0001 C CNN "Manuf"
 F 6 "DIST DIGIKEY 1276-6280-1-ND" H 5200 3300 60  0001 C CNN "BOM"
-F 7 "L2" H 5200 3300 50  0001 C CNN "OldReference"
+F 7 "IND CHIP 47nH" H 5200 3300 60  0001 C CNN "Description"
+F 8 "L2" H 5200 3300 50  0001 C CNN "OldReference"
 	1    5200 3300
 	0    1    1    0
@@
 F 5 "Samsung" H 5200 2950 60  0001 C CNN "Manuf"
 F 6 "DIST DIGIKEY 1276-1703-1-ND" H 6000 3500 60  0001 C CNN "BOM"
-F 7 "C47" H 5200 2950 50  0001 C CNN "OldReference"
+F 7 "CAP MLCC 4.7pF C0G [0402]" H 5200 2950 60  0001 C CNN "Description"
+F 8 "C47" H 5200 2950 50  0001 C CNN "OldReference"
 	1    5200 2950
 	0    1    1    0
@@
 F 5 "Samsung" H 5200 2550 60  0001 C CNN "Manuf"
 F 6 "DIST DIGIKEY 1276-1703-1-ND" H 6000 3100 60  0001 C CNN "BOM"
-F 7 "C46" H 5200 2550 50  0001 C CNN "OldReference"
+F 7 "CAP MLCC 4.7pF C0G [0402]" H 5200 2550 60  0001 C CNN "Description"
+F 8 "C46" H 5200 2550 50  0001 C CNN "OldReference"
 	1    5200 2550
 	0    1    1    0
@@
 F 5 "Samsung" H 5800 3300 60  0001 C CNN "Manuf"
 F 6 "DIST DIGIKEY 1276-6280-1-ND" H 5800 3300 60  0001 C CNN "BOM"
-F 7 "L3" H 5800 3300 50  0001 C CNN "OldReference"
+F 7 "IND CHIP 47nH" H 5800 3300 60  0001 C CNN "Description"
+F 8 "L3" H 5800 3300 50  0001 C CNN "OldReference"
 	1    5800 3300
 	0    1    1    0
@@
 F 5 "Samsung" H 5800 2950 60  0001 C CNN "Manuf"
 F 6 "DIST DIGIKEY 1276-1703-1-ND" H 6600 3500 60  0001 C CNN "BOM"
-F 7 "C49" H 5800 2950 50  0001 C CNN "OldReference"
+F 7 "CAP MLCC 4.7pF C0G [0402]" H 5800 2950 60  0001 C CNN "Description"
+F 8 "C49" H 5800 2950 50  0001 C CNN "OldReference"
 	1    5800 2950
 	0    1    1    0
@@
 F 5 "Samsung" H 4900 3600 60  0001 C CNN "Manuf"
 F 6 "DIST DIGIKEY 1276-1707-1-ND" H 5700 4150 60  0001 C CNN "BOM"
-F 7 "C45" H 4900 3600 50  0001 C CNN "OldReference"
+F 7 "CAP MLCC 56pF C0G [0402]" H 4900 3600 60  0001 C CNN "Description"
+F 8 "C45" H 4900 3600 50  0001 C CNN "OldReference"
 	1    4900 3600
 	1    0    0    -1
@@
 F 5 "Samsung" H 5500 3600 60  0001 C CNN "Manuf"
 F 6 "DIST DIGIKEY 1276-1707-1-ND" H 6300 4150 60  0001 C CNN "BOM"
-F 7 "C48" H 5500 3600 50  0001 C CNN "OldReference"
+F 7 "CAP MLCC 56pF C0G [0402]" H 5500 3600 60  0001 C CNN "Description"
+F 8 "C48" H 5500 3600 50  0001 C CNN "OldReference"
 	1    5500 3600
 	1    0    0    -1
@@
 F 5 "Murata" H 6100 3600 60  0001 C CNN "Manuf"
 F 6 "DIST DIGIKEY 490-6219-1-ND" H 6900 4150 60  0001 C CNN "BOM"
-F 7 "C50" H 6100 3600 50  0001 C CNN "OldReference"
+F 7 "CAP MLCC 22pF C0G [0402]" H 6100 3600 60  0001 C CNN "Description"
+F 8 "C50" H 6100 3600 50  0001 C CNN "OldReference"
 	1    6100 3600
 	1    0    0    -1
@@
 F 5 "Murata" H 6500 3600 60  0001 C CNN "Manuf"
 F 6 "DIST DIGIKEY 490-6219-1-ND" H 7300 4150 60  0001 C CNN "BOM"
-F 7 "C51" H 6500 3600 50  0001 C CNN "OldReference"
+F 7 "CAP MLCC 22pF C0G [0402]" H 6500 3600 60  0001 C CNN "Description"
+F 8 "C51" H 6500 3600 50  0001 C CNN "OldReference"
 	1    6500 3600
 	1    0    0    -1
@@
 C6 5F 05 4E E2 BB B2 02 2C AC E2 1F E1 4E C2 E1 06 D8 47 59 46 F6 AB CF 56 EE 9C BE 21 0E 51 00
 00 36 21 77 86 1F 00 00 D4 45 EA 03 00 B0 0B 52 1F 00 80 5D 90 FA 00 00 EC E2 7F 01 3B 40 24 1D
-60 0E DB 19 00 00 00 00 49 45 4E 44 AE 42 60 82 58
+60 0E DB 19 00 00 00 00 49 45 4E 44 AE 42 60 82 FF
 EndData
 $EndBitmap

Commit message: Schematic/doc work
Changed lines of the file:
@@
 Sheet 5 13
 Title "LPF for Output Amplifier"
-Date "2015-03-13"
+Date "2015-03-21"
 Rev ""
 Comp "WCP52"
@@
 Comment2 ""
 Comment3 ""
-Comment4 "Eng: Chris Pavlina"
+Comment4 ""
 $EndDescr
 Text HLabel 3100 3300 0    60   BiDi ~ 0
@@
 EndData
 $EndBitmap
-Text Notes 1000 5350 0    50   ~ 0
+Text Notes 1000 5350 0    60   ~ 0
 Intended frequency response of filter:
 $EndSCHEMATC

Commit message: Nicer BOM lines
Parts:
- C43: OldReference C42 -> (none)
- C44: OldReference C43 -> (none)
- C45: OldReference C44 -> (none)
- C46: OldReference C45 -> (none)
- C47: OldReference C46 -> (none)
- C48: OldReference C47 -> (none)
- C49: OldReference C48 -> (none)
- C50: OldReference C49 -> (none)
- C51: OldReference C50 -> (none)
- C52: OldReference C51 -> (none)
- L1: OldReference L1 -> (none)
- L2: OldReference L2 -> (none)
- L3: OldReference L3 -> (none)
Changed lines of the file:
@@
 F 6 "DIST DIGIKEY 490-6219-1-ND" H 4700 4150 60  0001 C CNN "BOM"
 F 7 "CAP MLCC 22pF C0G [0402]" H 3900 3600 60  0001 C CNN "Description"
-F 8 "C42" H 3900 3600 50  0001 C CNN "OldReference"
 	1    3900 3600
 	1    0    0    -1
@@
 F 6 "DIST DIGIKEY 1276-6281-1-ND" H 4600 3300 60  0001 C CNN "BOM"
 F 7 "IND CHIP 56nH" H 4600 3300 60  0001 C CNN "Description"
-F 8 "L1" H 4600 3300 50  0001 C CNN "OldReference"
 	1    4600 3300
 	0    1    1    0
@@
 F 6 "DIST DIGIKEY 490-6219-1-ND" H 5100 4150 60  0001 C CNN "BOM"
 F 7 "CAP MLCC 22pF C0G [0402]" H 4300 3600 60  0001 C CNN "Description"
-F 8 "C43" H 4300 3600 50  0001 C CNN "OldReference"
 	1    4300 3600
 	1    0    0    -1
@@
 F 6 "DIST DIGIKEY 1276-1656-1-ND" H 5400 3500 60  0001 C CNN "BOM"
 F 7 "CAP MLCC 1.5pF C0G [0402]" H 4600 2950 60  0001 C CNN "Description"
-F 8 "C44" H 4600 2950 50  0001 C CNN "OldReference"
 	1    4600 2950
 	0    1    1    0
@@
 F 6 "DIST DIGIKEY 1276-6280-1-ND" H 5200 3300 60  0001 C CNN "BOM"
 F 7 "IND CHIP 47nH" H 5200 3300 60  0001 C CNN "Description"
-F 8 "L2" H 5200 3300 50  0001 C CNN "OldReference"
 	1    5200 3300
 	0    1    1    0
@@
 F 6 "DIST DIGIKEY 1276-1703-1-ND" H 6000 3500 60  0001 C CNN "BOM"
 F 7 "CAP MLCC 4.7pF C0G [0402]" H 5200 2950 60  0001 C CNN "Description"
-F 8 "C47" H 5200 2950 50  0001 C CNN "OldReference"
 	1    5200 2950
 	0    1    1    0
@@
 F 6 "DIST DIGIKEY 1276-1703-1-ND" H 6000 3100 60  0001 C CNN "BOM"
 F 7 "CAP MLCC 4.7pF C0G [0402]" H 5200 2550 60  0001 C CNN "Description"
-F 8 "C46" H 5200 2550 50  0001 C CNN "OldReference"
 	1    5200 2550
 	0    1    1    0
@@
 F 6 "DIST DIGIKEY 1276-6280-1-ND" H 5800 3300 60  0001 C CNN "BOM"
 F 7 "IND CHIP 47nH" H 5800 3300 60  0001 C CNN "Description"
-F 8 "L3" H 5800 3300 50  0001 C CNN "OldReference"
 	1    5800 3300
 	0    1    1    0
@@
 F 6 "DIST DIGIKEY 1276-1703-1-ND" H 6600 3500 60  0001 C CNN "BOM"
 F 7 "CAP MLCC 4.7pF C0G [0402]" H 5800 2950 60  0001 C CNN "Description"
-F 8 "C49" H 5800 2950 50  0001 C CNN "OldReference"
 	1    5800 2950
 	0    1    1    0
@@
 F 6 "DIST DIGIKEY 1276-1707-1-ND" H 5700 4150 60  0001 C CNN "BOM"
 F 7 "CAP MLCC 56pF C0G [0402]" H 4900 3600 60  0001 C CNN "Description"
-F 8 "C45" H 4900 3600 50  0001 C CNN "OldReference"
 	1    4900 3600
 	1    0    0    -1
@@
 F 6 "DIST DIGIKEY 1276-1707-1-ND" H 6300 4150 60  0001 C CNN "BOM"
 F 7 "CAP MLCC 56pF C0G [0402]" H 5500 3600 60  0001 C CNN "Description"
-F 8 "C48" H 5500 3600 50  0001 C CNN "OldReference"
 	1    5500 3600
 	1    0    0    -1
@@
 F 6 "DIST DIGIKEY 490-6219-1-ND" H 6900 4150 60  0001 C CNN "BOM"
 F 7 "CAP MLCC 22pF C0G [0402]" H 6100 3600 60  0001 C CNN "Description"
-F 8 "C50" H 6100 3600 50  0001 C CNN "OldReference"
 	1    6100 3600
 	1    0    0    -1
@@
 F 6 "DIST DIGIKEY 490-6219-1-ND" H 7300 4150 60  0001 C CNN "BOM"
 F 7 "CAP MLCC 22pF C0G [0402]" H 6500 3600 60  0001 C CNN "Description"
-F 8 "C51" H 6500 3600 50  0001 C CNN "OldReference"
 	1    6500 3600
 	1    0    0    -1
@@
 F 2 "" H 3900 3800 60  0000 C CNN
 F 3 "" H 3900 3800 60  0000 C CNN
-F 4 "#PWR0157" H 3900 3800 50  0001 C CNN "OldReference"
 	1    3900 3800
 	1    0    0    -1
@@
 F 2 "" H 4300 3800 60  0000 C CNN
 F 3 "" H 4300 3800 60  0000 C CNN
-F 4 "#PWR0158" H 4300 3800 50  0001 C CNN "OldReference"
 	1    4300 3800
 	1    0    0    -1
@@
 F 2 "" H 4900 3800 60  0000 C CNN
 F 3 "" H 4900 3800 60  0000 C CNN
-F 4 "#PWR0159" H 4900 3800 50  0001 C CNN "OldReference"
 	1    4900 3800
 	1    0    0    -1
@@
 F 2 "" H 5500 3800 60  0000 C CNN
 F 3 "" H 5500 3800 60  0000 C CNN
-F 4 "#PWR0160" H 5500 3800 50  0001 C CNN "OldReference"
 	1    5500 3800
 	1    0    0    -1
@@
 F 2 "" H 6100 3800 60  0000 C CNN
 F 3 "" H 6100 3800 60  0000 C CNN
-F 4 "#PWR0161" H 6100 3800 50  0001 C CNN "OldReference"
 	1    6100 3800
 	1    0    0    -1
@@
 F 2 "" H 6500 3800 60  0000 C CNN
 F 3 "" H 6500 3800 60  0000 C CNN
-F 4 "#PWR0162" H 6500 3800 50  0001 C CNN "OldReference"
 	1    6500 3800
 	1    0    0    -1
@@
 C6 5F 05 4E E2 BB B2 02 2C AC E2 1F E1 4E C2 E1 06 D8 47 59 46 F6 AB CF 56 EE 9C BE 21 0E 51 00
 00 36 21 77 86 1F 00 00 D4 45 EA 03 00 B0 0B 52 1F 00 80 5D 90 FA 00 00 EC E2 7F 01 3B 40 24 1D
-60 0E DB 19 00 00 00 00 49 45 4E 44 AE 42 60 82 90
+60 0E DB 19 00 00 00 00 49 45 4E 44 AE 42 60 82 58
 EndData
 $EndBitmap
