File: wcp52/PowerInput.sch (KiCad schematic (older format))
At the start: 20 parts, among them Q11 MMBT3904, Q12 MMBT3906, Q13 IRLML6402, Q14 AOD417, U11 TL431AIDBZ, U12 LM393M

Commit message: BOM line fixes
Parts:
- C72, C73, C74, C75, Q11, Q12, R82, R86, R87, R88: Manuf Value -> (none)
- R81: Description (none) -> PPTC 350mA/750mA 30V [1206]
- R83, R84, R85: Description (none) -> RESPACK SMD 10k 5% [4x0603]
Changed lines of the file:
@@
 EESchema Schematic File Version 2
+LIBS:Altera
+LIBS:AnalogDevices
+LIBS:Atmel
+LIBS:conn-2mm
+LIBS:conn-100mil
+LIBS:conn-cui
+LIBS:conn-fci
+LIBS:conn-linx
+LIBS:conn-molex
+LIBS:conn-tagconnect
+LIBS:conn-test
+LIBS:DiodesInc
+LIBS:display
+LIBS:_electromech
+LIBS:Fairchild
+LIBS:FTDI
+LIBS:Intersil
+LIBS:Lattice
+LIBS:_linear
+LIBS:LinearTech
+LIBS:Littelfuse
+LIBS:logic-4000
+LIBS:logic-7400
+LIBS:MACOM
+LIBS:maxim
+LIBS:mechanical
+LIBS:Microchip
+LIBS:Micron
+LIBS:NXP
+LIBS:onsemi
+LIBS:passive
+LIBS:pasv-BiTech
+LIBS:pasv-Bourns
+LIBS:pasv-cap
+LIBS:pasv-ind
+LIBS:pasv-res
+LIBS:pcb
+LIBS:power
+LIBS:_semi
+LIBS:semi-diode-1N
+LIBS:semi-diode-BA
+LIBS:semi-diode-MCC
+LIBS:semi-diode-MMB
+LIBS:semi-diode-NXP
+LIBS:semi-diode-OnSemi
+LIBS:semi-diode-Vishay
+LIBS:semi-opto-misc
+LIBS:semi-thyristor-2N
+LIBS:semi-trans-2N
+LIBS:semi-trans-AO
+LIBS:semi-trans-BC
+LIBS:semi-trans-DiodesInc
+LIBS:semi-trans-Fairchild
+LIBS:semi-trans-Infineon
+LIBS:semi-trans-IntRect
+LIBS:semi-trans-IXYS
+LIBS:semi-trans-misc
+LIBS:semi-trans-MMB
+LIBS:semi-trans-MPS
+LIBS:semi-trans-NXP
+LIBS:semi-trans-PZT
+LIBS:semi-trans-TI
+LIBS:semi-trans-TIP
+LIBS:semi-trans-Toshiba
+LIBS:silabs
+LIBS:skyworks
+LIBS:ST
+LIBS:st_ic
+LIBS:st_semi
+LIBS:supertex
+LIBS:symbol
+LIBS:TexasInstruments
+LIBS:vishay_semi
+LIBS:Xilinx
+LIBS:pasv-xtal
+LIBS:conn-te
 LIBS:wcp52-cache
 EELAYER 25 0
@@
 F 5 "BelFuse" H 1800 1700 60  0001 C CNN "Manuf"
 F 6 "DIST DIGIKEY 507-1801-1-ND" H 1800 1700 60  0001 C CNN "BOM"
-F 7 "R1" H 1800 1700 50  0001 C CNN "OldReference"
+F 7 "PPTC 350mA/750mA 30V [1206]" H 1800 1700 60  0001 C CNN "Description"
+F 8 "R1" H 1800 1700 50  0001 C CNN "OldReference"
 	1    1800 1700
 	0    -1   1    0
@@
 F 2 "IPC7351-Nominal:CAPC2012X70" H 7400 1900 50  0001 C CNN
 F 3 "" H 7390 1875 60  0000 C CNN
-F 4 "Value" H 7400 1900 60  0001 C CNN "Manuf"
+F 4 "" H 7400 1900 60  0001 C CNN "Manuf"
 F 5 "CAP MLCC 100n ≥X5R 16V 10% [0805]" H 8200 2450 60  0001 C CNN "BOM"
 F 6 "C3" H 7400 1900 50  0001 C CNN "OldReference"
@@
 F 2 "smd-semi:SOT-23" H 4900 2900 50  0001 C CNN
 F 3 "" H 4900 2900 60  0000 C CNN
-F 4 "Value" H 4900 2900 60  0001 C CNN "Manuf"
+F 4 "" H 4900 2900 60  0001 C CNN "Manuf"
 F 5 "SEMI GENERIC MMBT3906" H 5700 3450 60  0001 C CNN "BOM"
 F 6 "Q1" H 4900 2900 50  0001 C CNN "OldReference"
@@
 F 2 "IPC7351-Nominal:CAPC2012X70" H 5850 3800 50  0001 C CNN
 F 3 "" H 5840 3775 60  0000 C CNN
-F 4 "Value" H 5850 3800 60  0001 C CNN "Manuf"
+F 4 "" H 5850 3800 60  0001 C CNN "Manuf"
 F 5 "CAP MLCC 100n ≥X5R 16V 10% [0805]" H 6650 4350 60  0001 C CNN "BOM"
 F 6 "C2" H 5850 3800 50  0001 C CNN "OldReference"
@@
 F 3 "" H 3250 5900 60  0000 C CNN
 F 4 "SEMI GENERIC MMBT3904" H 4050 6450 60  0001 C CNN "BOM"
-F 5 "Value" H 3250 5900 60  0001 C CNN "Manuf"
+F 5 "" H 3250 5900 60  0001 C CNN "Manuf"
 F 6 "Q14" H 3250 5900 50  0001 C CNN "OldReference"
 	1    3250 5900
@@
 F 5 "Yageo" H 3500 2500 60  0001 C CNN "Manuf"
 F 6 "DIST DIGIKEY YC164J-10KCT-ND" H 3500 2500 60  0001 C CNN "BOM"
-F 7 "R112" H 3500 2500 50  0001 C CNN "OldReference"
+F 7 "RESPACK SMD 10k 5% [4x0603]" H 3500 2500 60  0001 C CNN "Description"
+F 8 "R112" H 3500 2500 50  0001 C CNN "OldReference"
 	1    3500 2500
 	-1   0    0    -1
@@
 F 5 "Yageo" H 3500 2800 60  0001 C CNN "Manuf"
 F 6 "DIST DIGIKEY YC164J-10KCT-ND" H 3500 2800 60  0001 C CNN "BOM"
-F 7 "R112" H 3500 2800 50  0001 C CNN "OldReference"
+F 7 "RESPACK SMD 10k 5% [4x0603]" H 3500 2800 60  0001 C CNN "Description"
+F 8 "R112" H 3500 2800 50  0001 C CNN "OldReference"
 	2    3500 2800
 	-1   0    0    -1
@@
 F 5 "Yageo" H 3800 2500 60  0001 C CNN "Manuf"
 F 6 "DIST DIGIKEY YC164J-10KCT-ND" H 3800 2500 60  0001 C CNN "BOM"
-F 7 "R112" H 3800 2500 50  0001 C CNN "OldReference"
+F 7 "RESPACK SMD 10k 5% [4x0603]" H 3800 2500 60  0001 C CNN "Description"
+F 8 "R112" H 3800 2500 50  0001 C CNN "OldReference"
 	3    3800 2500
 	1    0    0    -1
@@
 F 5 "Yageo" H 3800 2800 60  0001 C CNN "Manuf"
 F 6 "DIST DIGIKEY YC164J-10KCT-ND" H 3800 2800 60  0001 C CNN "BOM"
-F 7 "R112" H 3800 2800 50  0001 C CNN "OldReference"
+F 7 "RESPACK SMD 10k 5% [4x0603]" H 3800 2800 60  0001 C CNN "Description"
+F 8 "R112" H 3800 2800 50  0001 C CNN "OldReference"
 	4    3800 2800
 	1    0    0    -1
@@
 F 5 "Yageo" H 3800 3100 60  0001 C CNN "Manuf"
 F 6 "DIST DIGIKEY YC164J-10KCT-ND" H 3800 3100 60  0001 C CNN "BOM"
-F 7 "R4" H 3800 3100 50  0001 C CNN "OldReference"
+F 7 "RESPACK SMD 10k 5% [4x0603]" H 3800 3100 60  0001 C CNN "Description"
+F 8 "R4" H 3800 3100 50  0001 C CNN "OldReference"
 	4    3800 3100
 	1    0    0    -1
@@
 F 5 "Yageo" H 3800 5400 60  0001 C CNN "Manuf"
 F 6 "DIST DIGIKEY YC164J-10KCT-ND" H 3800 5400 60  0001 C CNN "BOM"
-F 7 "R4" H 3800 5400 50  0001 C CNN "OldReference"
+F 7 "RESPACK SMD 10k 5% [4x0603]" H 3800 5400 60  0001 C CNN "Description"
+F 8 "R4" H 3800 5400 50  0001 C CNN "OldReference"
 	3    3800 5400
 	1    0    0    1
@@
 F 5 "Yageo" H 3500 5400 60  0001 C CNN "Manuf"
 F 6 "DIST DIGIKEY YC164J-10KCT-ND" H 3500 5400 60  0001 C CNN "BOM"
-F 7 "R4" H 3500 5400 50  0001 C CNN "OldReference"
+F 7 "RESPACK SMD 10k 5% [4x0603]" H 3500 5400 60  0001 C CNN "Description"
+F 8 "R4" H 3500 5400 50  0001 C CNN "OldReference"
 	1    3500 5400
 	1    0    0    -1
@@
 F 5 "Yageo" H 3050 6400 60  0001 C CNN "Manuf"
 F 6 "DIST DIGIKEY YC164J-10KCT-ND" H 3050 6400 60  0001 C CNN "BOM"
-F 7 "R3" H 3050 6400 50  0001 C CNN "OldReference"
+F 7 "RESPACK SMD 10k 5% [4x0603]" H 3050 6400 60  0001 C CNN "Description"
+F 8 "R3" H 3050 6400 50  0001 C CNN "OldReference"
 	2    3050 6400
 	1    0    0    -1
@@
 F 5 "Yageo" H 2750 6200 60  0001 C CNN "Manuf"
 F 6 "DIST DIGIKEY YC164J-10KCT-ND" H 2750 6200 60  0001 C CNN "BOM"
-F 7 "R3" H 2750 6200 50  0001 C CNN "OldReference"
+F 7 "RESPACK SMD 10k 5% [4x0603]" H 2750 6200 60  0001 C CNN "Description"
+F 8 "R3" H 2750 6200 50  0001 C CNN "OldReference"
 	3    2750 6200
 	0    1    1    0
@@
 F 5 "Yageo" H 3250 3800 60  0001 C CNN "Manuf"
 F 6 "DIST DIGIKEY YC164J-10KCT-ND" H 3250 3800 60  0001 C CNN "BOM"
-F 7 "R3" H 3250 3800 50  0001 C CNN "OldReference"
+F 7 "RESPACK SMD 10k 5% [4x0603]" H 3250 3800 60  0001 C CNN "Description"
+F 8 "R3" H 3250 3800 50  0001 C CNN "OldReference"
 	1    3250 3800
 	0    -1   1    0
@@
 F 5 "Yageo" H 4600 2700 60  0001 C CNN "Manuf"
 F 6 "DIST DIGIKEY YC164J-10KCT-ND" H 4600 2700 60  0001 C CNN "BOM"
-F 7 "R3" H 4600 2700 50  0001 C CNN "OldReference"
+F 7 "RESPACK SMD 10k 5% [4x0603]" H 4600 2700 60  0001 C CNN "Description"
+F 8 "R3" H 4600 2700 50  0001 C CNN "OldReference"
 	4    4600 2700
 	1    0    0    1
@@
 F 2 "IPC7351-Nominal:CAPC1608X55" H 8400 2100 50  0001 C CNN
 F 3 "" H 8390 2075 60  0000 C CNN
-F 4 "Value" H 8400 2100 60  0001 C CNN "Manuf"
+F 4 "" H 8400 2100 60  0001 C CNN "Manuf"
 F 5 "CAP MLCC 10n ≥X5R 50V 10% [0603]" H 9200 2650 60  0001 C CNN "BOM"
 F 6 "C4" H 8400 2100 50  0001 C CNN "OldReference"
@@
 F 2 "IPC7351-Nominal:CAPC1608X55" H 4150 5400 50  0001 C CNN
 F 3 "" H 4140 5375 60  0000 C CNN
-F 4 "Value" H 4150 5400 60  0001 C CNN "Manuf"
+F 4 "" H 4150 5400 60  0001 C CNN "Manuf"
 F 5 "CAP MLCC 10n ≥X5R 50V 10% [0603]" H 4950 5950 60  0001 C CNN "BOM"
 F 6 "C1" H 4150 5400 50  0001 C CNN "OldReference"
@@
 F 2 "IPC7351-Nominal:RESC1608X50" H 2400 2500 50  0001 C CNN
 F 3 "" H 2400 2550 60  0000 C CNN
-F 4 "Value" H 2400 2500 60  0001 C CNN "Manuf"
+F 4 "" H 2400 2500 60  0001 C CNN "Manuf"
 F 5 "RES SMD 3.3k 5% [0603]" H 3150 3050 60  0001 C CNN "BOM"
 F 6 "R2" H 2400 2500 50  0001 C CNN "OldReference"
@@
 F 2 "IPC7351-Nominal:RESC1608X50" H 4750 4600 50  0001 C CNN
 F 3 "" H 4750 4650 60  0000 C CNN
-F 4 "Value" H 4750 4600 60  0001 C CNN "Manuf"
+F 4 "" H 4750 4600 60  0001 C CNN "Manuf"
 F 5 "RES SMD 1M 5% [0603]" H 5500 5150 60  0001 C CNN "BOM"
 F 6 "R10" H 4750 4600 50  0001 C CNN "OldReference"
@@
 F 2 "IPC7351-Nominal:RESC1608X50" H 4600 3300 50  0001 C CNN
 F 3 "" H 4600 3350 60  0000 C CNN
-F 4 "Value" H 4600 3300 60  0001 C CNN "Manuf"
+F 4 "" H 4600 3300 60  0001 C CNN "Manuf"
 F 5 "RES SMD 3.3k 5% [0603]" H 5350 3850 60  0001 C CNN "BOM"
 F 6 "R9" H 4600 3300 50  0001 C CNN "OldReference"
@@
 F 2 "IPC7351-Nominal:RESC1608X50" H 7000 1900 50  0001 C CNN
 F 3 "" H 7000 1950 60  0000 C CNN
-F 4 "Value" H 7000 1900 60  0001 C CNN "Manuf"
+F 4 "" H 7000 1900 60  0001 C CNN "Manuf"
 F 5 "RES SMD 1M 5% [0603]" H 7750 2450 60  0001 C CNN "BOM"
 F 6 "R11" H 7000 1900 50  0001 C CNN "OldReference"

Commit message: BOM corrections/combinations, etc
Add configuration for bomtool
Remove old schematic file no longer used
Parts:
- C73, C74: BOM CAP MLCC 100n ≥X5R 16V 10% [0805] -> CAP MLCC 100n ≥X7R 20V 10% [0805]
- D5, D6: BOM (none) -> SEMI GENERIC MMBD4148
- U11: BOM (none) -> IC TI TL431AIDBZ
- U12: BOM (none) -> IC GENERIC LM393M
Changed lines of the file:
@@
 F 2 "IPC7351-Nominal:CAPC2012X70" H 7400 1900 50  0001 C CNN
 F 3 "" H 7390 1875 60  0000 C CNN
-F 4 "" H 7400 1900 60  0001 C CNN "Manuf"
-F 5 "CAP MLCC 100n ≥X5R 16V 10% [0805]" H 8200 2450 60  0001 C CNN "BOM"
-F 6 "C3" H 7400 1900 50  0001 C CNN "OldReference"
+F 4 "CAP MLCC 100n ≥X7R 20V 10% [0805]" H 8200 2450 60  0001 C CNN "BOM"
+F 5 "C3" H 7400 1900 50  0001 C CNN "OldReference"
 	1    7400 1900
 	1    0    0    -1
@@
 F 2 "IPC7351-Nominal:SOIC127P600X175-8" H 4200 3700 50  0001 C CNN
 F 3 "" V 4200 3850 60  0000 C CNN
-F 4 "U2" H 4200 3700 50  0001 C CNN "OldReference"
+F 4 "IC GENERIC LM393M" H 4200 3700 60  0001 C CNN "BOM"
+F 5 "U2" H 4200 3700 50  0001 C CNN "OldReference"
 	2    4200 3700
 	1    0    0    -1
@@
 F 2 "IPC7351-Nominal:SOIC127P600X175-8" H 4200 4600 50  0001 C CNN
 F 3 "" V 4200 4750 60  0000 C CNN
-F 4 "U2" H 4200 4600 50  0001 C CNN "OldReference"
+F 4 "IC GENERIC LM393M" H 4200 4600 60  0001 C CNN "BOM"
+F 5 "U2" H 4200 4600 50  0001 C CNN "OldReference"
 	1    4200 4600
 	1    0    0    -1
@@
 F 2 "smd-semi:SOT-23" H 4250 4100 50  0001 C CNN
 F 3 "" H 4250 4100 60  0000 C CNN
-F 4 "D1" H 4250 4100 50  0001 C CNN "OldReference"
+F 4 "SEMI GENERIC MMBD4148" H 4250 4100 60  0001 C CNN "BOM"
+F 5 "D1" H 4250 4100 50  0001 C CNN "OldReference"
 	1    4250 4100
 	0    -1   -1   0
@@
 F 2 "smd-semi:SOT-23" H 2400 5400 50  0001 C CNN
 F 3 "" H 2400 5400 60  0000 C CNN
-F 4 "U1" H 2400 5400 50  0001 C CNN "OldReference"
+F 4 "IC TI TL431AIDBZ" H 2400 5400 60  0001 C CNN "BOM"
+F 5 "U1" H 2400 5400 50  0001 C CNN "OldReference"
 	1    2400 5400
 	1    0    0    -1
@@
 F 2 "smd-semi:SOT-23" H 4600 2100 50  0001 C CNN
 F 3 "" H 4600 2100 60  0000 C CNN
-F 4 "D2" H 4600 2100 50  0001 C CNN "OldReference"
+F 4 "SEMI GENERIC MMBD4148" H 4600 2100 60  0001 C CNN "BOM"
+F 5 "D2" H 4600 2100 50  0001 C CNN "OldReference"
 	1    4600 2100
 	1    0    0    -1
@@
 F 2 "IPC7351-Nominal:SOIC127P600X175-8" H 5600 3800 50  0001 C CNN
 F 3 "" V 5600 3950 60  0000 C CNN
-F 4 "U2" H 5600 3800 50  0001 C CNN "OldReference"
+F 4 "IC GENERIC LM393M" H 5600 3800 60  0001 C CNN "BOM"
+F 5 "U2" H 5600 3800 50  0001 C CNN "OldReference"
 	3    5600 3800
 	1    0    0    -1
@@
 F 2 "IPC7351-Nominal:CAPC2012X70" H 5850 3800 50  0001 C CNN
 F 3 "" H 5840 3775 60  0000 C CNN
-F 4 "" H 5850 3800 60  0001 C CNN "Manuf"
-F 5 "CAP MLCC 100n ≥X5R 16V 10% [0805]" H 6650 4350 60  0001 C CNN "BOM"
-F 6 "C2" H 5850 3800 50  0001 C CNN "OldReference"
+F 4 "CAP MLCC 100n ≥X7R 20V 10% [0805]" H 6650 4350 60  0001 C CNN "BOM"
+F 5 "C2" H 5850 3800 50  0001 C CNN "OldReference"
 	1    5850 3800
 	1    0    0    -1

Commit message: Schematic/doc work
Changed lines of the file:
@@
 Sheet 11 13
 Title "Power Input Circuit"
-Date "2015-03-13"
+Date "2015-03-21"
 Rev ""
 Comp "WCP52"
@@
 Comment2 ""
 Comment3 ""
-Comment4 "Eng: Chris Pavlina"
+Comment4 ""
 $EndDescr
 $Comp
@@
 U 1 1 54F4B9D8
 P 4900 2900
-F 0 "Q12" H 5200 2950 50  0000 C CNN
-F 1 "MMBT3906" H 5200 2850 50  0000 C CNN
+F 0 "Q12" H 5100 3050 50  0000 C CNN
+F 1 "MMBT3906" H 5200 2850 50  0001 C CNN
 F 2 "smd-semi:SOT-23" H 4900 2900 50  0001 C CNN
 F 3 "" H 4900 2900 60  0000 C CNN
@@
 U 1 1 54F4BA7F
 P 4200 4600
-F 0 "U12" H 4200 4950 50  0000 C CNN
-F 1 "LM393M" H 4200 4850 50  0000 C CNN
+F 0 "U12" H 4200 4850 50  0000 C CNN
+F 1 "LM393M" H 4200 4850 50  0001 C CNN
 F 2 "IPC7351-Nominal:SOIC127P600X175-8" H 4200 4600 50  0001 C CNN
 F 3 "" V 4200 4750 60  0000 C CNN
@@
 	0    -1   -1   0
 $EndComp
-Text HLabel 9400 1700 2    50   Output ~ 0
+Text HLabel 9400 1700 2    60   Output ~ 0
 OUT
-Text HLabel 1350 1700 0    50   Input ~ 0
+Text HLabel 1350 1700 0    60   Input ~ 0
 IN
 Wire Wire Line

Commit message: More doc fixes
Changed lines of the file:
@@
 U 1 1 54F4B9D8
 P 4900 2900
-F 0 "Q12" H 5100 3050 50  0000 C CNN
+F 0 "Q12" H 5100 3000 50  0000 C CNN
 F 1 "MMBT3906" H 5200 2850 50  0001 C CNN
 F 2 "smd-semi:SOT-23" H 4900 2900 50  0001 C CNN

Commit message: Nicer BOM lines
Parts:
- C72: OldReference C1 -> (none)
- C73: OldReference C2 -> (none)
- C74: OldReference C3 -> (none)
- C75: OldReference C4 -> (none)
- D5: BOM SEMI GENERIC MMBD4148 -> DIODE MMBD4148; OldReference D1 -> (none)
- D6: BOM SEMI GENERIC MMBD4148 -> DIODE MMBD4148; OldReference D2 -> (none)
- Q11: BOM SEMI GENERIC MMBT3904 -> NPN MMBT3904; OldReference Q14 -> (none)
- Q12: BOM SEMI GENERIC MMBT3906 -> PNP MMBT3906; OldReference Q1 -> (none)
- Q13: BOM SEMI IRF IRLML6402 -> PMOS IRF IRLML6402; OldReference Q2 -> (none)
- Q14: BOM SEMI AOS AOD417 -> PMOS AOS AOD417; OldReference Q3 -> (none)
- R81: OldReference R1 -> (none)
- R82: OldReference R2 -> (none)
- R83: OldReference R3 -> (none)
- R84: OldReference R112 -> (none)
- R85: OldReference R4 -> (none)
- R86: OldReference R9 -> (none)
- R87: OldReference R10 -> (none)
- R88: OldReference R11 -> (none)
- U11: OldReference U1 -> (none)
- U12: OldReference U2 -> (none)
Changed lines of the file:
@@
 F 6 "DIST DIGIKEY 507-1801-1-ND" H 1800 1700 60  0001 C CNN "BOM"
 F 7 "PPTC 350mA/750mA 30V [1206]" H 1800 1700 60  0001 C CNN "Description"
-F 8 "R1" H 1800 1700 50  0001 C CNN "OldReference"
 	1    1800 1700
 	0    -1   1    0
@@
 F 3 "" H 7390 1875 60  0000 C CNN
 F 4 "CAP MLCC 100n ≥X7R 20V 10% [0805]" H 8200 2450 60  0001 C CNN "BOM"
-F 5 "C3" H 7400 1900 50  0001 C CNN "OldReference"
 	1    7400 1900
 	1    0    0    -1
@@
 F 3 "" V 4200 3850 60  0000 C CNN
 F 4 "IC GENERIC LM393M" H 4200 3700 60  0001 C CNN "BOM"
-F 5 "U2" H 4200 3700 50  0001 C CNN "OldReference"
 	2    4200 3700
 	1    0    0    -1
@@
 F 2 "smd-semi:SOT-23" H 4900 2900 50  0001 C CNN
 F 3 "" H 4900 2900 60  0000 C CNN
-F 4 "" H 4900 2900 60  0001 C CNN "Manuf"
-F 5 "SEMI GENERIC MMBT3906" H 5700 3450 60  0001 C CNN "BOM"
-F 6 "Q1" H 4900 2900 50  0001 C CNN "OldReference"
+F 4 "PNP MMBT3906" H 5700 3450 60  0001 C CNN "BOM"
 	1    4900 2900
 	1    0    0    -1
@@
 F 3 "" V 4200 4750 60  0000 C CNN
 F 4 "IC GENERIC LM393M" H 4200 4600 60  0001 C CNN "BOM"
-F 5 "U2" H 4200 4600 50  0001 C CNN "OldReference"
 	1    4200 4600
 	1    0    0    -1
@@
 F 2 "smd-semi:SOT-23" H 4250 4100 50  0001 C CNN
 F 3 "" H 4250 4100 60  0000 C CNN
-F 4 "SEMI GENERIC MMBD4148" H 4250 4100 60  0001 C CNN "BOM"
-F 5 "D1" H 4250 4100 50  0001 C CNN "OldReference"
+F 4 "DIODE MMBD4148" H 4250 4100 60  0001 C CNN "BOM"
 	1    4250 4100
 	0    -1   -1   0
@@
 F 3 "" H 2400 5400 60  0000 C CNN
 F 4 "IC TI TL431AIDBZ" H 2400 5400 60  0001 C CNN "BOM"
-F 5 "U1" H 2400 5400 50  0001 C CNN "OldReference"
 	1    2400 5400
 	1    0    0    -1
@@
 F 2 "" H 2400 5650 60  0000 C CNN
 F 3 "" H 2400 5650 60  0000 C CNN
-F 4 "#PWR0206" H 2400 5650 50  0001 C CNN "OldReference"
 	1    2400 5650
 	1    0    0    -1
@@
 F 2 "" H 3500 5600 60  0000 C CNN
 F 3 "" H 3500 5600 60  0000 C CNN
-F 4 "#PWR0207" H 3500 5600 50  0001 C CNN "OldReference"
 	1    3500 5600
 	1    0    0    -1
@@
 F 2 "" H 3800 5600 60  0000 C CNN
 F 3 "" H 3800 5600 60  0000 C CNN
-F 4 "#PWR0208" H 3800 5600 50  0001 C CNN "OldReference"
 	1    3800 5600
 	1    0    0    -1
@@
 F 2 "smd-semi:SOT-23" H 4600 2100 50  0001 C CNN
 F 3 "" H 4600 2100 60  0000 C CNN
-F 4 "SEMI GENERIC MMBD4148" H 4600 2100 60  0001 C CNN "BOM"
-F 5 "D2" H 4600 2100 50  0001 C CNN "OldReference"
+F 4 "DIODE MMBD4148" H 4600 2100 60  0001 C CNN "BOM"
 	1    4600 2100
 	1    0    0    -1
@@
 F 3 "" V 5600 3950 60  0000 C CNN
 F 4 "IC GENERIC LM393M" H 5600 3800 60  0001 C CNN "BOM"
-F 5 "U2" H 5600 3800 50  0001 C CNN "OldReference"
 	3    5600 3800
 	1    0    0    -1
@@
 F 3 "" H 5840 3775 60  0000 C CNN
 F 4 "CAP MLCC 100n ≥X7R 20V 10% [0805]" H 6650 4350 60  0001 C CNN "BOM"
-F 5 "C2" H 5850 3800 50  0001 C CNN "OldReference"
 	1    5850 3800
 	1    0    0    -1
@@
 F 2 "" H 5850 4000 60  0000 C CNN
 F 3 "" H 5850 4000 60  0000 C CNN
-F 4 "#PWR0209" H 5850 4000 50  0001 C CNN "OldReference"
 	1    5850 4000
 	1    0    0    -1
@@
 F 2 "" H 5600 4300 60  0000 C CNN
 F 3 "" H 5600 4300 60  0000 C CNN
-F 4 "#PWR0210" H 5600 4300 50  0001 C CNN "OldReference"
 	1    5600 4300
 	1    0    0    -1
@@
 F 2 "" H 4150 5600 60  0000 C CNN
 F 3 "" H 4150 5600 60  0000 C CNN
-F 4 "#PWR0211" H 4150 5600 50  0001 C CNN "OldReference"
 	1    4150 5600
 	1    0    0    -1
@@
 F 4 "IRLML6402TRPBF" H 7100 1900 60  0001 C CNN "PN"
 F 5 "IRF" H 6700 1750 100 0001 C CNN "Manuf"
-F 6 "SEMI IRF IRLML6402" H 7500 2300 60  0001 C CNN "BOM"
-F 7 "Q2" H 6700 1750 50  0001 C CNN "OldReference"
+F 6 "PMOS IRF IRLML6402" H 7500 2300 60  0001 C CNN "BOM"
 	1    6700 1750
 	0    1    -1   0
@@
 F 4 "AOD417" H 8450 1900 60  0001 C CNN "PN"
 F 5 "AOS" H 8100 1750 50  0001 C CNN "Manuf"
-F 6 "SEMI AOS AOD417" H 8850 2300 60  0001 C CNN "BOM"
-F 7 "Q3" H 8100 1750 50  0001 C CNN "OldReference"
+F 6 "PMOS AOS AOD417" H 8850 2300 60  0001 C CNN "BOM"
 	1    8100 1750
 	0    -1   -1   0
@@
 F 2 "smd-semi:SOT-23" H 3250 5900 50  0001 C CNN
 F 3 "" H 3250 5900 60  0000 C CNN
-F 4 "SEMI GENERIC MMBT3904" H 4050 6450 60  0001 C CNN "BOM"
-F 5 "" H 3250 5900 60  0001 C CNN "Manuf"
-F 6 "Q14" H 3250 5900 50  0001 C CNN "OldReference"
+F 4 "NPN MMBT3904" H 4050 6450 60  0001 C CNN "BOM"
 	1    3250 5900
 	1    0    0    -1
@@
 F 2 "" H 3300 6050 60  0000 C CNN
 F 3 "" H 3300 6050 60  0000 C CNN
-F 4 "#PWR0212" H 3300 6050 50  0001 C CNN "OldReference"
 	1    3300 6050
 	1    0    0    -1
@@
 F 2 "" H 3050 6600 60  0000 C CNN
 F 3 "" H 3050 6600 60  0000 C CNN
-F 4 "#PWR0213" H 3050 6600 50  0001 C CNN "OldReference"
 	1    3050 6600
 	1    0    0    -1
@@
 F 6 "DIST DIGIKEY YC164J-10KCT-ND" H 3500 2500 60  0001 C CNN "BOM"
 F 7 "RESPACK SMD 10k 5% [4x0603]" H 3500 2500 60  0001 C CNN "Description"
-F 8 "R112" H 3500 2500 50  0001 C CNN "OldReference"
 	1    3500 2500
 	-1   0    0    -1
@@
 F 6 "DIST DIGIKEY YC164J-10KCT-ND" H 3500 2800 60  0001 C CNN "BOM"
 F 7 "RESPACK SMD 10k 5% [4x0603]" H 3500 2800 60  0001 C CNN "Description"
-F 8 "R112" H 3500 2800 50  0001 C CNN "OldReference"
 	2    3500 2800
 	-1   0    0    -1
@@
 F 6 "DIST DIGIKEY YC164J-10KCT-ND" H 3800 2500 60  0001 C CNN "BOM"
 F 7 "RESPACK SMD 10k 5% [4x0603]" H 3800 2500 60  0001 C CNN "Description"
-F 8 "R112" H 3800 2500 50  0001 C CNN "OldReference"
 	3    3800 2500
 	1    0    0    -1
@@
 F 6 "DIST DIGIKEY YC164J-10KCT-ND" H 3800 2800 60  0001 C CNN "BOM"
 F 7 "RESPACK SMD 10k 5% [4x0603]" H 3800 2800 60  0001 C CNN "Description"
-F 8 "R112" H 3800 2800 50  0001 C CNN "OldReference"
 	4    3800 2800
 	1    0    0    -1
@@
 F 6 "DIST DIGIKEY YC164J-10KCT-ND" H 3800 3100 60  0001 C CNN "BOM"
 F 7 "RESPACK SMD 10k 5% [4x0603]" H 3800 3100 60  0001 C CNN "Description"
-F 8 "R4" H 3800 3100 50  0001 C CNN "OldReference"
 	4    3800 3100
 	1    0    0    -1
@@
 F 6 "DIST DIGIKEY YC164J-10KCT-ND" H 3800 5400 60  0001 C CNN "BOM"
 F 7 "RESPACK SMD 10k 5% [4x0603]" H 3800 5400 60  0001 C CNN "Description"
-F 8 "R4" H 3800 5400 50  0001 C CNN "OldReference"
 	3    3800 5400
 	1    0    0    1
@@
 F 6 "DIST DIGIKEY YC164J-10KCT-ND" H 3500 5400 60  0001 C CNN "BOM"
 F 7 "RESPACK SMD 10k 5% [4x0603]" H 3500 5400 60  0001 C CNN "Description"
-F 8 "R4" H 3500 5400 50  0001 C CNN "OldReference"
 	1    3500 5400
 	1    0    0    -1
@@
 F 6 "DIST DIGIKEY YC164J-10KCT-ND" H 3050 6400 60  0001 C CNN "BOM"
 F 7 "RESPACK SMD 10k 5% [4x0603]" H 3050 6400 60  0001 C CNN "Description"
-F 8 "R3" H 3050 6400 50  0001 C CNN "OldReference"
 	2    3050 6400
 	1    0    0    -1
@@
 F 6 "DIST DIGIKEY YC164J-10KCT-ND" H 2750 6200 60  0001 C CNN "BOM"
 F 7 "RESPACK SMD 10k 5% [4x0603]" H 2750 6200 60  0001 C CNN "Description"
-F 8 "R3" H 2750 6200 50  0001 C CNN "OldReference"
 	3    2750 6200
 	0    1    1    0
@@
 F 6 "DIST DIGIKEY YC164J-10KCT-ND" H 3250 3800 60  0001 C CNN "BOM"
 F 7 "RESPACK SMD 10k 5% [4x0603]" H 3250 3800 60  0001 C CNN "Description"
-F 8 "R3" H 3250 3800 50  0001 C CNN "OldReference"
 	1    3250 3800
 	0    -1   1    0
@@
 F 6 "DIST DIGIKEY YC164J-10KCT-ND" H 4600 2700 60  0001 C CNN "BOM"
 F 7 "RESPACK SMD 10k 5% [4x0603]" H 4600 2700 60  0001 C CNN "Description"
-F 8 "R3" H 4600 2700 50  0001 C CNN "OldReference"
 	4    4600 2700
 	1    0    0    1
@@
 F 4 "" H 8400 2100 60  0001 C CNN "Manuf"
 F 5 "CAP MLCC 10n ≥X5R 50V 10% [0603]" H 9200 2650 60  0001 C CNN "BOM"
-F 6 "C4" H 8400 2100 50  0001 C CNN "OldReference"
 	1    8400 2100
 	0    1    1    0
@@
 F 4 "" H 4150 5400 60  0001 C CNN "Manuf"
 F 5 "CAP MLCC 10n ≥X5R 50V 10% [0603]" H 4950 5950 60  0001 C CNN "BOM"
-F 6 "C1" H 4150 5400 50  0001 C CNN "OldReference"
 	1    4150 5400
 	1    0    0    -1
@@
 F 4 "" H 2400 2500 60  0001 C CNN "Manuf"
 F 5 "RES SMD 3.3k 5% [0603]" H 3150 3050 60  0001 C CNN "BOM"
-F 6 "R2" H 2400 2500 50  0001 C CNN "OldReference"
 	1    2400 2500
 	1    0    0    -1
@@
 F 4 "" H 4750 4600 60  0001 C CNN "Manuf"
 F 5 "RES SMD 1M 5% [0603]" H 5500 5150 60  0001 C CNN "BOM"
-F 6 "R10" H 4750 4600 50  0001 C CNN "OldReference"
 	1    4750 4600
 	0    1    1    0
@@
 F 4 "" H 4600 3300 60  0001 C CNN "Manuf"
 F 5 "RES SMD 3.3k 5% [0603]" H 5350 3850 60  0001 C CNN "BOM"
-F 6 "R9" H 4600 3300 50  0001 C CNN "OldReference"
 	1    4600 3300
 	1    0    0    -1
@@
 F 4 "" H 7000 1900 60  0001 C CNN "Manuf"
 F 5 "RES SMD 1M 5% [0603]" H 7750 2450 60  0001 C CNN "BOM"
-F 6 "R11" H 7000 1900 50  0001 C CNN "OldReference"
 	1    7000 1900
 	-1   0    0    1
