File: wcp52/PowerInput.sch (KiCad schematic (older format))
At the start: 20 parts, among them Q11 MMBT3904, Q12 MMBT3906, Q13 IRLML6402, Q14 AOD417, U11 TL431AIDBZ, U12 LM393M

Commit message: Add post-testing revision, todo notes
Connections:
- net D5A: now reaches D5.1, R83.8, U12.5
- net D5K: now reaches D5.3, R86.2, U12.7
Other:
- note added: "DO NOT POPULATE!"
- note added: "This diode exists on the PCB from pin 5 to pin 7 of U12. The\noriginal purpose was to provide a latching mechanism for the\novervoltage lockout, but it was a flawed design and prevented\nthe supply from starting.\n\nThis footprint should be left unpopulated. The power supply\nwill continue to function as intended, but with a non-latching\nOVLO.\n\nTODO (REV 2):\nRevise OVLO latching to work prope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"
- moved on the sheet: D5
Changed lines of the file:
@@
 Sheet 11 13
 Title "Power Input Circuit"
-Date "2015-03-21"
-Rev ""
+Date "2015-03-31"
+Rev "1"
 Comp "WCP52"
 Comment1 "Gain/Phase Analyzer"
@@
 $EndComp
 Wire Wire Line
-	4600 3400 4600 4100
-Wire Wire Line
 	4600 3700 4500 3700
 Wire Wire Line
@@
 L MMBD4148 D5
 U 1 1 54F4BCC5
-P 4250 4100
-F 0 "D5" V 4450 4100 50  0000 C CNN
-F 1 "MMBD4148" V 4350 4100 50  0000 C CNN
-F 2 "smd-semi:SOT-23" H 4250 4100 50  0001 C CNN
-F 3 "" H 4250 4100 60  0000 C CNN
-F 4 "DIODE MMBD4148" H 4250 4100 60  0001 C CNN "BOM"
-	1    4250 4100
+P 7850 5250
+F 0 "D5" V 7950 5250 50  0000 C CNN
+F 1 "MMBD4148" V 7950 5250 50  0001 C CNN
+F 2 "smd-semi:SOT-23" H 7850 5250 50  0001 C CNN
+F 3 "" H 7850 5250 60  0000 C CNN
+F 4 "DIODE MMBD4148" H 7850 5250 60  0001 C CNN "BOM"
+	1    7850 5250
 	0    -1   -1   0
 $EndComp
 Wire Wire Line
-	4600 4100 4350 4100
-Connection ~ 4600 3700
-Wire Wire Line
-	4150 4100 3900 4100
-Wire Wire Line
-	3900 4100 3900 3800
-Wire Wire Line
 	3350 3800 4000 3800
-Connection ~ 3900 3800
 Wire Wire Line
 	3500 4500 4000 4500
@@
 Connection ~ 2400 4700
 $Comp
-L GND #PWR207
+L GND #PWR0207
 U 1 1 54F4C586
 P 2400 5650
-F 0 "#PWR207" H 2400 5650 30  0001 C CNN
+F 0 "#PWR0207" H 2400 5650 30  0001 C CNN
 F 1 "GND" H 2400 5580 30  0001 C CNN
 F 2 "" H 2400 5650 60  0000 C CNN
@@
 $EndComp
 $Comp
-L GND #PWR210
+L GND #PWR0208
 U 1 1 54F4C600
 P 3500 5600
-F 0 "#PWR210" H 3500 5600 30  0001 C CNN
+F 0 "#PWR0208" H 3500 5600 30  0001 C CNN
 F 1 "GND" H 3500 5530 30  0001 C CNN
 F 2 "" H 3500 5600 60  0000 C CNN
@@
 	3500 5600 3500 5500
 $Comp
-L GND #PWR211
+L GND #PWR0209
 U 1 1 54F4C674
 P 3800 5600
-F 0 "#PWR211" H 3800 5600 30  0001 C CNN
+F 0 "#PWR0209" H 3800 5600 30  0001 C CNN
 F 1 "GND" H 3800 5530 30  0001 C CNN
 F 2 "" H 3800 5600 60  0000 C CNN
@@
 Connection ~ 5600 2500
 $Comp
-L GND #PWR214
+L GND #PWR0210
 U 1 1 54F4D4FF
 P 5850 4000
-F 0 "#PWR214" H 5850 4000 30  0001 C CNN
+F 0 "#PWR0210" H 5850 4000 30  0001 C CNN
 F 1 "GND" H 5850 3930 30  0001 C CNN
 F 2 "" H 5850 4000 60  0000 C CNN
@@
 	5850 4000 5850 3900
 $Comp
-L GND #PWR213
+L GND #PWR0211
 U 1 1 54F4D5D3
 P 5600 4300
-F 0 "#PWR213" H 5600 4300 30  0001 C CNN
+F 0 "#PWR0211" H 5600 4300 30  0001 C CNN
 F 1 "GND" H 5600 4230 30  0001 C CNN
 F 2 "" H 5600 4300 60  0000 C CNN
@@
 Connection ~ 3800 5200
 $Comp
-L GND #PWR212
+L GND #PWR0212
 U 1 1 54F4E909
 P 4150 5600
-F 0 "#PWR212" H 4150 5600 30  0001 C CNN
+F 0 "#PWR0212" H 4150 5600 30  0001 C CNN
 F 1 "GND" H 4150 5530 30  0001 C CNN
 F 2 "" H 4150 5600 60  0000 C CNN
@@
 	3300 4900 3300 5800
 $Comp
-L GND #PWR209
+L GND #PWR0213
 U 1 1 54F7D2C2
 P 3300 6050
-F 0 "#PWR209" H 3300 6050 30  0001 C CNN
+F 0 "#PWR0213" H 3300 6050 30  0001 C CNN
 F 1 "GND" H 3300 5980 30  0001 C CNN
 F 2 "" H 3300 6050 60  0000 C CNN
@@
 	3050 5900 3150 5900
 $Comp
-L GND #PWR208
+L GND #PWR0214
 U 1 1 54F7D63A
 P 3050 6600
-F 0 "#PWR208" H 3050 6600 30  0001 C CNN
+F 0 "#PWR0214" H 3050 6600 30  0001 C CNN
 F 1 "GND" H 3050 6530 30  0001 C CNN
 F 2 "" H 3050 6600 60  0000 C CNN
@@
 	-1   0    0    1
 $EndComp
+Wire Wire Line
+	4600 3400 4600 4000
+Text Notes 7450 5050 0    80   ~ 0
+DO NOT POPULATE!
+Text Notes 7450 6250 0    50   ~ 0
+This diode exists on the PCB from pin 5 to pin 7 of U12. The\noriginal purpose was to provide a latching mechanism for the\novervoltage lockout, but it was a flawed design and prevented\nthe supply from starting.\n\nThis footprint should be left unpopulated. The power supply\nwill continue to function as intended, but with a non-latching\nOVLO.\n\nTODO (REV 2):\nRevise OVLO latching to work properly.
+Wire Notes Line
+	7400 4850 10000 4850
+Wire Notes Line
+	10000 4850 10000 6350
+Wire Notes Line
+	10000 6350 7400 6350
+Wire Notes Line
+	7400 6350 7400 4850
+Wire Wire Line
+	3900 3800 3900 4000
+Wire Wire Line
+	3900 4000 4000 4000
+Connection ~ 3900 3800
+Text Label 4000 4000 0    50   ~ 0
+D5A
+Wire Wire Line
+	4600 4000 4500 4000
+Connection ~ 4600 3700
+Text Label 4500 4000 2    50   ~ 0
+D5K
+Text Label 7750 5250 2    50   ~ 0
+D5A
+Text Label 7950 5250 0    50   ~ 0
+D5K
 $EndSCHEMATC

Commit message: Fix BOM
D5 was removed, so should not be in the BOM
Parts:
- D5: BOM DIODE MMBD4148 -> #DIODE MMBD4148
Changed lines of the file:
@@
 F 2 "smd-semi:SOT-23" H 7850 5250 50  0001 C CNN
 F 3 "" H 7850 5250 60  0000 C CNN
-F 4 "DIODE MMBD4148" H 7850 5250 60  0001 C CNN "BOM"
+F 4 "#DIODE MMBD4148" H 7850 5250 60  0001 C CNN "BOM"
 	1    7850 5250
 	0    -1   -1   0
