File: PCB/wcp52/MPU.sch (KiCad schematic (older format))
At the start: 58 parts, among them J7 AVR-ICSP, J8 JLINK, U17 ATMEGA32U4-AU-DNP, U18 ATSAM4S16CA-AU, X2 12MHz

Commit message: Update documentation
Correct LaTeX Makefile: don't include README.rst

Add local .gitignore

Add microcontroller documentation

Update schematic renders
Parts:
- U18: value ATSAM4S16CA-AU -> ATSAM4S4CA-AU; BOM IC ATMEL ATSAM4S16CA-AU -> IC ATMEL ATSAM4S4CA-AU
Changed lines of the file:
@@
 EESchema Schematic File Version 2
-LIBS:Altera
-LIBS:AnalogDevices
-LIBS:Atmel
-LIBS:conn-2mm
-LIBS:conn-100mil
-LIBS:conn-cui
-LIBS:conn-fci
-LIBS:conn-linx
-LIBS:conn-molex
-LIBS:conn-tagconnect
-LIBS:conn-test
-LIBS:DiodesInc
-LIBS:display
-LIBS:_electromech
-LIBS:Fairchild
-LIBS:FTDI
-LIBS:Intersil
-LIBS:Lattice
-LIBS:_linear
-LIBS:LinearTech
-LIBS:Littelfuse
-LIBS:logic-4000
-LIBS:logic-7400
-LIBS:MACOM
-LIBS:maxim
-LIBS:mechanical
-LIBS:Microchip
-LIBS:Micron
-LIBS:NXP
-LIBS:onsemi
-LIBS:passive
-LIBS:pasv-BiTech
-LIBS:pasv-Bourns
-LIBS:pasv-cap
-LIBS:pasv-ind
-LIBS:pasv-res
-LIBS:pcb
-LIBS:power
-LIBS:_semi
-LIBS:semi-diode-1N
-LIBS:semi-diode-BA
-LIBS:semi-diode-MCC
-LIBS:semi-diode-MMB
-LIBS:semi-diode-NXP
-LIBS:semi-diode-OnSemi
-LIBS:semi-diode-Vishay
-LIBS:semi-opto-misc
-LIBS:semi-thyristor-2N
-LIBS:semi-trans-2N
-LIBS:semi-trans-AO
-LIBS:semi-trans-BC
-LIBS:semi-trans-DiodesInc
-LIBS:semi-trans-Fairchild
-LIBS:semi-trans-Infineon
-LIBS:semi-trans-IntRect
-LIBS:semi-trans-IXYS
-LIBS:semi-trans-misc
-LIBS:semi-trans-MMB
-LIBS:semi-trans-MPS
-LIBS:semi-trans-NXP
-LIBS:semi-trans-PZT
-LIBS:semi-trans-TI
-LIBS:semi-trans-TIP
-LIBS:semi-trans-Toshiba
-LIBS:silabs
-LIBS:skyworks
-LIBS:ST
-LIBS:st_ic
-LIBS:st_semi
-LIBS:supertex
-LIBS:symbol
-LIBS:TexasInstruments
-LIBS:vishay_semi
-LIBS:Xilinx
-LIBS:pasv-xtal
-LIBS:conn-te
 LIBS:wcp52-cache
 EELAYER 25 0
@@
 P 5700 3950
 F 0 "U18" H 5700 6850 50  0000 C CNN
-F 1 "ATSAM4S16CA-AU" H 5700 6750 50  0000 C CNN
+F 1 "ATSAM4S4CA-AU" H 5700 6750 50  0000 C CNN
 F 2 "IPC7351-Nominal:QFP50P1600X1600X160-100" H 5700 6700 50  0001 C CNN
 F 3 "" H 5700 6700 50  0000 C CNN
-F 4 "Atmel" H 6100 7250 50  0001 C CNN "Manuf"
-F 5 "ATSAM4S16CA-AU" H 5800 6950 50  0001 C CNN "PN"
-F 6 "IC ATMEL ATSAM4S16CA-AU" H 6200 7350 50  0001 C CNN "BOM"
+F 4 "ATSAM4S16CA-AU" H 5800 6950 50  0001 C CNN "PN"
+F 5 "Atmel" H 6100 7250 50  0001 C CNN "Manuf"
+F 6 "IC ATMEL ATSAM4S4CA-AU" H 6200 7350 50  0001 C CNN "BOM"
 	1    5700 3950
 	1    0    0    -1
